File: PCB_S/ALU/ALU.kicad_sch (KiCad schematic)
At the start: 293 parts, among them J1 Conn_01x08_Socket, J2 Conn_01x08_Socket, J3 Conn_01x08_Socket, J4 Conn_01x01_Socket, J5 Conn_01x10_Socket, Q1 2N7002, Q10 2N7002, Q100 2N7002, Q101 2N7002, Q102 2N7002, Q103 2N7002, Q104 2N7002, Q105 2N7002, Q106 2N7002, Q107 2N7002, Q108 2N7002, Q109 2N7002, Q11 2N7002, Q110 2N7002, Q111 2N7002, Q112 2N7002, Q113 2N7002, Q114 2N7002, Q115 2N7002, Q116 2N7002, Q117 2N7002, Q118 2N7002, Q119 2N7002, Q12 2N7002, Q120 2N7002, Q121 2N7002, Q122 2N7002, Q123 2N7002, Q124 2N7002, Q125 2N7002, Q126 2N7002, Q127 2N7002, Q128 2N7002, Q129 2N7002, Q13 2N7002, Q130 2N7002, Q131 2N7002, Q132 2N7002, Q133 2N7002, Q134 2N7002, Q135 2N7002, Q136 2N7002, Q137 2N7002, Q138 2N7002, Q139 2N7002, Q14 2N7002, Q140 2N7002, Q141 2N7002, Q142 2N7002, Q143 2N7002, Q144 2N7002, Q145 2N7002, Q146 2N7002, Q147 2N7002, Q148 2N7002, Q149 2N7002, Q15 2N7002, Q150 2N7002, Q151 2N7002, Q152 2N7002, Q153 2N7002, Q154 2N7002, Q155 2N7002, Q156 2N7002, Q157 2N7002, Q158 2N7002, Q159 2N7002, Q16 2N7002, Q160 2N7002, Q161 2N7002, Q162 2N7002, Q163 2N7002, Q164 2N7002, Q165 2N7002, Q166 2N7002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

Commit message: ALU_pcb
Parts:
- removed Q155, Q156, Q157, Q158, Q159, Q160, Q161, Q162, Q163, Q164, Q165, Q166, Q167, Q168, Q169, Q170, Q171, Q172, Q173, Q174, Q175, Q176: 2N7002, PCM_JLCPCB:Q_SOT-23, symbol PCM_JLCPCB-Transistors:NMOS,2N7002
- removed R105, R106, R107, R108, R109, R110, R111, R112: 10kΩ, PCM_JLCPCB:R_0402, symbol PCM_JLCPCB-Resistors:0402,10kΩ
- J4: footprint Connector_Hirose:Hirose_DF63R-1P-3.96DSA_1x01_P3.96mm_Vertical -> Connector_PinHeader_2.54mm:PinHeader_1x01_P2.54mm_Vertical
Connections:
- net GND: now also Q101.2 (S), Q106.2 (S), Q113.2 (S), Q116.2 (S), Q121.2 (S), Q128.2 (S), Q131.2 (S), Q136.2 (S), Q143.2 (S), Q26.2 (S), Q35.2 (S), Q38.2 (S), Q41.2 (S), Q61.2 (S), Q63.2 (S), Q65.2 (S), Q71.2 (S), Q76.2 (S), Q83.2 (S), Q86.2 (S), Q91.2 (S), Q98.2 (S); no longer Q100.2 (S), Q105.2 (S), Q112.2 (S), Q115.2 (S), Q120.2 (S), Q127.2 (S), Q130.2 (S), Q135.2 (S), Q142.2 (S), Q145.2 (S), Q148.2 (S), Q150.2 (S), Q153.2 (S), Q25.2 (S), Q27.2 (S), Q30.2 (S), Q34.2 (S), Q36.2 (S), Q37.2 (S), Q39.2 (S), Q40.2 (S), Q42.2 (S), Q45.2 (S), Q49.2 (S), Q51.2 (S), Q52.2 (S), Q54.2 (S), Q55.2 (S), Q60.2 (S), Q62.2 (S), Q64.2 (S), Q70.2 (S), Q75.2 (S), Q82.2 (S), Q85.2 (S), Q90.2 (S), Q97.2 (S)
- net at Q34.3 (D): now also Q25.1 (G), Q30.1 (G), Q35.1 (G), R23.2; no longer Q35.2 (S)
- net at R90.2: now also Q125.3 (D), Q126.2 (S); no longer Q139.3 (D)
- net at R26.2: now also Q29.1 (G), Q37.3 (D), Q38.1 (G); no longer Q39.3 (D)
- net at Q63.3 (D), R44.2: now also Q55.2 (S), Q64.2 (S); no longer Q61.1 (G)
- net at Q60.3 (D): now also Q73.1 (G), R42.2; no longer Q61.2 (S)
- net at J2.1 (Pin_1), Q23.1 (G): now also Q139.1 (G), Q141.1 (G); no longer Q47.1 (G)
- net at Q32.3 (D), R21.2: no longer Q33.1 (G)
- net at Q33.3 (D), R22.2: now also Q25.2 (S), Q34.2 (S)
- net at Q147.2 (S): now also Q145.2 (S), Q146.2 (S), Q148.2 (S), Q149.2 (S), Q150.2 (S), Q151.2 (S), Q152.2 (S), Q153.2 (S), Q154.2 (S)
- net at R37.2: now also Q44.1 (G), Q52.3 (D), Q53.1 (G); no longer Q53.3 (D)
- net at R28.2: now also Q40.3 (D), Q41.1 (G); no longer Q42.3 (D)
- net at J2.3 (Pin_3), Q17.1 (G): no longer Q140.1 (G), Q41.1 (G)
- net at R63.2: now also Q89.3 (D), Q91.1 (G); no longer Q94.3 (D)
- net at R98.2: now also Q137.3 (D); no longer Q152.3 (D)
- net at Q80.3 (D), Q81.2 (S): now also R57.2; no longer Q72.2 (S)
- net at Q28.3 (D), Q29.2 (S): now also Q37.2 (S)
- net at Q110.3 (D), Q111.2 (S): now also R79.2; no longer Q102.2 (S)
- net at J2.6 (Pin_6), Q8.1 (G): now also Q64.1 (G), Q66.1 (G); no longer Q32.1 (G), Q95.1 (G)
- net at J1.2 (Pin_2), Q19.1 (G): now also Q123.1 (G); no longer Q43.1 (G), Q55.1 (G)
- net at Q97.3 (D): now also Q89.1 (G), Q98.1 (G), R70.2; no longer Q98.2 (S)
- net at Q84.1 (G), R51.2: now also Q72.3 (D), Q82.1 (G); no longer Q74.3 (D), Q86.1 (G)
- net at Q54.3 (D), R38.2: now also Q47.1 (G)
- net at Q124.3 (D): now also Q115.1 (G), Q120.1 (G), Q125.1 (G), R89.2; no longer R81.2
- net at J2.2 (Pin_2), Q20.1 (G): now also Q124.1 (G), Q126.1 (G); no longer Q44.1 (G)
- net at Q148.3 (D): no longer Q149.2 (S)
- net at J2.5 (Pin_5), Q11.1 (G): now also Q79.1 (G), Q81.1 (G); no longer Q110.1 (G), Q35.1 (G)
- net at Q95.3 (D), Q96.2 (S): now also R68.2; no longer Q87.2 (S)
- net at R96.2: now also Q134.3 (D), Q136.1 (G); no longer Q149.3 (D)
- net at Q150.3 (D): no longer Q151.2 (S)
- net at R102.2: now also Q132.1 (G), Q141.3 (D); no longer Q151.1 (G)
- net at R103.2: now also Q134.1 (G), Q142.3 (D), Q143.1 (G); no longer Q154.1 (G)
- net at Q118.3 (D), Q119.2 (S): now also Q127.2 (S)
- net at R32.2: now also Q47.3 (D), Q62.3 (D), R43.2; no longer Q48.3 (D)
- net at R36.2: now also Q42.1 (G), Q51.3 (D); no longer Q52.3 (D)
- net at Q112.3 (D): now also Q104.1 (G), Q113.1 (G), R81.2; no longer Q113.2 (S)
- net at R104.2: now also Q137.1 (G), Q144.3 (D)
- net at Q73.3 (D), Q74.2 (S): now also Q82.2 (S)
- net at Q55.3 (D), R39.2: now also Q56.1 (G)
- net at R35.2: now also Q50.3 (D), Q51.2 (S); no longer Q51.3 (D)
- net at Q133.1 (G), R86.2: now also Q120.3 (D); no longer Q132.3 (D)
- net at R30.2: now also Q44.3 (D), Q46.1 (G); no longer Q45.3 (D)
- net at R101.2: now also Q140.3 (D), Q141.2 (S); no longer Q149.1 (G)
- net at J1.1 (Pin_1), Q22.1 (G): now also Q138.1 (G); no longer Q46.1 (G), Q56.1 (G)
- net at J4.1 (Pin_1): no longer Q64.1 (G)
- net at Q30.3 (D), R20.2: now also Q43.1 (G)
- net at Q70.3 (D): now also Q71.1 (G), R50.2; no longer Q71.2 (S)
- net at Q71.3 (D): now also Q72.2 (S); no longer R49.2
- net at R99.2: now also Q130.2 (S), Q138.3 (D), Q139.2 (S); no longer Q154.3 (D)
- net at Q108.3 (D), Q109.2 (S): now also Q100.2 (S), R77.2
- net at Q109.3 (D): now also Q100.1 (G), Q105.1 (G), Q110.1 (G), R78.2; no longer R72.2
- net at Q58.3 (D), Q59.2 (S): now also Q67.2 (S); no longer Q57.2 (S)
- net at Q127.3 (D): now also Q119.1 (G), Q128.1 (G), R92.2; no longer Q128.2 (S)
- net at Q133.3 (D), Q134.2 (S): now also Q142.2 (S)
- net at J2.7 (Pin_7), Q5.1 (G): now also Q49.1 (G), Q51.1 (G); no longer Q29.1 (G), Q80.1 (G)
- net at Q29.3 (D), R19.2: now also Q31.1 (G); no longer Q30.1 (G)
- net at Q68.3 (D), Q69.2 (S): now also Q60.2 (S); no longer Q67.2 (S)
- net at Q88.3 (D), Q89.2 (S): now also Q97.2 (S)
- net at Q49.3 (D): now also Q40.1 (G), Q45.1 (G), Q50.1 (G), R34.2; no longer R33.2
- net at Q123.3 (D), Q124.2 (S): now also Q115.2 (S), R88.2
- net at Q103.3 (D), Q104.2 (S): now also Q112.2 (S)
- net at Q78.3 (D), Q79.2 (S): now also Q70.2 (S), R55.2
- net at Q79.3 (D): now also Q70.1 (G), Q75.1 (G), Q80.1 (G), R56.2; no longer R54.2
- net at Q153.3 (D): no longer Q154.2 (S)
- net at Q93.3 (D), Q94.2 (S): now also Q85.2 (S), R66.2
- net at Q43.3 (D), Q44.2 (S): now also Q52.2 (S)
- net at J2.8 (Pin_8), Q2.1 (G): now also Q34.1 (G), Q36.1 (G); no longer Q26.1 (G), Q58.1 (G)
- net at J2.4 (Pin_4), Q14.1 (G): now also Q94.1 (G), Q96.1 (G); no longer Q125.1 (G), Q38.1 (G)
- net at R24.2: now also Q35.3 (D), Q36.2 (S); no longer Q36.3 (D)
- net at Q82.3 (D): now also Q74.1 (G), Q83.1 (G), R59.2; no longer Q83.2 (S)
- net at R40.2: now also Q57.3 (D), Q67.1 (G), Q69.1 (G); no longer Q56.3 (D)
- net at Q25.3 (D): now also Q26.1 (G), R17.2; no longer Q26.2 (S)
- new net: Q102.1 (G), Q111.3 (D), R80.2
- new net: Q101.3 (D), Q102.2 (S)
- new net: Q102.3 (D), Q112.1 (G), Q114.1 (G), R73.2
- new net: Q92.1 (G), Q99.3 (D), R71.2
- new net: Q91.3 (D), Q92.2 (S)
- new net: Q92.3 (D), R65.2
- new net: Q103.1 (G), Q90.3 (D), R64.2
- new net: Q74.3 (D), Q76.1 (G), R52.2
- new net: Q76.3 (D), Q77.2 (S)
- new net: Q117.1 (G), Q126.3 (D), R91.2
- new net: Q30.2 (S), Q38.3 (D), Q39.2 (S)
- new net: Q116.3 (D), Q117.2 (S)
- new net: Q117.3 (D), Q127.1 (G), Q129.1 (G), R84.2
- new net: Q72.1 (G), Q81.3 (D), R58.2
- new net: Q32.1 (G), Q39.3 (D), R27.2
- new net: Q109.1 (G), Q111.1 (G)
- new net: Q132.3 (D), Q142.1 (G), Q144.1 (G), R95.2
- new net: Q135.2 (S), Q143.3 (D), Q144.2 (S)
- new net: Q119.3 (D), Q121.1 (G), R85.2
- new net: Q121.3 (D), Q122.2 (S)
- new net: Q45.3 (D), Q58.1 (G), R31.2
- new net: Q37.1 (G), Q39.1 (G)
- new net: Q130.1 (G), Q135.1 (G), Q139.3 (D), Q140.1 (G), R100.2
- new net: Q135.3 (D), R97.2
- new net: Q130.3 (D), Q131.1 (G), R94.2
- new net: Q105.2 (S), Q113.3 (D), Q114.2 (S)
- new net: Q105.3 (D), Q118.1 (G), R75.2
- new net: Q131.3 (D), Q132.2 (S)
- new net: Q87.1 (G), Q96.3 (D), R69.2
- new net: Q86.3 (D), Q87.2 (S)
- new net: Q87.3 (D), Q97.1 (G), Q99.1 (G), R62.2
- new net: Q56.3 (D), Q57.2 (S)
- new net: J1.4 (Pin_4), Q13.1 (G), Q93.1 (G)
- new net: Q107.3 (D), R76.2
- new net: Q90.2 (S), Q98.3 (D), Q99.2 (S)
- new net: Q107.1 (G), Q114.3 (D), R82.2
- new net: Q104.3 (D), Q106.1 (G), R74.2
- new net: Q85.3 (D), Q86.1 (G), R61.2
- new net: Q85.1 (G), Q90.1 (G), Q94.3 (D), Q95.1 (G), R67.2
- new net: Q115.3 (D), Q116.1 (G), R83.2
- new net: Q106.3 (D), Q107.2 (S)
- new net: Q62.1 (G), Q69.3 (D), R49.2
- new net: Q61.3 (D), Q62.2 (S)
- new net: Q41.3 (D), Q42.2 (S)
- new net: Q40.2 (S), Q48.3 (D), Q49.2 (S), R33.2
- new net: Q42.3 (D), Q52.1 (G), Q54.1 (G), R29.2
- new net: Q55.1 (G), Q60.1 (G), Q64.3 (D), Q65.1 (G), R45.2
- new net: Q59.3 (D), Q61.1 (G), R41.2
- new net: Q100.3 (D), Q101.1 (G), R72.2
- new net: Q65.3 (D), Q66.2 (S), R46.2
- new net: Q57.1 (G), Q66.3 (D), R47.2
- new net: J1.6 (Pin_6), Q63.1 (G), Q7.1 (G)
- new net: Q26.3 (D), Q27.2 (S)
- new net: J1.7 (Pin_7), Q4.1 (G), Q48.1 (G)
- new net: Q59.1 (G), Q67.3 (D), Q68.1 (G), R48.2
- new net: Q27.1 (G), Q36.3 (D), R25.2
- new net: Q75.2 (S), Q83.3 (D), Q84.2 (S)
- new net: Q77.1 (G), Q84.3 (D), R60.2
- new net: Q77.3 (D), R54.2
- new net: J1.3 (Pin_3), Q108.1 (G), Q16.1 (G)
- new net: J1.8 (Pin_8), Q1.1 (G), Q33.1 (G)
- new net: Q75.3 (D), Q88.1 (G), R53.2
- new net: J1.5 (Pin_5), Q10.1 (G), Q78.1 (G)
- new net: Q45.2 (S), Q53.3 (D), Q54.2 (S)
- new net: Q122.3 (D), R87.2
- new net: Q120.2 (S), Q128.3 (D), Q129.2 (S)
- new net: Q122.1 (G), Q129.3 (D), R93.2
- new net: Q136.3 (D), Q137.2 (S)
- now unconnected: Q145.1 (G), Q145.3 (D), Q146.1 (G), Q146.3 (D), Q147.1 (G), Q147.3 (D), Q148.1 (G), Q150.1 (G), Q151.3 (D), Q152.1 (G), Q153.1 (G), Q28.1 (G)
Other:
- moved on the sheet: J1, J2, J3, J4, J5, Q1, Q10, Q11, Q12, Q13, Q14, Q15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
