File: PCB_S/REG8bit-SMD-V4.0/REG8bit-SMD-V4.0.kicad_sch (KiCad schematic)
At the start: 118 parts, among them J2 Conn_01x21_Pin, Q1 2N7002, Q10 2N7002, Q11 2N7002, Q12 2N7002, Q13 2N7002, Q14 2N7002, Q15 2N7002, Q17 2N7002, Q19 2N7002, Q2 2N7002, Q20 2N7002, Q21 2N7002, Q22 2N7002, Q23 2N7002, Q24 2N7002, Q25 2N7002, Q27 2N7002, Q29 2N7002, Q3 2N7002, Q30 2N7002, Q31 2N7002, Q32 2N7002, Q33 2N7002, Q34 2N7002, Q35 2N7002, Q37 2N7002, Q39 2N7002, Q4 2N7002, Q40 2N7002, Q41 2N7002, Q42 2N7002, Q43 2N7002, Q44 2N7002, Q45 2N7002, Q47 2N7002, Q49 2N7002, Q5 2N7002, Q50 2N7002, Q51 2N7002, Q52 2N7002, Q53 2N7002, Q54 2N7002, Q55 2N7002, Q57 2N7002, Q59 2N7002, Q6 2N7002, Q60 2N7002, Q61 2N7002, Q62 2N7002, Q63 2N7002, Q64 2N7002, Q65 2N7002, Q67 2N7002, Q69 2N7002, Q70 2N7002, Q71 2N7002, Q72 2N7002, Q73 2N7002, Q74 2N7002, Q75 2N7002, Q77 2N7002, Q79 2N7002, Q80 2N7002, Q81 2N7002, Q82 2N7002, Q83 2N7002, Q84 2N7002, Q85 2N7002, Q86 2N7002, Q87 2N7002, Q88 2N7002, Q89 2N7002, Q9 2N7002

Commit message: New Register half done
Parts:
- removed J2: Conn_01x21_Pin, Connector_PinHeader_2.54mm:PinHeader_1x21_P2.54mm_Horizontal, symbol Connector:Conn_01x21_Pin
- removed R42, R43, R44, R45, R46, R47, R48, R49, R50: 470Ω, PCM_JLCPCB:R_0402, symbol PCM_JLCPCB-Resistors:0402,470Ω
- added J1: Conn_01x20_Pin, Connector_PinHeader_2.54mm:PinHeader_1x20_P2.54mm_Horizontal, symbol Connector:Conn_01x20_Pin
- added R11, R13, R16, R18, R21, R23, R3, R6, R8: 470Ω, PCM_JLCPCB:R_0603, symbol PCM_JLCPCB-Resistors:0603,470Ω
- R1, R10, R12, R14, R15, R17, R19, R2, R20, R22, R24, R25, R27, R29, R30, R32, R34, R35, R37, R39, R4, R40, R5, R7, R9: value 20kΩ -> 10kΩ
Connections:
- net Earth: now also J1.19 (Pin_19)
- net R: now also J1.17 (Pin_17)
- net RST: now also J1.18 (Pin_18)
- net VCC: now also J1.20 (Pin_20), R11.1, R13.1, R16.1, R18.1, R21.1, R23.1, R3.1, R6.1, R8.1
- net at Q44.3 (D), Q45.3 (D), Q47.1 (G)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: now also J1.4 (Pin_4)
- net at Q24.3 (D), Q25.3 (D), Q27.1 (G)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: now also J1.6 (Pin_6)
- net at D2.2: now also R8.2
- net at Q64.3 (D), Q65.3 (D), Q67.1 (G)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: now also J1.2 (Pin_2)
- net at Q72.1 (G), Q81.1 (G): now also J1.9 (Pin_9)
- net at Q14.3 (D), Q15.3 (D), Q17.1 (G)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: now also J1.7 (Pin_7)
- net at D5.2: now also R16.2
- net at D7.2: now also R21.2
- net at D6.2: now also R18.2
- net at Q52.1 (G), Q61.1 (G): now also J1.11 (Pin_11)
- net at Q4.3 (D), Q5.3 (D), Q6.1 (G)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: now also J1.8 (Pin_8)
- net at Q34.3 (D), Q35.3 (D), Q37.1 (G)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: now also J1.5 (Pin_5)
- net at D3.2: now also R11.2
- net at Q11.1 (G), Q2.1 (G): now also J1.16 (Pin_16)
- net at Q42.1 (G), Q51.1 (G): now also J1.12 (Pin_12)
- net at Q74.3 (D), Q75.3 (D), Q77.1 (G)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: now also J1.1 (Pin_1)
- net at Q22.1 (G), Q31.1 (G): now also J1.14 (Pin_14)
- net at Q54.3 (D), Q55.3 (D), Q57.1 (G)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: now also J1.3 (Pin_3)
- net at Q62.1 (G), Q71.1 (G): now also J1.10 (Pin_10)
- net at D4.2: now also R13.2
- net at Q32.1 (G), Q41.1 (G): now also J1.13 (Pin_13)
- net at Q12.1 (G), Q21.1 (G): now also J1.15 (Pin_15)
- net at D9.2: now also R3.2
- net at D8.2: now also R23.2
- net at D1.2: now also R6.2

Commit message: sim
Tried the spice sim : the sim did not work at all
Parts:
- added D10: Red, PCM_JLCPCB:D_0603, symbol PCM_JLCPCB-Diodes:LED,0603,Red
- added Q7: 2N7002, Package_TO_SOT_SMD:SOT-23, symbol Transistor_FET:2N7002
- added R26: 2.2kΩ, PCM_JLCPCB:R_0603, symbol PCM_JLCPCB-Resistors:0603,470Ω
- R11, R13, R16, R18, R21, R23, R3, R6, R8: value 470Ω -> 2.2kΩ
Connections:
- net Earth: now also Q7.2 (S)
- net R: now also Q7.1 (G)
- net VCC: now also R26.1
- new net: D10.1, Q7.3 (D)
- new net: D10.2, R26.2
