File: PCB_S/REG8bit-SMD-V4.2/REG8bit-SMD-V4.2.kicad_sch (KiCad schematic)
At the start: 124 parts, among them J1 Conn_01x21_Pin, Q1 2N7002, Q10 2N7002, Q11 2N7002, Q12 2N7002, Q13 2N7002, Q14 2N7002, Q15 2N7002, Q16 2N7002, Q17 2N7002, Q19 2N7002, Q2 2N7002, Q20 2N7002, Q21 2N7002, Q22 2N7002, Q23 2N7002, Q24 2N7002, Q25 2N7002, Q27 2N7002, Q29 2N7002, Q3 2N7002, Q30 2N7002, Q31 2N7002, Q32 2N7002, Q33 2N7002, Q34 2N7002, Q35 2N7002, Q37 2N7002, Q39 2N7002, Q4 2N7002, Q40 2N7002, Q41 2N7002, Q42 2N7002, Q43 2N7002, Q44 2N7002, Q45 2N7002, Q47 2N7002, Q49 2N7002, Q5 2N7002, Q50 2N7002, Q51 2N7002, Q52 2N7002, Q53 2N7002, Q54 2N7002, Q55 2N7002, Q57 2N7002, Q59 2N7002, Q6 2N7002, Q60 2N7002, Q61 2N7002, Q62 2N7002, Q63 2N7002, Q64 2N7002, Q65 2N7002, Q67 2N7002, Q69 2N7002, Q7 2N7002, Q70 2N7002, Q71 2N7002, Q72 2N7002, Q73 2N7002, Q74 2N7002, Q75 2N7002, Q77 2N7002, Q79 2N7002, Q8 2N7002, Q80 2N7002, Q81 2N7002, Q82 2N7002, Q83 2N7002, Q84 2N7002, Q85 2N7002, Q86 2N7002, Q87 2N7002, Q88 2N7002, Q89 2N7002, Q9 2N7002

Commit message: 8-Bit register is done
Parts:
- removed C1: 10uF, PCM_JLCPCB:C_0805, symbol PCM_JLCPCB-Capacitors:0805,10uF
- removed R26: 10kΩ, PCM_JLCPCB:R_0402, symbol PCM_JLCPCB-Resistors:0402,20kΩ
- removed R28: 470Ω, PCM_JLCPCB:R_0603, symbol PCM_JLCPCB-Resistors:0603,470Ω
- added C1, C2, C3, C4: 22uF, PCM_JLCPCB:C_0805, symbol PCM_JLCPCB-Capacitors:0805,22uF
- added R26: 2.2kΩ, PCM_JLCPCB:R_0603, symbol PCM_JLCPCB-Resistors:0603,470Ω
- added R28: 10kΩ, PCM_JLCPCB:R_0402, symbol PCM_JLCPCB-Resistors:0402,20kΩ
- J1: footprint (none) -> Connector_PinHeader_2.54mm:PinHeader_1x21_P2.54mm_Horizontal
- R11, R13, R16, R18, R21, R23, R3, R6, R8: value 470Ω -> 2.2kΩ
Connections:
- net Earth: now also Q7.2 (S), C1.2, C2.2, C3.2, C4.2; no longer Q16.2 (S)
- net VCC: now also C1.1, C2.1, C3.1, C4.1, R26.1, R28.1
- net at Q8.3 (D): now also Q16.2 (S); no longer Q7.2 (S)
- net at Q1.1 (G), Q13.1 (G), Q23.1 (G)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: now also Q16.3 (D), R28.2; no longer Q7.3 (D)
- net at J1.11 (Pin_11), Q52.1 (G), Q61.1 (G): no longer J1.12 (Pin_12), Q42.1 (G), Q51.1 (G)
- net Rise_egde: now reaches J1.17 (Pin_17), Q16.1 (G)
- net Rise_egde: no longer Q7.1 (G)
- net at D10.1: now also Q7.3 (D); no longer Q16.3 (D)
- net at D10.2: now also R26.2
- net RisingEdge renamed R
- net R: now also Q7.1 (G)
- new net: J1.12 (Pin_12), Q42.1 (G), Q51.1 (G)
