File: PCB_S/REG8bit-SMD-V4.2/REG8bit-SMD-V4.2.kicad_pcb (KiCad board)
At the start: 4 copper layers, 73.7 x 31.8 mm, 128 parts, among them J1 Conn_01x21_Pin, Q1 2N7002, Q10 2N7002, Q11 2N7002, Q12 2N7002, Q13 2N7002, Q14 2N7002, Q15 2N7002, Q16 2N7002, Q17 2N7002, Q19 2N7002, Q2 2N7002, Q20 2N7002, Q21 2N7002, Q22 2N7002, Q23 2N7002, Q24 2N7002, Q25 2N7002, Q27 2N7002, Q29 2N7002, Q3 2N7002, Q30 2N7002, Q31 2N7002, Q32 2N7002, Q33 2N7002, Q34 2N7002, Q35 2N7002, Q37 2N7002, Q39 2N7002, Q4 2N7002, Q40 2N7002, Q41 2N7002, Q42 2N7002, Q43 2N7002, Q44 2N7002, Q45 2N7002, Q47 2N7002, Q49 2N7002, Q5 2N7002, Q50 2N7002, Q51 2N7002, Q52 2N7002, Q53 2N7002, Q54 2N7002, Q55 2N7002, Q57 2N7002, Q59 2N7002, Q6 2N7002, Q60 2N7002, Q61 2N7002, Q62 2N7002, Q63 2N7002, Q64 2N7002, Q65 2N7002, Q67 2N7002, Q69 2N7002, Q7 2N7002, Q70 2N7002, Q71 2N7002, Q72 2N7002, Q73 2N7002, Q74 2N7002, Q75 2N7002, Q77 2N7002, Q79 2N7002, Q8 2N7002, Q80 2N7002, Q81 2N7002, Q82 2N7002, Q83 2N7002, Q84 2N7002, Q85 2N7002, Q86 2N7002, Q87 2N7002, Q88 2N7002, Q89 2N7002, Q9 2N7002

Commit message: sendt the reg8bit
Routing:
- net Net-(J1-Pin_12): track 31.5 -> 24.5 mm
Changed lines of the file:
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@@
-	)
-	(segment
-		(start 89.8 146.1)
-		(end 90.5 146.8)
-		(width 0.2)
-		(layer "B.Cu")
-		(net 50)
 	)
 	(segment
@@
 		(start 82.8 148.2)
 		(end 89.1 148.2)
-		(width 0.2)
-		(layer "B.Cu")
-		(net 50)
-	)
-	(segment
-		(start 83.8 146.1)
-		(end 89.8 146.1)
 		(width 0.2)
 		(layer "B.Cu")
@@
 		(min_thickness 0.25)
 		(filled_areas_thickness no)
-		(fill
+		(fill yes
 			(thermal_gap 0.5)
 			(thermal_bridge_width 0.5)
@@
 		(min_thickness 0.25)
 		(filled_areas_thickness no)
-		(fill
+		(fill yes
 			(thermal_gap 0.5)
 			(thermal_bridge_width 0.5)
