File: PCB_S/ALU_V1.0/ALU_V1.0.kicad_pcb (KiCad board)
At the start: 6 copper layers, 127.5 x 100 mm, 543 parts, among them J1 Conn_01x08_Socket, J2 Conn_01x08_Socket, J3 Conn_01x08_Socket, J4 Conn_01x02_Pin, J5 Conn_01x02_Pin, J6 Conn_01x02_Pin, J8 Conn_01x14_Pin, Q1 2N7002, Q10 2N7002, Q100 2N7002, Q101 2N7002, Q102 2N7002, Q103 2N7002, Q104 2N7002, Q105 2N7002, Q106 2N7002, Q107 2N7002, Q108 2N7002, Q109 2N7002, Q11 2N7002, Q110 2N7002, Q111 2N7002, Q112 2N7002, Q113 2N7002, Q114 2N7002, Q115 2N7002, Q116 2N7002, Q117 2N7002, Q118 2N7002, Q119 2N7002, Q12 2N7002, Q120 2N7002, Q121 2N7002, Q122 2N7002, Q123 2N7002, Q124 2N7002, Q125 2N7002, Q126 2N7002, Q127 2N7002, Q128 2N7002, Q129 2N7002, Q13 2N7002, Q130 2N7002, Q131 2N7002, Q132 2N7002, Q133 2N7002, Q134 2N7002, Q135 2N7002, Q136 2N7002, Q137 2N7002, Q138 2N7002, Q139 2N7002, Q14 2N7002, Q140 2N7002, Q141 2N7002, Q142 2N7002, Q143 2N7002, Q144 2N7002, Q145 2N7002, Q146 2N7002, Q147 2N7002, Q148 2N7002, Q149 2N7002, Q15 2N7002, Q150 2N7002, Q151 2N7002, Q152 2N7002, Q153 2N7002, Q154 2N7002, Q155 2N7002, Q156 2N7002, Q157 2N7002, Q158 2N7002, Q159 2N7002, Q16 2N7002, Q160 2N7002, Q161 2N7002, Q162 2N7002, Q163 2N7002, Q164 2N7002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

Commit message: ALU_V1.0_Done
Parts:
- added G***: LOGO, HVL_L:HVL_LOGO_15mm, F.Cu at (56.7, 77.2)
Other:
- board text added: "ALU_V1.0"
- board text added: "Arithmetic"
- board text removed: "LOGIC"
Changed lines of the file:
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@@
 			(at 5.375 5.3 90)
 			(layer "F.SilkS")
+			(hide yes)
 			(effects
 				(font
@@
 			(at 0 -2.38 0)
 			(layer "F.SilkS")
+			(hide yes)
 			(effects
 				(font
@@
 		)
 	)
+	(footprint "HVL_L:HVL_LOGO_15mm"
+		(layer "F.Cu")
+		(at 56.7 77.2 -90)
+		(property "Reference" "G***"
+			(at 0 0 90)
+			(layer "F.SilkS")
+			(hide yes)
+			(effects
+				(font
+					(size 1.5 1.5)
+					(thickness 0.3)
+				)
+			)
+		)
+		(property "Value" "LOGO"
+			(at 0.75 0 90)
+			(layer "F.SilkS")
+			(hide yes)
+			(effects
+				(font
+					(size 1.5 1.5)
+					(thickness 0.3)
+				)
+			)
+		)
+		(property "Datasheet" ""
+			(at 0 0 90)
+			(layer "F.Fab")
+			(hide yes)
+			(effects
+				(font
+					(size 1.27 1.27)
+					(thickness 0.15)
+				)
+			)
+		)
+		(property "Description" ""
+			(at 0 0 90)
+			(layer "F.Fab")
+			(hide yes)
+			(effects
+				(font
+					(size 1.27 1.27)
+					(thickness 0.15)
+				)
+			)
+		)
+		(attr board_only exclude_from_pos_files exclude_from_bom)
+		(fp_poly
+			(pts
+				(xy -5.589789 -6.528044) (xy -4.471832 -4.59367) (xy -4.163325 -4.057163) (xy -3.885162 -3.568253)
+				(xy -3.649851 -3.149347) (xy -3.469899 -2.822851) (xy -3.357816 -2.611173) (xy -3.325605 -2.540407)
+				(xy -3.356708 -2.419783) (xy -3.460163 -2.187103) (xy -3.614705 -1.882732) (xy -3.799071 -1.547035)
+				(xy -3.991995 -1.220377) (xy -4.15041 -0.974721) (xy -4.190725 -0.960441) (xy -4.259259 -1.010625)
+				(xy -4.364138 -1.137804) (xy -4.513486 -1.354511) (xy -4.715429 -1.673278) (xy -4.978093 -2.106636)
+				(xy -5.309602 -2.667118) (xy -5.718083 -3.367255) (xy -5.858099 -3.608556) (xy -6.229822 -4.250338)
+				(xy -6.572882 -4.84368) (xy -6.876988 -5.370701) (xy -7.131846 -5.813521) (xy -7.327167 -6.15426)
+				(xy -7.452659 -6.375038) (xy -7.49777 -6.457251) (xy -7.42698 -6.486108) (xy -7.212235 -6.509324)
+				(xy -6.88843 -6.524255) (xy -6.558686 -6.528459)
+			)
+			(stroke
+				(width 0)
+				(type solid)
+			)
+			(fill yes)
+			(layer "F.SilkS")
+		)
+		(fp_poly
+			(pts
+				(xy 5.605307 -6.526464) (xy 6.198258 -6.519653) (xy 6.705589 -6.509066) (xy 7.105344 -6.49533) (xy 7.375568 -6.479069)
+				(xy 7.494305 -6.460911) (xy 7.497769 -6.456201) (xy 7.44242 -6.35266) (xy 7.306184 -6.110847) (xy 7.097115 -5.744612)
+				(xy 6.823273 -5.267806) (xy 6.492711 -4.694281) (xy 6.113488 -4.037887) (xy 5.693659 -3.312474)
+				(xy 5.241282 -2.531895) (xy 4.764411 -1.71) (xy 4.271105 -0.86064) (xy 3.769419 0.002335) (xy 3.26741 0.865072)
+				(xy 2.773133 1.713723) (xy 2.294647 2.534435) (xy 1.840007 3.313357) (xy 1.417269 4.036639) (xy 1.034491 4.69043)
+				(xy 0.699728 5.260879) (xy 0.421036 5.734135) (xy 0.206474 6.096347) (xy 0.064096 6.333664) (xy 0.001959 6.432235)
+				(xy -0.000001 6.434206) (xy -0.05457 6.359673) (xy -0.186055 6.149762) (xy -0.382571 5.824368) (xy -0.63223 5.403386)
+				(xy -0.923149 4.906712) (xy -1.243442 4.35424) (xy -1.267623 4.312312) (xy -1.590232 3.750782) (xy -1.883072 3.237301)
+				(xy -2.134267 2.792995) (xy -2.331942 2.438993) (xy -2.464221 2.196421) (xy -2.519229 2.086406)
+				(xy -2.519736 2.084772) (xy -2.481638 1.989481) (xy -2.361487 1.754069) (xy -2.167316 1.392945)
+				(xy -1.907156 0.920522) (xy -1.58904 0.35121) (xy -1.221 -0.300581) (xy -0.811068 -1.02044) (xy -0.367277 -1.793955)
+				(xy -0.089572 -2.275263) (xy 2.369801 -6.528874) (xy 4.948691 -6.528874)
+			)
+			(stroke
+				(width 0)
+				(type solid)
+			)
+			(fill yes)
+			(layer "F.SilkS")
+		)
+		(embedded_fonts no)
+	)
 	(footprint "PCM_JLCPCB:R_0402"
 		(layer "F.Cu")
@@
 			(at 0 -2.38 0)
 			(layer "F.SilkS")
+			(hide yes)
 			(effects
 				(font
@@
 			(at 16.25 3.4 90)
 			(layer "F.Fab")
+			(hide yes)
 			(effects
 				(font
@@
 			(layer "F.Fab")
 		)
-		(fp_text user "${REFERENCE}"
-			(at 16.25 1.5 90)
-			(layer "F.Fab")
-			(effects
-				(font
-					(size 1 1)
-					(thickness 0.15)
-				)
-			)
-		)
 		(pad "1" thru_hole roundrect
 			(at 0 0 90)
@@
 		)
 	)
+	(gr_text "ALU_V1.0"
+		(at 59.5 28.9 270)
+		(layer "F.SilkS")
+		(effects
+			(font
+				(size 1 1)
+				(thickness 0.15)
+			)
+			(justify left bottom)
+		)
+	)
 	(gr_text "PWR"
 		(at 164.1 33.7 0)
@@
 			(font
 				(size 3 3)
-				(thickness 0.4)
+				(thickness 0.6)
+				(bold yes)
 			)
 			(justify bottom)
@@
 		)
 	)
-	(gr_text "LOGIC"
+	(gr_text "Arithmetic"
 		(at 84.6 32.8 0)
 		(layer "F.SilkS")
@@
 			(font
 				(size 3 3)
-				(thickness 0.4)
+				(thickness 0.6)
+				(bold yes)
 			)
 			(justify bottom)
@@
 		)
 	)
+	(gr_text "MSB"
+		(at 166.4 123.2 0)
+		(layer "F.SilkS")
+		(effects
+			(font
+				(size 1 1)
+				(thickness 0.1)
+			)
+			(justify bottom)
+		)
+	)
 	(gr_text "SJ"
-		(at 61.6 70.4 270)
+		(at 51.8 84.1 270)
 		(layer "F.SilkS")
 		(effects
@@
 		)
 	)
+	(gr_text "ALU_V1.0"
+		(at 59.5 35.7 270)
+		(layer "B.SilkS")
+		(effects
+			(font
+				(size 1 1)
+				(thickness 0.15)
+			)
+			(justify left bottom mirror)
+		)
+	)
