File: PCB_S/ALU_V1.0/ALU_V1.0.kicad_pcb (KiCad board)
At the start: 6 copper layers, 127.5 x 100 mm, 544 parts, among them J1 Conn_01x08_Socket, J2 Conn_01x08_Socket, J3 Conn_01x08_Socket, J4 Conn_01x02_Pin, J5 Conn_01x02_Pin, J6 Conn_01x02_Pin, J8 Conn_01x14_Pin, Q1 2N7002, Q10 2N7002, Q100 2N7002, Q101 2N7002, Q102 2N7002, Q103 2N7002, Q104 2N7002, Q105 2N7002, Q106 2N7002, Q107 2N7002, Q108 2N7002, Q109 2N7002, Q11 2N7002, Q110 2N7002, Q111 2N7002, Q112 2N7002, Q113 2N7002, Q114 2N7002, Q115 2N7002, Q116 2N7002, Q117 2N7002, Q118 2N7002, Q119 2N7002, Q12 2N7002, Q120 2N7002, Q121 2N7002, Q122 2N7002, Q123 2N7002, Q124 2N7002, Q125 2N7002, Q126 2N7002, Q127 2N7002, Q128 2N7002, Q129 2N7002, Q13 2N7002, Q130 2N7002, Q131 2N7002, Q132 2N7002, Q133 2N7002, Q134 2N7002, Q135 2N7002, Q136 2N7002, Q137 2N7002, Q138 2N7002, Q139 2N7002, Q14 2N7002, Q140 2N7002, Q141 2N7002, Q142 2N7002, Q143 2N7002, Q144 2N7002, Q145 2N7002, Q146 2N7002, Q147 2N7002, Q148 2N7002, Q149 2N7002, Q15 2N7002, Q150 2N7002, Q151 2N7002, Q152 2N7002, Q153 2N7002, Q154 2N7002, Q155 2N7002, Q156 2N7002, Q157 2N7002, Q158 2N7002, Q159 2N7002, Q16 2N7002, Q160 2N7002, Q161 2N7002, Q162 2N7002, Q163 2N7002, Q164 2N7002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

Commit message: ALU_V1.0 silk
Routing:
- net GND: track 584.7 -> 588.8 mm
- net Net-(Q147-G): track 180.0 -> 176.4 mm
- net Net-(Q152-G): track 92.7 -> 90.0 mm
- net Net-(Q153-G): track 76.4 -> 73.7 mm
- net Net-(Q154-G): track 49.2 -> 46.5 mm
- net Net-(Q12-D): track 108.9 -> 106.2 mm
- net Net-(Q148-G): track 157.5 -> 154.8 mm
- net Net-(Q149-G): track 141.3 -> 138.6 mm
- net Net-(Q15-D): track 125.1 -> 122.5 mm
- net Net-(J1-Pin_8): track 174.0 -> 171.5 mm
Other:
- board text added: "+"
- board text added: "-"
- board text added: "- +"
- board text added: "0"
- board text added: "1"
- board text added: "2"
- board text added: "3"
- board text added: "4"
- board text added: "5"
- board text added: "6"
- board text added: "7"
- board text added: "Ci"
- board text added: "N"
- board text added: "Result"
