File: PCB_S/ALU_V1.0/ALU_V1.0.kicad_sch (KiCad schematic)
At the start: 534 parts, among them J1 Conn_01x08_Socket, J2 Conn_01x08_Socket, J3 Conn_01x08_Socket, J4 Conn_01x01_Socket, J5 Conn_01x05_Pin, J6 Conn_01x06_Pin, Q1 2N7002, Q10 2N7002, Q100 2N7002, Q101 2N7002, Q102 2N7002, Q103 2N7002, Q104 2N7002, Q105 2N7002, Q106 2N7002, Q107 2N7002, Q108 2N7002, Q109 2N7002, Q11 2N7002, Q110 2N7002, Q111 2N7002, Q112 2N7002, Q113 2N7002, Q114 2N7002, Q115 2N7002, Q116 2N7002, Q117 2N7002, Q118 2N7002, Q119 2N7002, Q12 2N7002, Q120 2N7002, Q121 2N7002, Q122 2N7002, Q123 2N7002, Q124 2N7002, Q125 2N7002, Q126 2N7002, Q127 2N7002, Q128 2N7002, Q129 2N7002, Q13 2N7002, Q130 2N7002, Q131 2N7002, Q132 2N7002, Q133 2N7002, Q134 2N7002, Q135 2N7002, Q136 2N7002, Q137 2N7002, Q138 2N7002, Q139 2N7002, Q14 2N7002, Q140 2N7002, Q141 2N7002, Q142 2N7002, Q143 2N7002, Q144 2N7002, Q145 2N7002, Q146 2N7002, Q147 2N7002, Q148 2N7002, Q149 2N7002, Q15 2N7002, Q150 2N7002, Q151 2N7002, Q152 2N7002, Q153 2N7002, Q154 2N7002, Q155 2N7002, Q156 2N7002, Q157 2N7002, Q158 2N7002, Q159 2N7002, Q16 2N7002, Q160 2N7002, Q161 2N7002, Q162 2N7002, Q163 2N7002, Q164 2N7002, Q165 2N7002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

Commit message: ALU_V1.0
Creating the ALU PCB
Parts:
- added J7: Conn_01x02_Pin, Connector_JST:JST_EH_B2B-EH-A_1x02_P2.50mm_Vertical, symbol Connector:Conn_01x02_Pin
- Q1, Q10, Q100, Q101, Q102, Q103, Q104, Q105, Q106, Q107, Q108, Q109, Q11, Q110, Q111, Q112, Q113, Q114, Q115, Q116, Q117, Q118, Q119, Q12, Q120, Q121, Q122, Q123, Q124, Q125, Q126, Q127, Q128, Q129, Q13, Q130, Q131, Q132, Q133, Q134, Q135, Q136, Q137, Q138, Q139, Q14, Q140, Q141, Q142, Q143, Q144, Q145, Q146, Q147, Q148, Q149, Q15, Q150, Q151, Q152, Q153, Q154, Q155, Q156, Q157, Q158, Q159, Q16, Q160, Q161, Q162, Q163, Q164, Q165, Q166, Q167, Q168, Q169, Q17, Q170, Q171, Q172, Q173, Q174, Q175, Q176, Q177, Q178, Q179, Q18, Q180, Q181, Q182, Q183, Q184, Q185, Q186, Q187, Q188, Q189, Q19, Q190, Q191, Q192, Q193, Q194, Q195, Q196, Q197, Q198, Q199, Q2, Q20, Q200, Q201, Q202, Q203, Q204, Q205, Q206, Q207, Q208, Q209, Q21, Q210, Q211, Q212, Q213, Q214, Q215, Q216, Q217, Q218, Q219, Q22, Q220, Q221, Q222, Q223, Q224, Q225, Q226, Q227, Q228, Q229, Q23, Q230, Q231, Q232, Q233, Q234, Q235, Q236, Q237, Q238, Q239, Q24, Q240, Q241, Q242, Q243, Q244, Q245, Q246, Q247, Q248, Q249, Q25, Q250, Q251, Q252, Q253, Q254, Q255, Q256, Q257, Q258, Q259, Q26, Q260, Q261, Q262, Q263, Q264, Q265, Q266, Q267, Q268, Q269, Q27, Q270, Q271, Q277, Q278, Q279, Q28, Q280, Q281, Q282, Q283, Q284, Q285, Q286, Q287, Q288, Q289, Q29, Q290, Q3, Q30, Q31, Q32, Q33, Q34, Q35, Q36, Q37, Q38, Q39, Q4, Q40, Q41, Q42, Q43, Q44, Q45, Q46, Q47, Q48, Q49, Q5, Q50, Q51, Q52, Q53, Q54, Q55, Q56, Q57, Q58, Q59, Q6, Q60, Q61, Q62, Q63, Q64, Q65, Q66, Q67, Q68, Q69, Q7, Q70, Q71, Q72, Q73, Q74, Q75, Q76, Q77, Q78, Q79, Q8, Q80, Q81, Q82, Q83, Q84, Q85, Q86, Q87, Q88, Q89, Q9, Q90, Q91, Q92, Q93, Q94, Q95, Q96, Q97, Q98, Q99: footprint PCM_JLCPCB:Q_SOT-23 -> Package_TO_SOT_SMD:SOT-23
Connections:
- net GND: now also J7.2 (Pin_2)
- net VCC: now also J7.1 (Pin_1)
- net at Q239.3 (D), Q268.1 (G), Q273.1 (G)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: now also J3.8 (Pin_8); no longer J3.1 (Pin_1)
- net at Q13.1 (G), Q231.1 (G), Q306.1 (G)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: now also J1.4 (Pin_4); no longer J1.5 (Pin_5)
- net at Q286.3 (D), Q319.1 (G), R133.2: now also J5.2 (Pin_2); no longer J5.4 (Pin_4)
- net at Q124.1 (G), Q126.1 (G), Q20.1 (G)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: now also J2.2 (Pin_2); no longer J2.7 (Pin_7)
- net at Q241.3 (D), Q269.1 (G), Q272.1 (G)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: now also J3.7 (Pin_7); no longer J3.2 (Pin_2)
- net at Q268.3 (D), Q269.3 (D), Q270.3 (D)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: now also J5.4 (Pin_4); no longer J5.2 (Pin_2)
- net at Q253.3 (D), Q279.1 (G), Q282.1 (G)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: now also J3.1 (Pin_1), J5.5 (Pin_5); no longer J3.8 (Pin_8), J5.1 (Pin_1)
- net at Q11.1 (G), Q297.1 (G), Q79.1 (G)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: now also J2.5 (Pin_5); no longer J2.4 (Pin_4)
- net at Q243.3 (D), Q270.1 (G), Q274.1 (G)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: now also J3.6 (Pin_6); no longer J3.3 (Pin_3)
- net at Q245.3 (D), Q271.1 (G), Q275.1 (G)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: now also J3.5 (Pin_5); no longer J3.4 (Pin_4)
- net at Q247.3 (D), Q276.1 (G), Q287.1 (G)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: now also J3.4 (Pin_4); no longer J3.5 (Pin_5)
- net at Q249.3 (D), Q288.1 (G), Q291.1 (G)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: now also J3.3 (Pin_3); no longer J3.6 (Pin_6)
- net at Q251.3 (D), Q289.1 (G), Q292.1 (G)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: now also J3.2 (Pin_2); no longer J3.7 (Pin_7)
- net at Q109.1 (G), Q111.1 (G), Q17.1 (G)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: now also J2.3 (Pin_3); no longer J2.6 (Pin_6)
- net at Q123.1 (G), Q19.1 (G), Q235.1 (G)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: now also J1.2 (Pin_2); no longer J1.7 (Pin_7)
- net at Q108.1 (G), Q16.1 (G), Q233.1 (G)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: now also J1.3 (Pin_3); no longer J1.6 (Pin_6)
- net at Q10.1 (G), Q229.1 (G), Q305.1 (G)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: now also J1.5 (Pin_5); no longer J1.4 (Pin_4)
- net at Q138.1 (G), Q22.1 (G), Q237.1 (G)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: now also J1.1 (Pin_1); no longer J1.8 (Pin_8)
- net at Q227.1 (G), Q304.1 (G), Q63.1 (G)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: now also J1.6 (Pin_6); no longer J1.3 (Pin_3)
- net at Q265.3 (D), Q320.1 (G), R125.2: now also J5.1 (Pin_1); no longer J5.5 (Pin_5)
- net at Q225.1 (G), Q303.1 (G), Q4.1 (G)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: now also J1.7 (Pin_7); no longer J1.2 (Pin_2)
- net at Q139.1 (G), Q141.1 (G), Q23.1 (G)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: now also J2.1 (Pin_1); no longer J2.8 (Pin_8)
- net at Q295.1 (G), Q49.1 (G), Q5.1 (G)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: now also J2.7 (Pin_7); no longer J2.2 (Pin_2)
- net at Q1.1 (G), Q262.1 (G), Q302.1 (G)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: now also J1.8 (Pin_8); no longer J1.1 (Pin_1)
- net at Q296.1 (G), Q64.1 (G), Q66.1 (G)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: now also J2.6 (Pin_6); no longer J2.3 (Pin_3)
- net at Q14.1 (G), Q298.1 (G), Q94.1 (G)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: now also J2.4 (Pin_4); no longer J2.5 (Pin_5)
- net at Q2.1 (G), Q294.1 (G), Q34.1 (G)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: now also J2.8 (Pin_8); no longer J2.1 (Pin_1)
Other:
- note added: "Pin 1 is Most Significant Bit"
- moved on the sheet: J1, J2, J3

Commit message: ALU_V1.0 WIP
PCB size doesnt matter??
Parts:
- removed C1, C2, C3, C4: 22uF, PCM_JLCPCB:C_0805, symbol PCM_JLCPCB-Capacitors:0805,22uF
- removed J4: Conn_01x01_Socket, Connector_PinHeader_2.54mm:PinHeader_1x01_P2.54mm_Vertical, symbol Connector:Conn_01x01_Socket
- removed J5: Conn_01x05_Pin, Connector_JST:JST_EH_B5B-EH-A_1x05_P2.50mm_Vertical, symbol Connector:Conn_01x05_Pin
- removed J6: Conn_01x06_Pin, Connector_JST:JST_EH_B6B-EH-A_1x06_P2.50mm_Vertical, symbol Connector:Conn_01x06_Pin
- removed J7: Conn_01x02_Pin, Connector_JST:JST_EH_B2B-EH-A_1x02_P2.50mm_Vertical, symbol Connector:Conn_01x02_Pin
- added J8: Conn_01x14_Pin, Connector_JST:JST_EH_B14B-EH-A_1x14_P2.50mm_Vertical, symbol Connector:Conn_01x14_Pin
Connections:
- net Earth: now also J8.13 (Pin_13)
- net VCC: now also J8.14 (Pin_14)
- net at Q226.1 (G), Q228.1 (G), Q230.1 (G)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: now also J8.9 (Pin_9)
- net at Q155.1 (G), Q156.1 (G), Q157.1 (G)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: now also J8.11 (Pin_11)
- net at Q286.3 (D), Q319.1 (G), R133.2: now also J8.2 (Pin_2)
- net at Q178.1 (G), Q182.1 (G), Q186.1 (G)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: now also J8.8 (Pin_8)
- net at Q146.1 (G), Q164.1 (G), Q166.1 (G)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: now also J8.10 (Pin_10)
- net at Q210.1 (G), Q212.1 (G), Q214.1 (G)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: now also J8.6 (Pin_6)
- net at Q180.1 (G), Q184.1 (G), Q188.1 (G)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: now also J8.7 (Pin_7)
- net at Q268.3 (D), Q269.3 (D), Q270.3 (D)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: now also J8.4 (Pin_4)
- net at J3.1 (Pin_1), Q253.3 (D), Q279.1 (G)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: now also J8.5 (Pin_5)
- net at Q264.3 (D), Q318.1 (G), R124.2: now also J8.3 (Pin_3)
- net at Q265.3 (D), Q320.1 (G), R125.2: now also J8.1 (Pin_1)
- net at Q28.1 (G): now also J8.12 (Pin_12)

Commit message: ALU_V1.0 WIP
making pcb
Connections:
- net Earth is gone; now on net GND: D36.1, J8.13 (Pin_13), Q272.2 (S), Q273.2 (S), Q274.2 (S), Q275.2 (S), Q276.2 (S), Q291.2 (S), Q292.2 (S), Q293.2 (S), Q294.2 (S), Q295.2 (S), Q296.2 (S), Q297.2 (S), Q298.2 (S), Q299.2 (S), Q300.2 (S), Q301.2 (S), Q302.2 (S), Q303.2 (S), Q304.2 (S), Q305.2 (S), Q306.2 (S), Q307.2 (S), Q308.2 (S), Q309.2 (S), Q310.2 (S), Q311.2 (S), Q312.2 (S), Q313.2 (S), Q314.2 (S), Q315.2 (S), Q316.2 (S), Q317.2 (S), Q318.2 (S), Q319.2 (S), Q320.2 (S)

Commit message: ALU V1.0 done?
Parts:
- added H1, H2, H3, H4: MountingHole, MountingHole:MountingHole_3.2mm_M3, symbol Mechanical:MountingHole
Connections:
- net at Q213.1 (G), Q62.3 (D), R43.2: no longer Q211.1 (G), Q47.3 (D), R32.2
- new net: Q211.1 (G), Q47.3 (D), R32.2

Commit message: ALU V1.0 more done
Parts:
- added C1, C2, C3, C4, C5, C6, C7, C8: 22uF, PCM_JLCPCB:C_0805, symbol PCM_JLCPCB-Capacitors:0805,22uF
- added J4, J5, J6: Conn_01x02_Pin, Connector_PinHeader_2.54mm:PinHeader_1x02_P2.54mm_Vertical, symbol Connector:Conn_01x02_Pin
Connections:
- net GND: now also C1.2, C2.2, C3.2, C4.2, C5.2, C6.2, C7.2, C8.2, J4.2 (Pin_2), J5.2 (Pin_2), J6.2 (Pin_2)
- net VCC: now also C1.1, C2.1, C3.1, C4.1, C5.1, C6.1, C7.1, C8.1, J4.1 (Pin_1), J5.1 (Pin_1), J6.1 (Pin_1)
