File: PCB_S/Register_Holder_V1.0/Register_Holder_V1.0/Register_Holder_V1.0.kicad_sch (KiCad schematic)
At the start: 139 parts, among them J1 Conn_01x21_Socket, J10 Conn_01x08, J11 Conn_01x08, J2 Conn_01x21_Socket, J3 Conn_01x21_Socket, J4 Conn_01x21_Socket, J5 Conn_01x04_Pin, J6 Conn_01x04_Pin, J7 Conn_01x04_Pin, J8 Conn_01x04_Pin, J9 Conn_01x08, Q1 2N7002, Q10 2N7002, Q100 2N7002, Q101 2N7002, Q102 2N7002, Q103 2N7002, Q104 2N7002, Q105 2N7002, Q106 2N7002, Q107 2N7002, Q108 2N7002, Q109 2N7002, Q11 2N7002, Q110 2N7002, Q111 2N7002, Q112 2N7002, Q113 2N7002, Q114 2N7002, Q115 2N7002, Q116 2N7002, Q117 2N7002, Q118 2N7002, Q119 2N7002, Q12 2N7002, Q120 2N7002, Q121 2N7002, Q122 2N7002, Q123 2N7002, Q124 2N7002, Q125 2N7002, Q126 2N7002, Q127 2N7002, Q128 2N7002, Q13 2N7002, Q14 2N7002, Q15 2N7002, Q16 2N7002, Q17 2N7002, Q18 2N7002, Q19 2N7002, Q2 2N7002, Q20 2N7002, Q21 2N7002, Q22 2N7002, Q23 2N7002, Q24 2N7002, Q25 2N7002, Q26 2N7002, Q27 2N7002, Q28 2N7002, Q29 2N7002, Q3 2N7002, Q30 2N7002, Q31 2N7002, Q32 2N7002, Q33 2N7002, Q34 2N7002, Q35 2N7002, Q36 2N7002, Q37 2N7002, Q38 2N7002, Q39 2N7002, Q4 2N7002, Q40 2N7002, Q41 2N7002, Q42 2N7002, Q43 2N7002, Q44 2N7002, Q45 2N7002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

Commit message: REG holder V1.0
Parts:
- removed J6: Conn_01x04_Pin, Connector_PinHeader_2.54mm:PinHeader_1x04_P2.54mm_Vertical, symbol Connector:Conn_01x04_Pin
- added C1, C10, C11, C12, C13, C14, C15, C16, C2, C3, C4, C5, C6, C7, C8, C9: 22uF, PCM_JLCPCB:C_0805, symbol PCM_JLCPCB-Capacitors:0805,22uF
- added D1, D10, D11, D12, D13, D14, D15, D16, D2, D24, D3, D4, D5, D6, D7, D8, D9: Red, PCM_JLCPCB:D_0603, symbol PCM_JLCPCB-Diodes:LED,0603,Red
- added H1, H10, H11, H12, H13, H14, H15, H16, H2, H3, H4, H5, H6, H7, H8, H9: MountingHole, MountingHole:MountingHole_2.2mm_M2, symbol Mechanical:MountingHole
- added H17, H18, H19, H20: MountingHole, MountingHole:MountingHole_3.2mm_M3, symbol Mechanical:MountingHole
- added J12: Conn_01x08, Connector_PinHeader_2.54mm:PinHeader_1x08_P2.54mm_Vertical, symbol Connector_Generic:Conn_01x08
- added J13, J14, J15: Conn_01x02_Pin, Connector_PinHeader_2.54mm:PinHeader_1x02_P2.54mm_Vertical, symbol Connector:Conn_01x02_Pin
- added Q129, Q130, Q131, Q132, Q133, Q134, Q135, Q136, Q137, Q138, Q139, Q140, Q141, Q142, Q143, Q144, Q145, Q146, Q147, Q148, Q149, Q150, Q151, Q152, Q153, Q154, Q155, Q156, Q157, Q158, Q159, Q160: 2N7002, Package_TO_SOT_SMD:SOT-23, symbol Transistor_FET:2N7002
- added R1, R10, R11, R12, R13, R14, R15, R16, R17, R18, R19, R2, R20, R21, R22, R23, R24, R25, R26, R27, R28, R29, R3, R30, R31, R32, R4, R5, R6, R7, R8, R9: 10kΩ, PCM_JLCPCB:R_0402, symbol PCM_JLCPCB-Resistors:0402,10kΩ
- added R156, R33, R34, R35, R36, R37, R38, R39, R40, R41, R42, R43, R44, R45, R46, R47, R48: 2.2kΩ, PCM_JLCPCB:R_0603, symbol PCM_JLCPCB-Resistors:0603,470Ω
Connections:
- net GND: now also C1.2, C10.2, C11.2, C12.2, C13.2, C14.2, C15.2, C16.2, C2.2, C3.2, C4.2, C5.2, C6.2, C7.2, C8.2, C9.2, D8.1, J13.2 (Pin_2), J14.2 (Pin_2), J15.2 (Pin_2), Q129.2 (S), Q130.2 (S), Q131.2 (S), Q132.2 (S), Q133.2 (S), Q134.2 (S), Q135.2 (S), Q136.2 (S), Q137.2 (S), Q138.2 (S), Q139.2 (S), Q140.2 (S), Q141.2 (S), Q142.2 (S), Q143.2 (S), Q144.2 (S), Q145.2 (S), Q146.2 (S), Q147.2 (S), Q148.2 (S), Q149.2 (S), Q150.2 (S), Q151.2 (S), Q152.2 (S), Q153.2 (S), Q154.2 (S), Q155.2 (S), Q156.2 (S), Q157.2 (S), Q158.2 (S), Q159.2 (S), Q160.2 (S)
- net VCC: now also C1.1, C10.1, C11.1, C12.1, C13.1, C14.1, C15.1, C16.1, C2.1, C3.1, C4.1, C5.1, C6.1, C7.1, C8.1, C9.1, J13.1 (Pin_1), J14.1 (Pin_1), J15.1 (Pin_1), R1.1, R10.1, R11.1, R12.1, R13.1, R14.1, R15.1, R156.1, R16.1, R17.1, R18.1, R19.1, R2.1, R20.1, R21.1, R22.1, R23.1, R24.1, R25.1, R26.1, R27.1, R28.1, R29.1, R3.1, R30.1, R31.1, R32.1, R33.1, R34.1, R35.1, R36.1, R37.1, R38.1, R39.1, R4.1, R40.1, R41.1, R42.1, R43.1, R44.1, R45.1, R46.1, R47.1, R48.1, R5.1, R6.1, R7.1, R8.1, R9.1
- net at Q53.1 (G): now also J7.3 (Pin_3), Q49.1 (G), Q50.1 (G), Q51.1 (G), Q52.1 (G), Q54.1 (G), Q55.1 (G), Q56.1 (G), Q149.1 (G)
- net at Q115.1 (G): now also J8.4 (Pin_4), Q113.1 (G), Q114.1 (G), Q116.1 (G), Q117.1 (G), Q118.1 (G), Q119.1 (G), Q120.1 (G), Q152.1 (G)
- net at Q127.3 (D), Q47.3 (D), Q79.3 (D)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: now also Q138.1 (G), R18.2; no longer J11.7 (Pin_7)
- net at Q106.3 (D), Q26.3 (D), Q3.3 (D)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: now also Q135.1 (G), R15.2; no longer J10.2 (Pin_2)
- net at Q126.3 (D), Q46.3 (D), Q78.3 (D)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: now also Q139.1 (G), R19.2; no longer J11.6 (Pin_6)
- net at Q11.3 (D), Q110.3 (D), Q30.3 (D)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: now also Q131.1 (G), R11.2; no longer J10.6 (Pin_6)
- net at Q121.3 (D), Q41.3 (D), Q73.3 (D)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: now also Q144.1 (G), R24.2; no longer J11.1 (Pin_1)
- net at J1.10 (Pin_10), J2.10 (Pin_10), J3.10 (Pin_10)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: now also J9.5 (Pin_5), J12.5 (Pin_5), Q156.1 (G); no longer J9.4 (Pin_4)
- net at J1.11 (Pin_11), J2.11 (Pin_11), J3.11 (Pin_11)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: now also J9.6 (Pin_6), J12.6 (Pin_6), Q155.1 (G); no longer J9.3 (Pin_3)
- net at J1.12 (Pin_12), J2.12 (Pin_12), J3.12 (Pin_12)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: now also J9.7 (Pin_7), J12.7 (Pin_7), Q153.1 (G); no longer J9.2 (Pin_2)
- net at J1.13 (Pin_13), J2.13 (Pin_13), J3.13 (Pin_13)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: now also J9.8 (Pin_8), J12.8 (Pin_8), Q154.1 (G); no longer J9.1 (Pin_1)
- net RST: now reaches J4.3 (Pin_3)
- net RST: now also J1.3 (Pin_3), J2.3 (Pin_3), J3.3 (Pin_3)
- net at J1.6 (Pin_6), J2.6 (Pin_6), J3.6 (Pin_6)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: now also J9.1 (Pin_1), J12.1 (Pin_1), Q160.1 (G); no longer J9.8 (Pin_8)
- net at J1.7 (Pin_7), J2.7 (Pin_7), J3.7 (Pin_7)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: now also J9.2 (Pin_2), J12.2 (Pin_2), Q159.1 (G); no longer J9.7 (Pin_7)
- net at J1.8 (Pin_8), J2.8 (Pin_8), J3.8 (Pin_8)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: now also J9.3 (Pin_3), J12.3 (Pin_3), Q158.1 (G); no longer J9.6 (Pin_6)
- net at J1.9 (Pin_9), J2.9 (Pin_9), J3.9 (Pin_9)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: now also J9.4 (Pin_4), J12.4 (Pin_4), Q157.1 (G); no longer J9.5 (Pin_5)
- net at Q124.3 (D), Q44.3 (D), Q76.3 (D)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: now also Q141.1 (G), R21.2; no longer J11.4 (Pin_4)
- net at Q18.1 (G): now also J7.2 (Pin_2), Q17.1 (G), Q19.1 (G), Q20.1 (G), Q21.1 (G), Q22.1 (G), Q23.1 (G), Q24.1 (G), Q147.1 (G)
- net at Q112.3 (D), Q15.3 (D), Q32.3 (D)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: now also Q129.1 (G), R9.2; no longer J10.8 (Pin_8)
- net at Q72.1 (G): now also J8.1 (Pin_1), Q65.1 (G), Q66.1 (G), Q67.1 (G), Q68.1 (G), Q69.1 (G), Q70.1 (G), Q71.1 (G), Q146.1 (G)
- net at Q122.3 (D), Q42.3 (D), Q74.3 (D)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: now also Q143.1 (G), R23.2; no longer J11.2 (Pin_2)
- net at Q123.3 (D), Q43.3 (D), Q75.3 (D)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: now also Q142.1 (G), R22.2; no longer J11.3 (Pin_3)
- net at Q1.3 (D), Q105.3 (D), Q25.3 (D)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: now also Q136.1 (G), R16.2; no longer J10.1 (Pin_1)
- net at Q107.3 (D), Q27.3 (D), Q5.3 (D)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: now also Q134.1 (G), R14.2; no longer J10.3 (Pin_3)
- net at Q108.3 (D), Q28.3 (D), Q60.3 (D)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: now also Q133.1 (G), R13.2; no longer J10.4 (Pin_4)
- net at Q109.3 (D), Q29.3 (D), Q61.3 (D)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: now also Q132.1 (G), R12.2; no longer J10.5 (Pin_5)
- net at Q111.3 (D), Q13.3 (D), Q31.3 (D)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: now also Q130.1 (G), R10.2; no longer J10.7 (Pin_7)
- net at Q4.1 (G): now also J7.1 (Pin_1), Q10.1 (G), Q12.1 (G), Q14.1 (G), Q16.1 (G), Q2.1 (G), Q6.1 (G), Q8.1 (G), Q145.1 (G)
- net at Q128.3 (D), Q48.3 (D), Q80.3 (D)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: now also Q137.1 (G), R17.2; no longer J11.8 (Pin_8)
- net at Q98.1 (G): now also J7.4 (Pin_4), Q100.1 (G), Q101.1 (G), Q102.1 (G), Q103.1 (G), Q104.1 (G), Q97.1 (G), Q99.1 (G), Q151.1 (G)
- net at Q35.1 (G): now also J8.2 (Pin_2), Q33.1 (G), Q34.1 (G), Q36.1 (G), Q37.1 (G), Q38.1 (G), Q39.1 (G), Q40.1 (G), Q148.1 (G)
- net at Q86.1 (G): now also J8.3 (Pin_3), Q81.1 (G), Q82.1 (G), Q83.1 (G), Q84.1 (G), Q85.1 (G), Q87.1 (G), Q88.1 (G), Q150.1 (G)
- net at Q125.3 (D), Q45.3 (D), Q77.3 (D)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: now also Q140.1 (G), R20.2; no longer J11.5 (Pin_5)
- new net: D24.2, R156.2
- new net: J11.2 (Pin_2), Q138.3 (D), R26.2
- new net: D24.1, Q145.3 (D)
- new net: D7.1, Q152.3 (D)
- new net: D7.2, R39.2
- new net: D6.1, Q151.3 (D)
- new net: D6.2, R38.2
- new net: J10.7 (Pin_7), Q135.3 (D), R7.2
- new net: J10.4 (Pin_4), Q132.3 (D), R4.2
- new net: D14.1, Q158.3 (D)
- new net: D14.2, R46.2
- new net: D15.1, Q159.3 (D)
- new net: D15.2, R47.2
- new net: J11.3 (Pin_3), Q139.3 (D), R27.2
- new net: J11.6 (Pin_6), Q142.3 (D), R30.2
- new net: D5.1, Q150.3 (D)
- new net: D5.2, R37.2
- new net: J10.2 (Pin_2), Q130.3 (D), R2.2
- new net: J10.1 (Pin_1), Q129.3 (D), R1.2
- new net: J10.3 (Pin_3), Q131.3 (D), R3.2
- new net: J10.5 (Pin_5), Q133.3 (D), R5.2
- new net: J10.6 (Pin_6), Q134.3 (D), R6.2
- new net: J10.8 (Pin_8), Q136.3 (D), R8.2
- new net: J11.1 (Pin_1), Q137.3 (D), R25.2
- new net: D4.2, R36.2
- new net: D2.1, Q147.3 (D)
- new net: D2.2, R34.2
- new net: D8.2, R40.2
- new net: D16.2, R48.2
- new net: D10.1, Q154.3 (D)
- new net: D10.2, R42.2
- new net: D9.2, R41.2
- new net: D3.2, R35.2
- new net: J11.8 (Pin_8), Q144.3 (D), R32.2
- new net: D13.2, R45.2
- new net: J11.5 (Pin_5), Q141.3 (D), R29.2
- new net: J11.4 (Pin_4), Q140.3 (D), R28.2
- new net: D3.1, Q148.3 (D)
- new net: D13.1, Q157.3 (D)
- new net: D11.1, Q155.3 (D)
- new net: D9.1, Q153.3 (D)
- new net: D16.1, Q160.3 (D)
- new net: D1.1, Q146.3 (D)
- new net: D12.1, Q156.3 (D)
- new net: D12.2, R44.2
- new net: D1.2, R33.2
- new net: J11.7 (Pin_7), Q143.3 (D), R31.2
- new net: D4.1, Q149.3 (D)
- new net: D11.2, R43.2
Other:
- moved on the sheet: J1, J2, J3, J4, J5, J7, J8, J9

Commit message: ssss
Parts:
- added J6: Conn_01x02_Pin, Connector_PinHeader_2.54mm:PinHeader_1x02_P2.54mm_Vertical, symbol Connector:Conn_01x02_Pin
Connections:
- net RST: now also J6.2 (Pin_2)
- net Rising_Edge: now also J6.1 (Pin_1)
Changed lines of the file:
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@@
 	)
 	(junction
+		(at 172.72 110.49)
+		(diameter 0)
+		(color 0 0 0 0)
+	)
+	(junction
 		(at 483.87 302.26)
 		(diameter 0)
@@
 	)
 	(junction
+		(at 168.91 118.11)
+		(diameter 0)
+		(color 0 0 0 0)
+	)
+	(junction
 		(at 339.09 382.27)
 		(diameter 0)
@@
 	(wire
 		(pts
-			(xy 172.72 93.98) (xy 172.72 123.19)
+			(xy 172.72 93.98) (xy 172.72 110.49)
 		)
 		(stroke
@@
 	(wire
 		(pts
+			(xy 165.1 110.49) (xy 172.72 110.49)
+		)
+		(stroke
+			(width 0)
+			(type default)
+		)
+	)
+	(wire
+		(pts
 			(xy 87.63 140.97) (xy 144.78 140.97)
 		)
@@
 	(wire
 		(pts
+			(xy 168.91 118.11) (xy 259.08 118.11)
+		)
+		(stroke
+			(width 0)
+			(type default)
+		)
+	)
+	(wire
+		(pts
 			(xy 506.73 353.06) (xy 478.79 353.06)
 		)
@@
 	(wire
 		(pts
-			(xy 137.16 118.11) (xy 259.08 118.11)
+			(xy 137.16 118.11) (xy 168.91 118.11)
 		)
 		(stroke
@@
 	(wire
 		(pts
+			(xy 172.72 110.49) (xy 172.72 123.19)
+		)
+		(stroke
+			(width 0)
+			(type default)
+		)
+	)
+	(wire
+		(pts
 			(xy 172.72 374.65) (xy 185.42 374.65)
 		)
@@
 	(wire
 		(pts
+			(xy 168.91 113.03) (xy 165.1 113.03)
+		)
+		(stroke
+			(width 0)
+			(type default)
+		)
+	)
+	(wire
+		(pts
 			(xy 250.19 353.06) (xy 250.19 146.05)
 		)
@@
 	(wire
 		(pts
+			(xy 168.91 118.11) (xy 168.91 113.03)
+		)
+		(stroke
+			(width 0)
+			(type default)
+		)
+	)
+	(wire
+		(pts
 			(xy 232.41 264.16) (xy 259.08 264.16)
 		)
@@
 					(unit 1)
 				)
+			)
+		)
+	)
+	(symbol
+		(lib_id "Connector:Conn_01x02_Pin")
+		(at 160.02 110.49 0)
+		(unit 1)
+		(exclude_from_sim no)
+		(in_bom yes)
+		(on_board yes)
+		(dnp no)
+		(property "Reference" "J6"
+			(at 161.544 107.696 0)
+			(effects
+				(font
+					(size 1.27 1.27)
+				)
+			)
+		)
+		(property "Value" "Conn_01x02_Pin"
+			(at 160.655 107.95 0)
+			(effects
+				(font
+					(size 1.27 1.27)
+				)
+				(hide yes)
+			)
+		)
+		(property "Footprint" "Connector_PinHeader_2.54mm:PinHeader_1x02_P2.54mm_Vertical"
+			(at 160.02 110.49 0)
+			(effects
+				(font
+					(size 1.27 1.27)
+				)
+				(hide yes)
+			)
+		)
+		(property "Datasheet" "~"
+			(at 160.02 110.49 0)
+			(effects
+				(font
+					(size 1.27 1.27)
+				)
+				(hide yes)
+			)
+		)
+		(property "Description" "Generic connector, single row, 01x02, script generated"
+			(at 160.02 110.49 0)
+			(effects
+				(font
+					(size 1.27 1.27)
+				)
+				(hide yes)
+			)
+		)
+		(pin "1"
+		)
+		(pin "2"
+		)
+		(instances
+			(project "Register_Holder_V1.0"
+				(path "/2b76aa95-bd88-401b-8670-df1c96d69959"
+					(reference "J6")
+					(unit 1)
+				)
