File: PCB_S/Register_Holder_V1.0/Register_Holder_V1.0/Register_Holder_V1.0.kicad_pcb (KiCad board)
At the start: 6 copper layers, 160.1 x 100 mm, 277 parts, among them J1 Conn_01x21_Socket, J10 Conn_01x08, J11 Conn_01x08, J12 Conn_01x08, J13 Conn_01x02_Pin, J14 Conn_01x02_Pin, J15 Conn_01x02_Pin, J2 Conn_01x21_Socket, J3 Conn_01x21_Socket, J4 Conn_01x21_Socket, J5 Conn_01x04_Pin, J7 Conn_01x04_Pin, J8 Conn_01x04_Pin, J9 Conn_01x08, Q1 2N7002, Q10 2N7002, Q100 2N7002, Q101 2N7002, Q102 2N7002, Q103 2N7002, Q104 2N7002, Q105 2N7002, Q106 2N7002, Q107 2N7002, Q108 2N7002, Q109 2N7002, Q11 2N7002, Q110 2N7002, Q111 2N7002, Q112 2N7002, Q113 2N7002, Q114 2N7002, Q115 2N7002, Q116 2N7002, Q117 2N7002, Q118 2N7002, Q119 2N7002, Q12 2N7002, Q120 2N7002, Q121 2N7002, Q122 2N7002, Q123 2N7002, Q124 2N7002, Q125 2N7002, Q126 2N7002, Q127 2N7002, Q128 2N7002, Q129 2N7002, Q13 2N7002, Q130 2N7002, Q131 2N7002, Q132 2N7002, Q133 2N7002, Q134 2N7002, Q135 2N7002, Q136 2N7002, Q137 2N7002, Q138 2N7002, Q139 2N7002, Q14 2N7002, Q140 2N7002, Q141 2N7002, Q142 2N7002, Q143 2N7002, Q144 2N7002, Q145 2N7002, Q146 2N7002, Q147 2N7002, Q148 2N7002, Q149 2N7002, Q15 2N7002, Q150 2N7002, Q151 2N7002, Q152 2N7002, Q153 2N7002, Q154 2N7002, Q155 2N7002, Q156 2N7002, Q157 2N7002, Q158 2N7002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

Commit message: ssss
Parts:
- added J6: Conn_01x02_Pin, Connector_PinHeader_2.54mm:PinHeader_1x02_P2.54mm_Vertical, F.Cu at (63.5, 23.7)
Routing:
- net Rising_Edge: track 96.0 -> 122.7 mm
- net RST: track 96.0 -> 116.6 mm
Changed lines of the file:
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@@
 		)
 	)
+	(footprint "Connector_PinHeader_2.54mm:PinHeader_1x02_P2.54mm_Vertical"
+		(layer "F.Cu")
+		(at 63.46 23.7 90)
+		(descr "Through hole straight pin header, 1x02, 2.54mm pitch, single row")
+		(tags "Through hole pin header THT 1x02 2.54mm single row")
+		(property "Reference" "J6"
+			(at 0 -2.38 90)
+			(layer "F.SilkS")
+			(effects
+				(font
+					(size 1 1)
+					(thickness 0.15)
+				)
+			)
+		)
+		(property "Value" "Conn_01x02_Pin"
+			(at 0 4.92 90)
+			(layer "F.Fab")
+			(effects
+				(font
+					(size 1 1)
+					(thickness 0.15)
+				)
+			)
+		)
+		(property "Datasheet" "~"
+			(at 0 0 90)
+			(layer "F.Fab")
+			(hide yes)
+			(effects
+				(font
+					(size 1.27 1.27)
+					(thickness 0.15)
+				)
+			)
+		)
+		(property "Description" "Generic connector, single row, 01x02, script generated"
+			(at 0 0 90)
+			(layer "F.Fab")
+			(hide yes)
+			(effects
+				(font
+					(size 1.27 1.27)
+					(thickness 0.15)
+				)
+			)
+		)
+		(property ki_fp_filters "Connector*:*_1x??_*")
+		(sheetname "/")
+		(sheetfile "Register_Holder_V1.0.kicad_sch")
+		(attr through_hole)
+		(fp_line
+			(start -1.38 -1.38)
+			(end 0 -1.38)
+			(stroke
+				(width 0.12)
+				(type solid)
+			)
+			(layer "F.SilkS")
+		)
+		(fp_line
+			(start -1.38 0)
+			(end -1.38 -1.38)
+			(stroke
+				(width 0.12)
+				(type solid)
+			)
+			(layer "F.SilkS")
+		)
+		(fp_line
+			(start 1.38 1.27)
+			(end 1.38 3.92)
+			(stroke
+				(width 0.12)
+				(type solid)
+			)
+			(layer "F.SilkS")
+		)
+		(fp_line
+			(start -1.38 1.27)
+			(end 1.38 1.27)
+			(stroke
+				(width 0.12)
+				(type solid)
+			)
+			(layer "F.SilkS")
+		)
+		(fp_line
+			(start -1.38 1.27)
+			(end -1.38 3.92)
+			(stroke
+				(width 0.12)
+				(type solid)
+			)
+			(layer "F.SilkS")
+		)
+		(fp_line
+			(start -1.38 3.92)
+			(end 1.38 3.92)
+			(stroke
+				(width 0.12)
+				(type solid)
+			)
+			(layer "F.SilkS")
+		)
+		(fp_rect
+			(start -1.77 -1.77)
+			(end 1.77 4.32)
+			(stroke
+				(width 0.05)
+				(type solid)
+			)
+			(fill no)
+			(layer "F.CrtYd")
+		)
+		(fp_line
+			(start 1.27 -1.27)
+			(end 1.27 3.81)
+			(stroke
+				(width 0.1)
+				(type solid)
+			)
+			(layer "F.Fab")
+		)
+		(fp_line
+			(start -0.635 -1.27)
+			(end 1.27 -1.27)
+			(stroke
+				(width 0.1)
+				(type solid)
+			)
+			(layer "F.Fab")
+		)
+		(fp_line
+			(start -1.27 -0.635)
+			(end -0.635 -1.27)
+			(stroke
+				(width 0.1)
+				(type solid)
+			)
+			(layer "F.Fab")
+		)
+		(fp_line
+			(start 1.27 3.81)
+			(end -1.27 3.81)
+			(stroke
+				(width 0.1)
+				(type solid)
+			)
+			(layer "F.Fab")
+		)
+		(fp_line
+			(start -1.27 3.81)
+			(end -1.27 -0.635)
+			(stroke
+				(width 0.1)
+				(type solid)
+			)
+			(layer "F.Fab")
+		)
+		(fp_text user "${REFERENCE}"
+			(at 0 1.27 0)
+			(layer "F.Fab")
+			(effects
+				(font
+					(size 1 1)
+					(thickness 0.15)
+				)
+			)
+		)
+		(pad "1" thru_hole rect
+			(at 0 0 90)
+			(size 1.7 1.7)
+			(drill 1)
+			(layers "*.Cu" "*.Mask")
+			(remove_unused_layers no)
+			(net 11 "Rising_Edge")
+			(pinfunction "Pin_1")
+			(pintype "passive")
+		)
+		(pad "2" thru_hole circle
+			(at 0 2.54 90)
+			(size 1.7 1.7)
+			(drill 1)
+			(layers "*.Cu" "*.Mask")
+			(remove_unused_layers no)
+			(net 169 "RST")
+			(pinfunction "Pin_2")
+			(pintype "passive")
+		)
+		(embedded_fonts no)
+		(model "${KICAD9_3DMODEL_DIR}/Connector_PinHeader_2.54mm.3dshapes/PinHeader_1x02_P2.54mm_Vertical.step"
+			(offset
+				(xyz 0 0 0)
+			)
+			(scale
+				(xyz 1 1 1)
+			)
+			(rotate
+				(xyz 0 0 0)
+			)
+		)
+	)
 	(footprint "Package_TO_SOT_SMD:SOT-23"
 		(layer "F.Cu")
@@
 	)
 	(segment
+		(start 63.46 23.7)
+		(end 63.46 26.13)
+		(width 0.6)
+		(layer "B.Cu")
+		(net 11)
+	)
+	(segment
+		(start 63.46 26.13)
+		(end 80.59 43.26)
+		(width 0.6)
+		(layer "B.Cu")
+		(net 11)
+	)
+	(segment
 		(start 80.59 43.26)
 		(end 176.59 43.26)
@@
 	)
 	(segment
+		(start 66 23.7)
+		(end 80.48 38.18)
+		(width 0.4)
+		(layer "B.Cu")
+		(net 169)
+	)
+	(segment
+		(start 80.48 38.18)
+		(end 80.59 38.18)
+		(width 0.2)
+		(layer "B.Cu")
+		(net 169)
+	)
+	(segment

Commit message: REG_HOLDER_V1.0 done
Parts:
- moved J6 36.1 mm to (57.2, 59.2), turned to 180 degrees
- moved J5 3.20 mm to (57.2, 66.2)
- moved J7 3.20 mm to (57.2, 79.4)
- moved J8 3.20 mm to (57.2, 92.6)
- moved J15 2.80 mm to (57.2, 105.7)
Routing:
- net RST: track 116.6 -> 127.2 mm
- net Net-(J4-Pin_4): track 141.2 -> 144.6 mm
- net Rising_Edge: track 122.7 -> 126.0 mm
- net Net-(J3-Pin_4): track 107.1 -> 110.4 mm
- net Net-(J2-Pin_4): track 72.9 -> 76.1 mm
- net Net-(J1-Pin_4): track 38.7 -> 41.8 mm
- net Net-(J7-Pin_1): track 95.8 -> 97.2 mm
- net Net-(J7-Pin_3): track 155.1 -> 156.5 mm
- net Net-(J7-Pin_2): track 117.4 -> 118.8 mm
- net Net-(J7-Pin_4): track 185.5 -> 186.9 mm
- net Net-(J8-Pin_2): track 126.4 -> 127.8 mm
- net Net-(J8-Pin_1): track 92.1 -> 93.4 mm
- net Net-(J8-Pin_3): track 159.1 -> 160.4 mm
- net Net-(J8-Pin_4): track 195.8 -> 197.1 mm
Other:
- board text added: "RE"
- board text added: "rst"
