File: PCB_S/Controller_Unit_V1.0/Controller_Unit_V1.0.kicad_sch (KiCad schematic)
At the start: 179 parts, among them J1 Conn_01x21_Socket, Q1 2N7002, Q10 2N7002, Q100 2N7002, Q101 2N7002, Q102 2N7002, Q103 2N7002, Q104 2N7002, Q105 2N7002, Q106 2N7002, Q107 2N7002, Q108 2N7002, Q109 2N7002, Q11 2N7002, Q110 2N7002, Q111 2N7002, Q112 2N7002, Q113 2N7002, Q114 2N7002, Q115 2N7002, Q116 2N7002, Q117 2N7002, Q118 2N7002, Q119 2N7002, Q12 2N7002, Q120 2N7002, Q121 2N7002, Q122 2N7002, Q123 2N7002, Q124 2N7002, Q125 2N7002, Q126 2N7002, Q127 2N7002, Q13 2N7002, Q14 2N7002, Q15 2N7002, Q16 2N7002, Q17 2N7002, Q18 2N7002, Q19 2N7002, Q2 2N7002, Q20 2N7002, Q21 2N7002, Q22 2N7002, Q23 2N7002, Q24 2N7002, Q25 2N7002, Q26 2N7002, Q27 2N7002, Q28 2N7002, Q29 2N7002, Q3 2N7002, Q30 2N7002, Q31 2N7002, Q32 2N7002, Q33 2N7002, Q34 2N7002, Q35 2N7002, Q36 2N7002, Q37 2N7002, Q38 2N7002, Q39 2N7002, Q4 2N7002, Q40 2N7002, Q41 2N7002, Q42 2N7002, Q43 2N7002, Q44 2N7002, Q45 2N7002, Q46 2N7002, Q47 2N7002, Q48 2N7002, Q49 2N7002, Q5 2N7002, Q50 2N7002, Q51 2N7002, Q52 2N7002, Q53 2N7002, Q54 2N7002, Q55 2N7002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

Commit message: Controller V1.0 work
Parts:
- removed Q117, Q118, Q119, Q120, Q121, Q122, Q123, Q124, Q125, Q126, Q127: 2N7002, Package_TO_SOT_SMD:SOT-23, symbol Transistor_FET:2N7002
- removed R51: 10kΩ, PCM_JLCPCB:R_0402, symbol PCM_JLCPCB-Resistors:0402,20kΩ
- added Q128, Q129, Q130, Q131, Q132, Q133, Q134, Q135: 2N7002, Package_TO_SOT_SMD:SOT-23, symbol Transistor_FET:2N7002
- added R52: 10kΩ, PCM_JLCPCB:R_0402, symbol PCM_JLCPCB-Resistors:0402,20kΩ
Connections:
- net ADC is gone; now on net !ADC: Q61.3 (D), R34.2
- net ADD is gone; now on net !ADD: Q60.3 (D), R33.2
- net AND is gone; now on net !AND: Q54.3 (D), R30.2
- net Clear is gone; now on net !Clear: Q43.3 (D), R23.2
- net DEC is gone; now on net !DEC: Q50.3 (D), R27.2
- net INC is gone; now on net !INC: Q46.3 (D), R26.2
- net Load is gone; now on net !Load: Q44.3 (D), R24.2
- net MOV is gone; now on net !MOV: Q65.3 (D), R35.2
- net NOT is gone; now on net !NOT: Q52.3 (D), R29.2
- net OR is gone; now on net !OR: Q55.3 (D), R31.2
- net RS is gone; now on net !RS: Q51.3 (D), R28.2
- net Store is gone; now on net !Store: Q45.3 (D), R25.2
- net XOR is gone; now on net !XOR: Q58.3 (D), R32.2
- net GND: now also Q99.2 (S)
- net READ FALG: now also Q135.3 (D), R52.2
- net REG -> ALU A: now also Q109.3 (D), Q80.1 (G); no longer Q110.3 (D)
- net REG -> ALU B: now also Q79.1 (G)
- net REG Read: now also Q78.1 (G), Q98.3 (D); no longer Q99.3 (D)
- net VCC: now also R52.1
- net !MOV: now reaches Q116.1 (G)
- net !MOV: now also Q98.1 (G)
- net !OR: now reaches Q112.1 (G)
- net !OR: now also Q106.1 (G), Q94.1 (G), Q131.1 (G)
- net !Load: now reaches Q88.1 (G)
- net !INC: now reaches Q101.1 (G)
- net !INC: now also Q89.1 (G), Q99.1 (G)
- net !XOR: now reaches Q95.1 (G)
- net !XOR: now also Q107.1 (G), Q113.1 (G), Q132.1 (G)
- net !Store: now reaches Q100.1 (G)
- net !Clear: now reaches Q87.1 (G)
- net !ADC: now reaches Q97.1 (G)
- net !ADC: now also Q109.1 (G), Q115.1 (G), Q134.1 (G)
- net !RS: now reaches Q91.1 (G)
- net !RS: now also Q103.1 (G), Q128.1 (G)
- net !ADD: now reaches Q96.1 (G)
- net !ADD: now also Q108.1 (G), Q114.1 (G), Q133.1 (G)
- net !DEC: now reaches Q110.1 (G)
- net !DEC: now also Q102.1 (G), Q90.1 (G)
- net at Q110.2 (S): now also Q99.3 (D); no longer Q109.3 (D)
- net !AND: now reaches Q111.1 (G)
- net !AND: now also Q105.1 (G), Q93.1 (G), Q130.1 (G)
- net !NOT: now reaches Q92.1 (G)
- net !NOT: now also Q104.1 (G), Q129.1 (G)
- net AA renamed A ->ALU A
- net AB renamed B ->ALU A
- net AC renamed C ->ALU A
- net AD renamed D ->ALU A
- net BA renamed A ->ALU B
- net BB renamed B ->ALU B
- net BC renamed C ->ALU B
- net BD renamed D ->ALU B
- net BNC renamed !BNC
- net BNO renamed !BNO
- net BNU renamed !BNU
- net BNZ renamed !BNZ
- net BOC renamed !BOC
- net BON renamed !BON
- net BOO renamed !BOO
- net BOP renamed !BOP
- net BOU renamed !BOU
- net BOZ renamed !BOZ
- net CLF renamed !CLF
- net !CLF: now also Q135.1 (G)
- net CLR renamed !CLR
- net JMP renamed !JMP
- net RA renamed READ A
- net RB renamed READ B
- net RC renamed READ C
- net RD renamed READ D
- net RST renamed !RST
- new net: Q128.3 (D), Q129.2 (S)
- new net: Q129.3 (D), Q130.2 (S)
- new net: Q131.3 (D), Q132.2 (S)
- new net: Q132.3 (D), Q133.2 (S)
- new net: Q134.3 (D), Q135.2 (S)
- new net: Q133.3 (D), Q134.2 (S)
- new net: Q130.3 (D), Q131.2 (S)
- new net: Q110.3 (D), Q128.2 (S)

Commit message: small
Parts:
- added D1, D10, D11, D12, D13, D14, D15, D16, D17, D18, D19, D2, D20, D21, D22, D23, D24, D25, D26, D27, D3, D4, D5, D6, D7, D8, D9: Red, PCM_JLCPCB:D_0603, symbol PCM_JLCPCB-Diodes:LED,0603,Red
- added R100, R101, R102, R103, R104, R105, R51, R53, R54, R55, R56, R57, R58, R59, R60, R61, R62, R63, R64, R65, R66, R67, R68, R69, R70, R71, R72, R73, R74, R75, R76, R77, R78, R79, R80, R81, R82, R83, R84, R85, R86, R87, R88, R89, R90, R91, R92, R93, R94, R95, R96, R97, R98, R99: 10kΩ, PCM_JLCPCB:R_0402, symbol PCM_JLCPCB-Resistors:0402,20kΩ
Connections:
- net !ADC: now also D26.1
- net !ADD: now also D25.1
- net !AND: now also D22.1
- net !BNC: now also D11.1
- net !BNO: now also D7.1
- net !BNU: now also D9.1
- net !BNZ: now also D5.1
- net !BOC: now also D10.1
- net !BON: now also D3.1
- net !BOO: now also D6.1
- net !BOP: now also D2.1
- net !BOU: now also D8.1
- net !BOZ: now also D4.1
- net !CLF: now also D13.1
- net !CLR: now also D14.1
- net !Clear: now also D15.1
- net !DEC: now also D19.1
- net !INC: now also D18.1
- net !JMP: now also D1.1
- net !Load: now also D16.1
- net !MOV: now also D27.1
- net !NOT: now also D21.1
- net !OR: now also D23.1
- net !RS: now also D20.1
- net !RST: now also D12.1
- net !Store: now also D17.1
- net !XOR: now also D24.1
- net VCC: now also R100.1, R101.1, R102.1, R103.1, R104.1, R105.1, R51.1, R53.1, R54.1, R55.1, R56.1, R57.1, R58.1, R59.1, R60.1, R61.1, R62.1, R63.1, R64.1, R65.1, R66.1, R67.1, R68.1, R69.1, R70.1, R71.1, R72.1, R73.1, R74.1, R75.1, R76.1, R77.1, R78.1, R79.1, R80.1, R81.1, R82.1, R83.1, R84.1, R85.1, R86.1, R87.1, R88.1, R89.1, R90.1, R91.1, R92.1, R93.1, R94.1, R95.1, R96.1, R97.1, R98.1, R99.1
- new net: D15.2, R80.2, R81.2
- new net: D2.2, R54.2, R55.2
- new net: D8.2, R66.2, R67.2
- new net: D3.2, R56.2, R57.2
- new net: D18.2, R86.2, R87.2
- new net: D22.2, R94.2, R95.2
- new net: D19.2, R88.2, R89.2
- new net: D20.2, R90.2, R91.2
- new net: D11.2, R72.2, R73.2
- new net: D7.2, R64.2, R65.2
- new net: D24.2, R98.2, R99.2
- new net: D5.2, R60.2, R61.2
- new net: D27.2, R104.2, R105.2
- new net: D14.2, R78.2, R79.2
- new net: D9.2, R68.2, R69.2
- new net: D23.2, R96.2, R97.2
- new net: D12.2, R74.2, R75.2
- new net: D13.2, R76.2, R77.2
- new net: D17.2, R84.2, R85.2
- new net: D1.2, R51.2, R53.2
- new net: D16.2, R82.2, R83.2
- new net: D21.2, R92.2, R93.2
- new net: D26.2, R102.2, R103.2
- new net: D25.2, R100.2, R101.2
- new net: D6.2, R62.2, R63.2
- new net: D10.2, R70.2, R71.2
- new net: D4.2, R58.2, R59.2

Commit message: controll uint work
Parts:
- added D28, D29, D30, D31, D32, D33, D34, D35, D36, D37, D38, D39: Red, PCM_JLCPCB:D_0603, symbol PCM_JLCPCB-Diodes:LED,0603,Red
- added J2, J3, J4, J5: Conn_01x21_Socket, symbol Connector:Conn_01x21_Socket
- added Q117, Q118, Q119, Q120, Q121, Q122, Q123, Q124, Q125, Q126, Q127, Q136, Q137, Q138, Q139, Q140, Q141, Q142, Q143, Q144, Q145, Q146, Q147, Q148, Q149, Q150, Q151, Q152, Q153, Q154, Q155, Q156, Q157, Q158, Q159, Q160, Q161, Q162, Q163, Q164, Q165, Q166, Q167, Q168, Q169, Q170, Q171, Q172, Q173, Q174, Q175, Q176, Q177, Q178, Q179, Q180, Q181, Q182, Q183, Q184, Q185, Q186, Q187, Q188, Q189, Q190, Q191, Q192, Q193, Q194, Q195, Q196, Q197, Q198, Q199, Q200, Q201, Q202, Q203, Q204, Q205, Q206, Q207, Q208, Q209, Q210, Q211, Q212, Q213, Q214, Q215, Q216, Q217, Q218, Q219, Q220, Q221, Q222, Q223, Q224, Q225, Q226, Q227, Q228, Q229, Q230, Q231, Q232, Q233, Q234, Q235, Q236, Q237, Q238, Q239, Q240, Q241, Q242, Q243, Q244, Q245, Q246, Q247, Q248, Q249, Q250, Q251, Q252, Q253, Q254, Q255, Q256, Q257, Q258, Q259, Q260, Q261, Q262, Q263, Q264, Q265, Q266, Q267, Q268, Q269, Q270, Q271, Q272, Q273, Q274, Q275, Q276, Q277, Q278, Q279, Q280, Q281, Q282, Q283, Q284, Q285, Q286, Q287, Q288, Q289, Q290, Q291, Q292, Q293, Q294, Q295, Q296, Q297, Q298, Q299, Q300, Q301, Q302, Q303, Q304, Q305, Q306, Q307, Q308, Q309, Q310, Q311, Q312, Q313, Q314, Q315, Q316, Q317, Q318, Q319, Q320, Q321, Q322, Q323, Q324, Q325, Q326, Q327, Q328: 2N7002, Package_TO_SOT_SMD:SOT-23, symbol Transistor_FET:2N7002
- added R106, R107, R108, R109, R110, R111, R112, R113, R114, R115, R116, R117, R118, R119, R120, R121, R122, R123, R124, R125, R126, R127, R128, R129, R130, R131, R132, R133, R134, R135, R136, R137, R138, R139, R140, R141, R142, R143, R144, R145, R146, R147, R148, R149, R150, R151, R152, R153, R154, R155, R156, R157, R158, R159, R160, R161, R162, R163, R164, R165, R166, R167, R168, R169, R170, R171, R172, R173, R174, R175, R176, R177, R178, R179, R180, R181, R182, R183, R184, R185, R186, R187, R188, R189, R190, R191, R192, R193, R194, R195, R196, R197, R198, R199, R200, R201, R202, R203, R204, R205, R206, R207, R208, R209, R210, R211, R212, R213, R214, R215, R216, R217, R218, R219, R220, R221, R222, R223, R224, R225, R226, R227, R228, R229, R230, R231, R232, R233, R234, R235, R236, R237: 10kΩ, PCM_JLCPCB:R_0402, symbol PCM_JLCPCB-Resistors:0402,20kΩ
Connections:
- net A ->ALU A: now also Q121.3 (D), R120.1; no longer Q83.3 (D), R44.2
- net A ->ALU B: now also Q125.3 (D), R132.1; no longer Q74.3 (D), R40.2
- net B ->ALU A: now also Q122.3 (D), R123.1; no longer Q84.3 (D), R45.2
- net B ->ALU B: now also Q126.3 (D), R135.1; no longer Q75.3 (D), R41.2
- net C ->ALU A: now also Q123.3 (D), R126.1; no longer Q85.3 (D), R46.2
- net C ->ALU B: now also Q127.3 (D), R138.1; no longer Q76.3 (D), R42.2
- net D ->ALU A: now also Q124.3 (D), R129.1; no longer Q86.3 (D), R47.2
- net D ->ALU B: now also Q136.3 (D), R141.1; no longer Q77.3 (D), R43.2
- net GND: now also J2.2 (Pin_2), J3.2 (Pin_2), J4.2 (Pin_2), J5.2 (Pin_2), Q117.2 (S), Q118.2 (S), Q119.2 (S), Q120.2 (S), Q121.2 (S), Q122.2 (S), Q123.2 (S), Q124.2 (S), Q125.2 (S), Q126.2 (S), Q127.2 (S), Q136.2 (S), Q137.2 (S), Q139.2 (S), Q142.2 (S), Q144.2 (S), Q146.2 (S), Q148.2 (S), Q150.2 (S), Q152.2 (S), Q154.2 (S), Q156.2 (S), Q158.2 (S), Q160.2 (S), Q162.2 (S), Q164.2 (S), Q166.2 (S), Q168.2 (S), Q170.2 (S), Q172.2 (S), Q173.2 (S), Q174.2 (S), Q175.2 (S), Q176.2 (S), Q177.2 (S), Q178.2 (S), Q179.2 (S), Q180.2 (S), Q181.2 (S), Q182.2 (S), Q183.2 (S), Q184.2 (S), Q185.2 (S), Q186.2 (S), Q187.2 (S), Q188.2 (S), Q189.2 (S), Q190.2 (S), Q191.2 (S), Q192.2 (S), Q193.2 (S), Q194.2 (S), Q195.2 (S), Q196.2 (S), Q197.2 (S), Q198.2 (S), Q199.2 (S), Q200.2 (S), Q201.2 (S), Q202.2 (S), Q203.2 (S), Q220.2 (S), Q221.2 (S), Q222.2 (S), Q223.2 (S), Q224.2 (S), Q225.2 (S), Q226.2 (S), Q227.2 (S), Q228.2 (S), Q229.2 (S), Q230.2 (S), Q231.2 (S), Q232.2 (S), Q233.2 (S), Q234.2 (S), Q235.2 (S), Q236.2 (S), Q237.2 (S), Q238.2 (S), Q239.2 (S), Q240.2 (S), Q241.2 (S), Q242.2 (S), Q243.2 (S), Q244.2 (S), Q245.2 (S), Q246.2 (S), Q247.2 (S), Q248.2 (S), Q249.2 (S), Q250.2 (S), Q251.2 (S), Q252.2 (S), Q253.2 (S), Q254.2 (S), Q255.2 (S), Q256.2 (S), Q257.2 (S), Q258.2 (S), Q259.2 (S), Q260.2 (S), Q261.2 (S), Q262.2 (S), Q263.2 (S), Q264.2 (S), Q265.2 (S), Q266.2 (S), Q267.2 (S), Q268.2 (S), Q269.2 (S), Q270.2 (S), Q271.2 (S), Q272.2 (S), Q273.2 (S), Q274.2 (S), Q275.2 (S), Q276.2 (S), Q277.2 (S), Q278.2 (S), Q279.2 (S), Q280.2 (S), Q281.2 (S), Q282.2 (S), Q283.2 (S), Q284.2 (S), Q286.2 (S), Q288.2 (S), Q290.2 (S), Q292.2 (S), Q294.2 (S), Q296.2 (S), Q298.2 (S), Q300.2 (S), Q302.2 (S), Q304.2 (S), Q306.2 (S), Q308.2 (S), Q310.2 (S), Q312.2 (S), Q313.2 (S), Q314.2 (S), Q315.2 (S), Q316.2 (S), Q317.2 (S), Q318.2 (S), Q319.2 (S), Q320.2 (S), Q321.2 (S), Q322.2 (S), Q323.2 (S), Q324.2 (S), Q325.2 (S), Q326.2 (S), Q327.2 (S), Q328.2 (S)
- net READ A: now also Q117.3 (D), R108.1; no longer Q68.3 (D), R36.2
- net READ B: now also Q118.3 (D), R111.1; no longer Q69.3 (D), R37.2
- net READ C: now also Q119.3 (D), R114.1; no longer Q70.3 (D), R38.2
- net READ D: now also Q120.3 (D), R117.1; no longer Q71.3 (D), R39.2
- net VCC: now also J2.1 (Pin_1), J3.1 (Pin_1), J4.1 (Pin_1), J5.1 (Pin_1), R106.1, R107.1, R108.2, R109.1, R110.1, R111.2, R112.1, R113.1, R114.2, R115.1, R116.1, R117.2, R118.1, R119.1, R120.2, R121.1, R122.1, R123.2, R124.1, R125.1, R126.2, R127.1, R128.1, R129.2, R130.1, R131.1, R132.2, R133.1, R134.1, R135.2, R136.1, R137.1, R138.2, R139.1, R140.1, R141.2, R142.1, R143.1, R144.1, R145.1, R146.1, R147.1, R148.1, R149.1, R150.1, R151.1, R152.1, R153.1, R154.1, R155.1, R156.1, R157.1, R158.1, R159.1, R160.1, R161.1, R162.1, R163.1, R164.1, R165.1, R166.1, R167.1, R168.1, R169.1, R170.1, R171.1, R172.1, R173.1, R174.1, R175.1, R176.1, R177.1, R178.1, R179.1, R180.1, R181.1, R182.1, R183.1, R184.1, R185.1, R186.1, R187.1, R188.1, R189.1, R190.1, R191.1, R192.1, R193.1, R194.1, R195.1, R196.1, R197.1, R198.1, R199.1, R200.1, R201.1, R202.1, R203.1, R204.1, R205.1, R206.1, R207.1, R208.1, R209.1, R210.1, R211.1, R212.1, R213.1, R214.1, R215.1, R216.1, R217.1, R218.1, R219.1, R220.1, R221.1, R222.1, R223.1, R224.1, R225.1, R226.1, R227.1, R228.1, R229.1, R230.1, R231.1, R232.1, R233.1, R234.1, R235.1, R236.1, R237.1
- net rst: now also J2.3 (Pin_3), J3.3 (Pin_3), J4.3 (Pin_3), J5.3 (Pin_3)
- net Buss4: now reaches J1.10 (Pin_10)
- net Buss4: now also J4.10 (Pin_10), J5.10 (Pin_10)
- net Buss5: now reaches J1.11 (Pin_11)
- net Buss5: now also J4.11 (Pin_11), J5.11 (Pin_11)
- net Buss6: now reaches J1.12 (Pin_12)
- net Buss6: now also J4.12 (Pin_12), J5.12 (Pin_12)
- net Buss7: now reaches J1.13 (Pin_13)
- net Buss7: now also J4.13 (Pin_13), J5.13 (Pin_13)
- net Buss0: now reaches J1.6 (Pin_6)
- net Buss0: now also J4.6 (Pin_6), J5.6 (Pin_6)
- net Buss1: now reaches J1.7 (Pin_7)
- net Buss1: now also J4.7 (Pin_7), J5.7 (Pin_7)
- net Buss2: now reaches J1.8 (Pin_8)
- net Buss2: now also J4.8 (Pin_8), J5.8 (Pin_8)
- net Buss3: now reaches J1.9 (Pin_9)
- net Buss3: now also J4.9 (Pin_9), J5.9 (Pin_9)
- net RNI renamed Read New Instruction
- new net: Q203.3 (D), Q235.3 (D), Q267.1 (G), R209.2
- new net: Q137.3 (D), Q138.2 (S)
- new net: Q138.3 (D), Q169.3 (D), Q313.1 (G), R143.2
- new net: Q299.2 (S), Q300.3 (D)
- new net: Q218.1 (G), Q234.1 (G), Q251.3 (D), Q283.1 (G), R193.2
- new net: Q202.3 (D), Q234.3 (D), Q266.1 (G), R208.2
- new net: D36.1, Q125.1 (G), Q74.3 (D), R40.2
- new net: Q167.3 (D), Q311.3 (D), Q328.1 (G), R236.2
- new net: Q197.3 (D), Q229.3 (D), Q261.1 (G), R203.2
- new net: Q172.3 (D), Q204.2 (S)
- new net: Q305.2 (S), Q306.3 (D)
- new net: D34.1, Q123.1 (G), Q85.3 (D), R46.2
- new net: D34.2, R124.2, R125.2
- new net: Q194.3 (D), Q226.3 (D), Q258.1 (G), R200.2
- new net: Q149.2 (S), Q150.3 (D)
- new net: Q143.2 (S), Q144.3 (D)
- new net: Q143.3 (D), Q287.3 (D), Q316.1 (G), R148.2
- new net: Q211.1 (G), Q227.1 (G), Q244.3 (D), Q276.1 (G), R186.2
- new net: Q209.1 (G), Q225.1 (G), Q242.3 (D), Q274.1 (G), R184.2
- new net: Q217.3 (D), Q249.1 (G), R175.2
- new net: D38.2, R136.2, R137.2
- new net: Q291.2 (S), Q292.3 (D)
- new net: Q147.3 (D), Q291.3 (D), Q318.1 (G), R152.2
- new net: Q211.3 (D), Q243.1 (G), R169.2
- new net: Q210.1 (G), Q226.1 (G), Q243.3 (D), Q275.1 (G), R185.2
- new net: Q212.1 (G), Q228.1 (G), Q245.3 (D), Q277.1 (G), R187.2
- new net: Q141.2 (S), Q142.3 (D)
- new net: Q212.3 (D), Q244.1 (G), R170.2
- new net: Q204.3 (D), Q236.1 (G), R162.2
- new net: Q236.3 (D), Q268.1 (G), R178.2
- new net: Q206.3 (D), Q238.1 (G), R164.2
- new net: Q215.1 (G), Q231.1 (G), Q248.3 (D), Q280.1 (G), R190.2
- new net: Q167.2 (S), Q168.3 (D)
- new net: Q184.3 (D), Q216.2 (S)
- new net: Q157.3 (D), Q301.3 (D), Q323.1 (G), R226.2
- new net: Q217.1 (G), Q233.1 (G), Q250.3 (D), Q282.1 (G), R192.2
- new net: Q201.3 (D), Q233.3 (D), Q265.1 (G), R207.2
- new net: Q209.3 (D), Q241.1 (G), R167.2
- new net: Q208.1 (G), Q224.1 (G), Q241.3 (D), Q273.1 (G), R183.2
- new net: Q159.2 (S), Q160.3 (D)
- new net: Q192.3 (D), Q224.3 (D), Q256.1 (G), R198.2
- new net: Q293.2 (S), Q294.3 (D)
- new net: Q149.3 (D), Q293.3 (D), Q319.1 (G), R154.2
- new net: Q151.2 (S), Q152.3 (D)
- new net: Q151.3 (D), Q295.3 (D), Q320.1 (G), R156.2
- new net: D30.1, Q119.1 (G), Q70.3 (D), R38.2
- new net: D30.2, R112.2, R113.2
- new net: D31.2, R115.2, R116.2
- new net: D28.1, Q117.1 (G), Q68.3 (D), R36.2
- new net: Q155.3 (D), Q299.3 (D), Q322.1 (G), R160.2
- new net: Q163.2 (S), Q164.3 (D)
- new net: Q163.3 (D), Q307.3 (D), Q326.1 (G), R232.2
- new net: Q200.3 (D), Q232.3 (D), Q264.1 (G), R206.2
- new net: D36.2, R130.2, R131.2
- new net: Q193.3 (D), Q225.3 (D), Q257.1 (G), R199.2
- new net: Q147.2 (S), Q148.3 (D)
- new net: Q198.3 (D), Q230.3 (D), Q262.1 (G), R204.2
- new net: D29.1, Q118.1 (G), Q69.3 (D), R37.2
- new net: Q171.2 (S), Q284.3 (D)
- new net: Q140.3 (D), Q171.3 (D), Q314.1 (G), R144.2
- new net: Q181.3 (D), Q213.2 (S)
- new net: Q175.3 (D), Q207.2 (S)
- new net: Q165.2 (S), Q166.3 (D)
- new net: Q165.3 (D), Q309.3 (D), Q327.1 (G), R234.2
- new net: Q178.3 (D), Q210.2 (S)
- new net: Q210.3 (D), Q242.1 (G), R168.2
- new net: Q195.3 (D), Q227.3 (D), Q259.1 (G), R201.2
- new net: Q309.2 (S), Q310.3 (D)
- new net: D33.1, Q122.1 (G), Q84.3 (D), R45.2
- new net: D33.2, R121.2, R122.2
- new net: Q205.1 (G), Q221.1 (G), Q238.3 (D), Q270.1 (G), R180.2
- new net: Q173.3 (D), Q205.2 (S)
- new net: Q205.3 (D), Q237.1 (G), R163.2
- new net: Q207.1 (G), Q223.1 (G), Q240.3 (D), Q272.1 (G), R182.2
- new net: Q216.1 (G), Q232.1 (G), Q249.3 (D), Q281.1 (G), R191.2
- new net: Q301.2 (S), Q302.3 (D)
- new net: D35.2, R127.2, R128.2
- new net: Q139.3 (D), Q140.2 (S)
- new net: Q206.1 (G), Q222.1 (G), Q239.3 (D), Q271.1 (G), R181.2
- new net: Q190.3 (D), Q222.3 (D), Q254.1 (G), R196.2
- new net: Q186.3 (D), Q218.2 (S)
- new net: D38.1, Q127.1 (G), Q76.3 (D), R42.2
- new net: D37.1, Q126.1 (G), Q75.3 (D), R41.2
- new net: Q204.1 (G), Q220.1 (G), Q237.3 (D), Q269.1 (G), R179.2
- new net: Q215.3 (D), Q247.1 (G), R173.2
- new net: Q214.1 (G), Q230.1 (G), Q247.3 (D), Q279.1 (G), R189.2
- new net: Q153.3 (D), Q297.3 (D), Q321.1 (G), R158.2
- new net: Q188.3 (D), Q220.3 (D), Q252.1 (G), R194.2
- new net: Q157.2 (S), Q158.3 (D)
- new net: Q219.3 (D), Q251.1 (G), R177.2
- new net: D35.1, Q124.1 (G), Q86.3 (D), R47.2
- new net: D32.1, Q121.1 (G), Q83.3 (D), R44.2
- new net: D32.2, R118.2, R119.2
- new net: Q218.3 (D), Q250.1 (G), R176.2
- new net: Q191.3 (D), Q223.3 (D), Q255.1 (G), R197.2
- new net: Q287.2 (S), Q288.3 (D)
- new net: Q189.3 (D), Q221.3 (D), Q253.1 (G), R195.2
- new net: Q208.3 (D), Q240.1 (G), R166.2
- new net: Q185.3 (D), Q217.2 (S)
- new net: Q295.2 (S), Q296.3 (D)
- new net: D37.2, R133.2, R134.2
- new net: Q213.1 (G), Q229.1 (G), Q246.3 (D), Q278.1 (G), R188.2
- new net: Q303.2 (S), Q304.3 (D)
- new net: Q159.3 (D), Q303.3 (D), Q324.1 (G), R228.2
- new net: Q297.2 (S), Q298.3 (D)
- new net: Q179.3 (D), Q211.2 (S)
- new net: Q145.2 (S), Q146.3 (D)
- new net: D28.2, R106.2, R107.2
- new net: D39.2, R139.2, R140.2
- new net: D31.1, Q120.1 (G), Q71.3 (D), R39.2
- new net: Q180.3 (D), Q212.2 (S)
- new net: Q145.3 (D), Q289.3 (D), Q317.1 (G), R150.2
- new net: Q161.3 (D), Q305.3 (D), Q325.1 (G), R230.2
- new net: Q153.2 (S), Q154.3 (D)
- new net: Q213.3 (D), Q245.1 (G), R171.2
- new net: Q214.3 (D), Q246.1 (G), R172.2
- new net: Q199.3 (D), Q231.3 (D), Q263.1 (G), R205.2
- new net: Q289.2 (S), Q290.3 (D)
- new net: Q174.3 (D), Q206.2 (S)
- new net: D39.1, Q136.1 (G), Q77.3 (D), R43.2
- new net: Q196.3 (D), Q228.3 (D), Q260.1 (G), R202.2
- new net: Q176.3 (D), Q208.2 (S)
- new net: Q216.3 (D), Q248.1 (G), R174.2
- new net: Q183.3 (D), Q215.2 (S)
- new net: Q141.3 (D), Q285.3 (D), Q315.1 (G), R146.2
- new net: Q285.2 (S), Q286.3 (D)
- new net: Q155.2 (S), Q156.3 (D)
- new net: Q307.2 (S), Q308.3 (D)
- new net: D29.2, R109.2, R110.2
- new net: Q161.2 (S), Q162.3 (D)
- new net: Q311.2 (S), Q312.3 (D)
- new net: Q207.3 (D), Q239.1 (G), R165.2
- new net: Q187.3 (D), Q219.2 (S)
- new net: Q177.3 (D), Q209.2 (S)
- new net: Q182.3 (D), Q214.2 (S)
- new net: Q169.2 (S), Q170.3 (D)
- new net ADR 0: J2.14 (Pin_14), Q187.1 (G), Q203.1 (G), Q219.1 (G), Q235.1 (G)
- new net ADR 1: J2.15 (Pin_15), Q186.1 (G), Q202.1 (G)
- new net ADR 10: J3.16 (Pin_16), Q177.1 (G), Q193.1 (G)
- new net ADR 11: J3.17 (Pin_17), Q176.1 (G), Q192.1 (G)
- new net ADR 12: J3.18 (Pin_18), Q175.1 (G), Q191.1 (G)
- new net ADR 13: J3.19 (Pin_19), Q174.1 (G), Q190.1 (G)
- new net ADR 14: J3.20 (Pin_20), Q173.1 (G), Q189.1 (G)
- new net ADR 15: J3.21 (Pin_21), Q172.1 (G), Q188.1 (G)
- new net ADR 2: J2.16 (Pin_16), Q185.1 (G), Q201.1 (G)
- new net ADR 3: J2.17 (Pin_17), Q184.1 (G), Q200.1 (G)
- new net ADR 4: J2.18 (Pin_18), Q183.1 (G), Q199.1 (G)
- new net ADR 5: J2.19 (Pin_19), Q182.1 (G), Q198.1 (G)
- new net ADR 6: J2.20 (Pin_20), Q181.1 (G), Q197.1 (G)
- new net ADR 7: J2.21 (Pin_21), Q180.1 (G), Q196.1 (G)
- new net ADR 8: J3.14 (Pin_14), Q179.1 (G), Q195.1 (G)
- new net ADR 9: J3.15 (Pin_15), Q178.1 (G), Q194.1 (G)
- new net ADR TEMP HH: J3.4 (Pin_4), J5.4 (Pin_4)
- new net ADR TEMP LL: J2.4 (Pin_4), J4.4 (Pin_4)
- new net ADR++ 0: Q138.1 (G), Q267.3 (D), Q283.3 (D), R225.2
- new net ADR++ 1: Q140.1 (G), Q266.3 (D), Q282.3 (D), R224.2
- new net ADR++ 10: Q157.1 (G), Q257.3 (D), Q273.3 (D), R215.2
- new net ADR++ 11: Q159.1 (G), Q256.3 (D), Q272.3 (D), R214.2
- new net ADR++ 12: Q161.1 (G), Q255.3 (D), Q271.3 (D), R213.2
- new net ADR++ 13: Q163.1 (G), Q254.3 (D), Q270.3 (D), R212.2
- new net ADR++ 14: Q165.1 (G), Q253.3 (D), Q269.3 (D), R211.2
- new net ADR++ 15: Q167.1 (G), Q252.3 (D), Q268.3 (D), R210.2
- new net ADR++ 2: Q141.1 (G), Q265.3 (D), Q281.3 (D), R223.2
- new net ADR++ 3: Q143.1 (G), Q264.3 (D), Q280.3 (D), R222.2
- new net ADR++ 4: Q145.1 (G), Q263.3 (D), Q279.3 (D), R221.2
- new net ADR++ 5: Q147.1 (G), Q262.3 (D), Q278.3 (D), R220.2
- new net ADR++ 6: Q149.1 (G), Q261.3 (D), Q277.3 (D), R219.2
- new net ADR++ 7: Q151.1 (G), Q260.3 (D), Q276.3 (D), R218.2
- new net ADR++ 8: Q153.1 (G), Q259.3 (D), Q275.3 (D), R217.2
- new net ADR++ 9: Q155.1 (G), Q258.3 (D), Q274.3 (D), R216.2
- new net NEXT ADR 0: J2.6 (Pin_6), Q313.3 (D), R142.2
- new net NEXT ADR 1: J2.7 (Pin_7), Q314.3 (D), R145.2
- new net NEXT ADR 10: J3.8 (Pin_8), Q323.3 (D), R227.2
- new net NEXT ADR 11: J3.9 (Pin_9), Q324.3 (D), R229.2
- new net NEXT ADR 12: J3.10 (Pin_10), Q325.3 (D), R231.2
- new net NEXT ADR 13: J3.11 (Pin_11), Q326.3 (D), R233.2
- new net NEXT ADR 14: J3.12 (Pin_12), Q327.3 (D), R235.2
- new net NEXT ADR 15: J3.13 (Pin_13), Q328.3 (D), R237.2
- new net NEXT ADR 2: J2.8 (Pin_8), Q315.3 (D), R147.2
- new net NEXT ADR 3: J2.9 (Pin_9), Q316.3 (D), R149.2
- new net NEXT ADR 4: J2.10 (Pin_10), Q317.3 (D), R151.2
- new net NEXT ADR 5: J2.11 (Pin_11), Q318.3 (D), R153.2
- new net NEXT ADR 6: J2.12 (Pin_12), Q319.3 (D), R155.2
- new net NEXT ADR 7: J2.13 (Pin_13), Q320.3 (D), R157.2
- new net NEXT ADR 8: J3.6 (Pin_6), Q321.3 (D), R159.2
- new net NEXT ADR 9: J3.7 (Pin_7), Q322.3 (D), R161.2
- new net Read Next Address: Q137.1 (G), Q139.1 (G), Q142.1 (G), Q144.1 (G), Q146.1 (G), Q148.1 (G), Q150.1 (G), Q152.1 (G), Q154.1 (G), Q156.1 (G), Q158.1 (G), Q160.1 (G), Q162.1 (G), Q164.1 (G), Q166.1 (G), Q168.1 (G)
- new net Read Temp Address: Q170.1 (G), Q284.1 (G), Q286.1 (G), Q288.1 (G), Q290.1 (G), Q292.1 (G), Q294.1 (G), Q296.1 (G), Q298.1 (G), Q300.1 (G), Q302.1 (G), Q304.1 (G), Q306.1 (G), Q308.1 (G), Q310.1 (G), Q312.1 (G)
- new net Rising Edge: J2.5 (Pin_5), J3.5 (Pin_5), J4.5 (Pin_5), J5.5 (Pin_5)
- new net TEMP ADR 0: J4.14 (Pin_14), Q169.1 (G)
- new net TEMP ADR 1: J4.15 (Pin_15), Q171.1 (G)
- new net TEMP ADR 10: J5.16 (Pin_16), Q301.1 (G)
- new net TEMP ADR 11: J5.17 (Pin_17), Q303.1 (G)
- new net TEMP ADR 12: J5.18 (Pin_18), Q305.1 (G)
- new net TEMP ADR 13: J5.19 (Pin_19), Q307.1 (G)
- new net TEMP ADR 14: J5.20 (Pin_20), Q309.1 (G)
- new net TEMP ADR 15: J5.21 (Pin_21), Q311.1 (G)
- new net TEMP ADR 2: J4.16 (Pin_16), Q285.1 (G)
- new net TEMP ADR 3: J4.17 (Pin_17), Q287.1 (G)
- new net TEMP ADR 4: J4.18 (Pin_18), Q289.1 (G)
- new net TEMP ADR 5: J4.19 (Pin_19), Q291.1 (G)
- new net TEMP ADR 6: J4.20 (Pin_20), Q293.1 (G)
- new net TEMP ADR 7: J4.21 (Pin_21), Q295.1 (G)
- new net TEMP ADR 8: J5.14 (Pin_14), Q297.1 (G)
- new net TEMP ADR 9: J5.15 (Pin_15), Q299.1 (G)
Other:
- note added: "ALU A (which register is used in the ALU A input)"
- note added: "ALU B (which register is used in the ALU B input)"
- note added: "Address incrementer (for the next address in the program)"
- note added: "Endre navn på "ADR x" til "SAVED ADR x""
- note added: "INSTRUCTION DECODER"
- note added: "MEMORY ADDRESS"
- note added: "NEXT ADR MUX (decides the next stored address with multiplexer)"
- note added: "READ (for the which registers should read)"
- note added: "Read Flag (when the flags should be read)"
- note added: "TEMP MEMORY ADDRES"
- note removed: "ALU A"
- note removed: "ALU B"
- note removed: "READ"
- moved on the sheet: D1, D10, D11, D12, D13, D14, D15, D16, D17, D18, D19, D2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

Commit message: Controller unit v1.0 wip
Parts:
- added J6: Conn_01x21_Socket, symbol Connector:Conn_01x21_Socket
- added Q329, Q330, Q331, Q332, Q333, Q334, Q335, Q336, Q337, Q338, Q339, Q340, Q341, Q342, Q343, Q344, Q345, Q346, Q347, Q348, Q349, Q350, Q351, Q352, Q353, Q354, Q355, Q356, Q357, Q358, Q359, Q360, Q361, Q362, Q363, Q364, Q365, Q366, Q367, Q368, Q369, Q370, Q371, Q372, Q373, Q374, Q375, Q376, Q377, Q378, Q379, Q380, Q381, Q382, Q383, Q384, Q385, Q386, Q387, Q388, Q389, Q390, Q391, Q392, Q393, Q394, Q395, Q396, Q397, Q398, Q399, Q400, Q401, Q402, Q403, Q404, Q405, Q406, Q407, Q408, Q409, Q410, Q411, Q412, Q413, Q414, Q415, Q416, Q417, Q418, Q419, Q420, Q421, Q422, Q423, Q424, Q425, Q426, Q427, Q428, Q429, Q430, Q431, Q432, Q433, Q434, Q435, Q436, Q437, Q438, Q439, Q440, Q441, Q442: 2N7002, Package_TO_SOT_SMD:SOT-23, symbol Transistor_FET:2N7002
- added R238, R239, R240, R241, R242, R243, R244, R245, R246, R247, R248, R249, R250, R251, R252, R253, R254, R255, R256, R257, R258, R259, R260, R261, R262, R263, R264, R265, R266, R267, R268, R269, R270, R271, R272, R273, R274, R275, R276, R277, R278, R279, R280, R281, R282, R283, R284, R285, R286, R287, R288: 10kΩ, PCM_JLCPCB:R_0402, symbol PCM_JLCPCB-Resistors:0402,20kΩ
Connections:
- net ADR 0: now also Q333.3 (D), R239.2; no longer J2.14 (Pin_14), Q187.1 (G), Q203.1 (G), Q219.1 (G), Q235.1 (G)
- net ADR 1: now also Q338.3 (D), R241.2; no longer J2.15 (Pin_15), Q186.1 (G), Q202.1 (G)
- net ADR 10: now also Q383.3 (D), R259.2; no longer J3.16 (Pin_16), Q177.1 (G), Q193.1 (G)
- net ADR 11: now also Q388.3 (D), R261.2; no longer J3.17 (Pin_17), Q176.1 (G), Q192.1 (G)
- net ADR 12: now also Q393.3 (D), R263.2; no longer J3.18 (Pin_18), Q175.1 (G), Q191.1 (G)
- net ADR 13: now also Q398.3 (D), R265.2; no longer J3.19 (Pin_19), Q174.1 (G), Q190.1 (G)
- net ADR 14: now also Q403.3 (D), R267.2; no longer J3.20 (Pin_20), Q173.1 (G), Q189.1 (G)
- net ADR 15: now also Q408.3 (D), R269.2; no longer J3.21 (Pin_21), Q172.1 (G), Q188.1 (G)
- net ADR 2: now also Q343.3 (D), R243.2; no longer J2.16 (Pin_16), Q185.1 (G), Q201.1 (G)
- net ADR 3: now also Q348.3 (D), R245.2; no longer J2.17 (Pin_17), Q184.1 (G), Q200.1 (G)
- net ADR 4: now also Q353.3 (D), R247.2; no longer J2.18 (Pin_18), Q183.1 (G), Q199.1 (G)
- net ADR 5: now also Q358.3 (D), R249.2; no longer J2.19 (Pin_19), Q182.1 (G), Q198.1 (G)
- net ADR 6: now also Q363.3 (D), R251.2; no longer J2.20 (Pin_20), Q181.1 (G), Q197.1 (G)
- net ADR 7: now also Q368.3 (D), R253.2; no longer J2.21 (Pin_21), Q180.1 (G), Q196.1 (G)
- net ADR 8: now also Q373.3 (D), R255.2; no longer J3.14 (Pin_14), Q179.1 (G), Q195.1 (G)
- net ADR 9: now also Q378.3 (D), R257.2; no longer J3.15 (Pin_15), Q178.1 (G), Q194.1 (G)
- net GND: now also J6.2 (Pin_2), Q330.2 (S), Q332.2 (S), Q333.2 (S), Q335.2 (S), Q337.2 (S), Q338.2 (S), Q340.2 (S), Q342.2 (S), Q343.2 (S), Q345.2 (S), Q347.2 (S), Q348.2 (S), Q350.2 (S), Q352.2 (S), Q353.2 (S), Q355.2 (S), Q357.2 (S), Q358.2 (S), Q360.2 (S), Q362.2 (S), Q363.2 (S), Q365.2 (S), Q367.2 (S), Q368.2 (S), Q370.2 (S), Q372.2 (S), Q373.2 (S), Q375.2 (S), Q377.2 (S), Q378.2 (S), Q380.2 (S), Q382.2 (S), Q383.2 (S), Q385.2 (S), Q387.2 (S), Q388.2 (S), Q390.2 (S), Q392.2 (S), Q393.2 (S), Q395.2 (S), Q397.2 (S), Q398.2 (S), Q400.2 (S), Q402.2 (S), Q403.2 (S), Q405.2 (S), Q407.2 (S), Q408.2 (S), Q409.2 (S), Q410.2 (S), Q411.2 (S), Q412.2 (S), Q413.2 (S), Q414.2 (S), Q415.2 (S), Q416.2 (S), Q418.2 (S), Q420.2 (S), Q421.2 (S), Q423.2 (S), Q425.2 (S), Q426.2 (S), Q428.2 (S), Q430.2 (S), Q431.2 (S), Q433.2 (S), Q435.2 (S), Q436.2 (S), Q438.2 (S), Q440.2 (S), Q441.2 (S), Q442.2 (S)
- net READ FALG: now also Q420.1 (G), Q425.1 (G), Q430.1 (G), Q435.1 (G), Q440.1 (G), Q442.1 (G)
- net Rising Edge: now also J6.5 (Pin_5)
- net TEMP ADR 0: now also Q331.1 (G)
- net TEMP ADR 1: now also Q336.1 (G)
- net TEMP ADR 10: now also Q381.1 (G)
- net TEMP ADR 11: now also Q386.1 (G)
- net TEMP ADR 12: now also Q391.1 (G)
- net TEMP ADR 13: now also Q396.1 (G)
- net TEMP ADR 14: now also Q401.1 (G)
- net TEMP ADR 15: now also Q406.1 (G)
- net TEMP ADR 2: now also Q341.1 (G)
- net TEMP ADR 3: now also Q346.1 (G)
- net TEMP ADR 4: now also Q351.1 (G)
- net TEMP ADR 5: now also Q356.1 (G)
- net TEMP ADR 6: now also Q361.1 (G)
- net TEMP ADR 7: now also Q366.1 (G)
- net TEMP ADR 8: now also Q371.1 (G)
- net TEMP ADR 9: now also Q376.1 (G)
- net VCC: now also J2.4 (Pin_4), J3.4 (Pin_4), J6.1 (Pin_1), J6.4 (Pin_4), R238.1, R239.1, R240.1, R241.1, R242.1, R243.1, R244.1, R245.1, R246.1, R247.1, R248.1, R249.1, R250.1, R251.1, R252.1, R253.1, R254.1, R255.1, R256.1, R257.1, R258.1, R259.1, R260.1, R261.1, R262.1, R263.1, R264.1, R265.1, R266.1, R267.1, R268.1, R269.1, R270.1, R271.1, R272.1, R273.1, R274.1, R275.1, R276.1, R277.1, R278.1, R279.1, R280.1, R281.1, R282.1, R283.1, R284.1, R285.1, R286.1, R287.1, R288.1
- net rst: now also J6.3 (Pin_3)
- net ADR TEMP HH renamed TIME STEP 0
- net TIME STEP 0: now also J6.14 (Pin_14), Q409.1 (G); no longer J3.4 (Pin_4)
- net ADR TEMP LL renamed TIME STEP 1
- net TIME STEP 1: now also J6.15 (Pin_15), Q413.1 (G); no longer J2.4 (Pin_4)
- net Read Next Address renamed Store Next Address
- net Read Temp Address renamed Store Temp Address
- new net: Q369.3 (D), Q371.3 (D), Q373.1 (G), R254.2
- new net: Q439.2 (S), Q440.3 (D)
- new net: Q349.3 (D), Q351.3 (D), Q353.1 (G), R246.2
- new net: Q339.3 (D), Q341.3 (D), Q343.1 (G), R242.2
- new net: Q401.2 (S), Q402.3 (D)
- new net: Q359.2 (S), Q360.3 (D)
- new net: Q359.3 (D), Q361.3 (D), Q363.1 (G), R250.2
- new net: Q351.2 (S), Q352.3 (D)
- new net: Q381.2 (S), Q382.3 (D)
- new net: Q341.2 (S), Q342.3 (D)
- new net: Q389.3 (D), Q391.3 (D), Q393.1 (G), R262.2
- new net: Q376.2 (S), Q377.3 (D)
- new net: Q374.3 (D), Q376.3 (D), Q378.1 (G), R256.2
- new net: Q411.3 (D), Q412.1 (G), R272.2
- new net: Q379.3 (D), Q381.3 (D), Q383.1 (G), R258.2
- new net: Q386.2 (S), Q387.3 (D)
- new net: Q384.3 (D), Q386.3 (D), Q388.1 (G), R260.2
- new net: Q394.3 (D), Q396.3 (D), Q398.1 (G), R264.2
- new net: Q361.2 (S), Q362.3 (D)
- new net: Q389.2 (S), Q390.3 (D)
- new net: Q369.2 (S), Q370.3 (D)
- new net: Q346.2 (S), Q347.3 (D)
- new net: Q334.2 (S), Q335.3 (D)
- new net: Q334.3 (D), Q336.3 (D), Q338.1 (G), R240.2
- new net: Q371.2 (S), Q372.3 (D)
- new net: Q406.2 (S), Q407.3 (D)
- new net: Q404.3 (D), Q406.3 (D), Q408.1 (G), R268.2
- new net: Q422.3 (D), Q424.3 (D), Q426.1 (G), R280.2
- new net: Q399.2 (S), Q400.3 (D)
- new net: Q399.3 (D), Q401.3 (D), Q403.1 (G), R266.2
- new net: Q414.3 (D), Q415.1 (G), R275.2
- new net: Q427.3 (D), Q429.3 (D), Q431.1 (G), R282.2
- new net: Q409.3 (D), Q410.1 (G), R270.2
- new net: Q329.3 (D), Q331.3 (D), Q333.1 (G), R238.2
- new net: Q366.2 (S), Q367.3 (D)
- new net: Q384.2 (S), Q385.3 (D)
- new net: Q349.2 (S), Q350.3 (D)
- new net: Q437.3 (D), Q439.3 (D), Q441.1 (G), R286.2
- new net: Q404.2 (S), Q405.3 (D)
- new net: Q432.3 (D), Q434.3 (D), Q436.1 (G), R284.2
- new net: Q364.3 (D), Q366.3 (D), Q368.1 (G), R252.2
- new net: Q331.2 (S), Q332.3 (D)
- new net: Q329.2 (S), Q330.3 (D)
- new net: Q396.2 (S), Q397.3 (D)
- new net: Q391.2 (S), Q392.3 (D)
- new net: Q354.3 (D), Q356.3 (D), Q358.1 (G), R248.2
- new net: Q418.1 (G), Q423.1 (G), Q428.1 (G), Q433.1 (G), Q438.1 (G), Q442.3 (D), R288.2
- new net: Q427.2 (S), Q428.3 (D)
- new net: Q413.3 (D), Q414.1 (G), R274.2
- new net: Q336.2 (S), Q337.3 (D)
- new net: Q415.3 (D), Q416.1 (G), R276.2
- new net: Q434.2 (S), Q435.3 (D)
- new net: Q394.2 (S), Q395.3 (D)
- new net: Q344.3 (D), Q346.3 (D), Q348.1 (G), R244.2
- new net: Q429.2 (S), Q430.3 (D)
- new net: Q410.3 (D), Q411.1 (G), R271.2
- new net: Q422.2 (S), Q423.3 (D)
- new net: Q364.2 (S), Q365.3 (D)
- new net: Q417.3 (D), Q419.3 (D), Q421.1 (G), R278.2
- new net: Q344.2 (S), Q345.3 (D)
- new net: Q432.2 (S), Q433.3 (D)
- new net: Q354.2 (S), Q355.3 (D)
- new net: Q424.2 (S), Q425.3 (D)
- new net: Q379.2 (S), Q380.3 (D)
- new net: Q437.2 (S), Q438.3 (D)
- new net: Q374.2 (S), Q375.3 (D)
- new net: Q417.2 (S), Q418.3 (D)
- new net: Q419.2 (S), Q420.3 (D)
- new net: Q356.2 (S), Q357.3 (D)
- new net: Q339.2 (S), Q340.3 (D)
- new net ALU FLAG C: Q439.1 (G)
- new net ALU FLAG N: Q419.1 (G)
- new net ALU FLAG O: Q434.1 (G)
- new net ALU FLAG U: Q429.1 (G)
- new net ALU FLAG Z: Q424.1 (G)
- new net FLAG C: J6.21 (Pin_21), Q437.1 (G)
- new net FLAG N: J6.17 (Pin_17), Q417.1 (G)
- new net FLAG O: J6.20 (Pin_20), Q432.1 (G)
- new net FLAG STORE C: J6.13 (Pin_13), Q441.3 (D), R287.2
- new net FLAG STORE N: J6.9 (Pin_9), Q421.3 (D), R279.2
- new net FLAG STORE O: J6.12 (Pin_12), Q436.3 (D), R285.2
- new net FLAG STORE U: J6.11 (Pin_11), Q431.3 (D), R283.2
- new net FLAG STORE Z: J6.10 (Pin_10), Q426.3 (D), R281.2
- new net FLAG U: J6.19 (Pin_19), Q427.1 (G)
- new net FLAG Z: J6.18 (Pin_18), Q422.1 (G)
- new net Itterate address: Q219.1 (G), Q235.1 (G)
- new net Read From Temp Address: Q332.1 (G), Q337.1 (G), Q342.1 (G), Q347.1 (G), Q352.1 (G), Q357.1 (G), Q362.1 (G), Q367.1 (G), Q372.1 (G), Q377.1 (G), Q382.1 (G), Q387.1 (G), Q392.1 (G), Q397.1 (G), Q402.1 (G), Q407.1 (G)
- new net Read From stored Address: Q330.1 (G), Q335.1 (G), Q340.1 (G), Q345.1 (G), Q350.1 (G), Q355.1 (G), Q360.1 (G), Q365.1 (G), Q370.1 (G), Q375.1 (G), Q380.1 (G), Q385.1 (G), Q390.1 (G), Q395.1 (G), Q400.1 (G), Q405.1 (G)
- new net STORED ADR 0: J2.14 (Pin_14), Q187.1 (G), Q203.1 (G), Q329.1 (G)
- new net STORED ADR 1: J2.15 (Pin_15), Q186.1 (G), Q202.1 (G), Q334.1 (G)
- new net STORED ADR 10: J3.16 (Pin_16), Q177.1 (G), Q193.1 (G), Q379.1 (G)
- new net STORED ADR 11: J3.17 (Pin_17), Q176.1 (G), Q192.1 (G), Q384.1 (G)
- new net STORED ADR 12: J3.18 (Pin_18), Q175.1 (G), Q191.1 (G), Q389.1 (G)
- new net STORED ADR 13: J3.19 (Pin_19), Q174.1 (G), Q190.1 (G), Q394.1 (G)
- new net STORED ADR 14: J3.20 (Pin_20), Q173.1 (G), Q189.1 (G), Q399.1 (G)
- new net STORED ADR 15: J3.21 (Pin_21), Q172.1 (G), Q188.1 (G), Q404.1 (G)
- new net STORED ADR 2: J2.16 (Pin_16), Q185.1 (G), Q201.1 (G), Q339.1 (G)
- new net STORED ADR 3: J2.17 (Pin_17), Q184.1 (G), Q200.1 (G), Q344.1 (G)
- new net STORED ADR 4: J2.18 (Pin_18), Q183.1 (G), Q199.1 (G), Q349.1 (G)
- new net STORED ADR 5: J2.19 (Pin_19), Q182.1 (G), Q198.1 (G), Q354.1 (G)
- new net STORED ADR 6: J2.20 (Pin_20), Q181.1 (G), Q197.1 (G), Q359.1 (G)
- new net STORED ADR 7: J2.21 (Pin_21), Q180.1 (G), Q196.1 (G), Q364.1 (G)
- new net STORED ADR 8: J3.14 (Pin_14), Q179.1 (G), Q195.1 (G), Q369.1 (G)
- new net STORED ADR 9: J3.15 (Pin_15), Q178.1 (G), Q194.1 (G), Q374.1 (G)
- new net TIME STEP 2: J6.16 (Pin_16)
- new net TIME STEP IN 0: J6.6 (Pin_6)
- new net TIME STEP IN 1: J6.7 (Pin_7), Q412.3 (D), R273.2
- new net TIME STEP IN 2: J6.8 (Pin_8), Q416.3 (D), R277.2
Other:
- note added: "ADR MUX (decides the address to read from with multiplexer)"
- note added: "Buffer mellom ins reg til decoderen"
- note added: "DELAY FOR TIMING SIGNALS"
- note added: "LEGGE TIL TIME STEP IN 0"
- note added: "MUX FOR FLAG"
- note added: "NEXT STORED ADR MUX (decides the next stored address with multiplexer)"
- note added: "TIMING AND FLAGS"
- note removed: "Endre navn på "ADR x" til "SAVED ADR x""
- note removed: "NEXT ADR MUX (decides the next stored address with multiplexer)"
