File: PCB_S/Controller_Unit_V1.0/Controller_Unit_V1.0.kicad_sch (KiCad schematic)
At the start: 775 parts, among them J1 Conn_01x21_Socket, J2 Conn_01x21_Socket, J3 Conn_01x21_Socket, J4 Conn_01x21_Socket, J5 Conn_01x21_Socket, J6 Conn_01x21_Socket, Q1 2N7002, Q10 2N7002, Q100 2N7002, Q101 2N7002, Q102 2N7002, Q103 2N7002, Q104 2N7002, Q105 2N7002, Q106 2N7002, Q107 2N7002, Q108 2N7002, Q109 2N7002, Q11 2N7002, Q110 2N7002, Q111 2N7002, Q112 2N7002, Q113 2N7002, Q114 2N7002, Q115 2N7002, Q116 2N7002, Q117 2N7002, Q118 2N7002, Q119 2N7002, Q12 2N7002, Q120 2N7002, Q121 2N7002, Q122 2N7002, Q123 2N7002, Q124 2N7002, Q125 2N7002, Q126 2N7002, Q127 2N7002, Q128 2N7002, Q129 2N7002, Q13 2N7002, Q130 2N7002, Q131 2N7002, Q132 2N7002, Q133 2N7002, Q134 2N7002, Q135 2N7002, Q136 2N7002, Q137 2N7002, Q138 2N7002, Q139 2N7002, Q14 2N7002, Q140 2N7002, Q141 2N7002, Q142 2N7002, Q143 2N7002, Q144 2N7002, Q145 2N7002, Q146 2N7002, Q147 2N7002, Q148 2N7002, Q149 2N7002, Q15 2N7002, Q150 2N7002, Q151 2N7002, Q152 2N7002, Q153 2N7002, Q154 2N7002, Q155 2N7002, Q156 2N7002, Q157 2N7002, Q158 2N7002, Q159 2N7002, Q16 2N7002, Q160 2N7002, Q161 2N7002, Q162 2N7002, Q163 2N7002, Q164 2N7002, Q165 2N7002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

Commit message: controller unit v1.0 wip
Parts:
- added J10, J11, J12, J7, J8, J9: Conn_01x01_Pin, Connector_PinSocket_2.54mm:PinSocket_1x01_P2.54mm_Vertical, symbol Connector:Conn_01x01_Pin
- added Q443, Q444, Q445, Q446, Q447, Q448, Q449, Q450, Q451, Q452, Q453, Q454, Q455, Q456, Q457, Q458, Q459, Q460, Q461, Q462, Q463, Q464, Q465, Q466, Q467, Q468, Q469, Q470, Q471, Q472, Q473, Q475, Q476, Q477, Q478, Q479, Q480, Q481, Q482, Q483, Q484, Q485, Q486, Q487, Q488, Q489, Q490, Q491, Q492, Q493, Q494, Q495, Q496, Q497, Q498, Q499, Q500, Q501, Q502, Q503, Q504, Q505, Q506, Q507, Q508, Q509, Q510, Q511, Q512, Q513, Q514, Q515, Q516, Q517, Q518, Q519, Q520, Q521, Q522, Q523, Q524, Q525, Q526, Q527, Q528, Q529, Q530, Q531, Q532, Q533, Q534, Q535, Q536, Q537, Q538, Q539, Q540, Q541, Q542, Q543, Q544, Q545, Q546, Q547, Q548, Q549, Q550, Q551, Q552, Q553, Q554, Q555, Q556, Q557, Q558, Q559, Q560, Q561, Q562, Q563, Q564, Q565, Q566, Q567, Q568, Q569, Q570, Q571, Q572, Q573, Q574, Q575, Q576, Q577, Q578, Q579, Q580, Q581, Q582, Q583, Q584: 2N7002, Package_TO_SOT_SMD:SOT-23, symbol Transistor_FET:2N7002
- added R289, R290, R291, R292, R293, R294, R295, R296, R297, R298, R299, R300, R301, R302, R303, R304, R305, R306, R307, R308, R309, R310, R311, R312, R313, R314, R315, R316, R317, R318, R319, R320, R321, R322, R323, R324, R325, R326, R327, R328, R329, R330, R331, R332, R333, R334, R335, R336, R337, R338, R339, R340, R341, R342, R343, R344, R345: 10kΩ, PCM_JLCPCB:R_0402, symbol PCM_JLCPCB-Resistors:0402,20kΩ
Connections:
- net !ADC: now also Q568.1 (G), Q582.1 (G)
- net !ADD: now also Q567.1 (G)
- net !AND: now also Q576.1 (G)
- net !BNC: now also Q453.1 (G), Q472.1 (G)
- net !BNO: now also Q449.1 (G), Q464.1 (G)
- net !BNU: now also Q451.1 (G), Q468.1 (G)
- net !BNZ: now also Q447.1 (G), Q460.1 (G)
- net !BOC: now also Q452.1 (G), Q470.1 (G)
- net !BON: now also Q445.1 (G), Q454.1 (G)
- net !BOO: now also Q448.1 (G), Q462.1 (G)
- net !BOP: now also Q444.1 (G), Q456.1 (G)
- net !BOU: now also Q450.1 (G), Q466.1 (G)
- net !BOZ: now also Q446.1 (G), Q458.1 (G)
- net !DEC: now also Q565.1 (G), Q572.1 (G)
- net !INC: now also Q566.1 (G), Q583.1 (G)
- net !JMP: now also Q443.1 (G), Q492.1 (G)
- net !Load: now also Q497.1 (G)
- net !MOV: now also Q578.1 (G)
- net !NOT: now also Q574.1 (G)
- net !OR: now also Q579.1 (G)
- net !RS: now also Q575.1 (G)
- net !Store: now also Q496.1 (G), Q515.1 (G), Q577.1 (G)
- net !XOR: now also Q573.1 (G)
- net Buss0: now also Q517.3 (D), Q541.1 (G)
- net Buss1: now also Q521.3 (D), Q544.1 (G)
- net Buss2: now also Q524.3 (D), Q547.1 (G)
- net Buss3: now also Q527.3 (D), Q550.1 (G)
- net Buss4: now also Q530.3 (D), Q553.1 (G)
- net Buss5: now also Q533.3 (D), Q556.1 (G)
- net Buss6: now also Q536.3 (D), Q559.1 (G)
- net Buss7: now also Q539.3 (D), Q562.1 (G)
- net FLAG C: now also Q471.1 (G), Q479.1 (G), Q580.1 (G)
- net FLAG N: now also Q455.1 (G), Q457.1 (G)
- net FLAG O: now also Q463.1 (G), Q477.1 (G)
- net FLAG U: now also Q467.1 (G), Q478.1 (G)
- net FLAG Z: now also Q459.1 (G), Q475.1 (G), Q476.1 (G)
- net GND: now also J11.1 (Pin_1), Q443.2 (S), Q454.2 (S), Q455.2 (S), Q456.2 (S), Q457.2 (S), Q458.2 (S), Q459.2 (S), Q460.2 (S), Q461.2 (S), Q462.2 (S), Q463.2 (S), Q464.2 (S), Q465.2 (S), Q466.2 (S), Q467.2 (S), Q468.2 (S), Q469.2 (S), Q470.2 (S), Q471.2 (S), Q472.2 (S), Q473.2 (S), Q475.2 (S), Q476.2 (S), Q477.2 (S), Q478.2 (S), Q479.2 (S), Q480.2 (S), Q481.2 (S), Q482.2 (S), Q483.2 (S), Q484.2 (S), Q485.2 (S), Q486.2 (S), Q487.2 (S), Q488.2 (S), Q489.2 (S), Q490.2 (S), Q491.2 (S), Q492.2 (S), Q493.2 (S), Q494.2 (S), Q497.2 (S), Q499.2 (S), Q501.2 (S), Q502.2 (S), Q503.2 (S), Q504.2 (S), Q505.2 (S), Q506.2 (S), Q507.2 (S), Q508.2 (S), Q509.2 (S), Q511.2 (S), Q513.2 (S), Q515.2 (S), Q518.2 (S), Q519.2 (S), Q520.2 (S), Q522.2 (S), Q523.2 (S), Q525.2 (S), Q526.2 (S), Q528.2 (S), Q529.2 (S), Q531.2 (S), Q532.2 (S), Q534.2 (S), Q535.2 (S), Q537.2 (S), Q538.2 (S), Q540.2 (S), Q541.2 (S), Q543.2 (S), Q544.2 (S), Q546.2 (S), Q547.2 (S), Q549.2 (S), Q550.2 (S), Q552.2 (S), Q553.2 (S), Q555.2 (S), Q556.2 (S), Q558.2 (S), Q559.2 (S), Q561.2 (S), Q562.2 (S), Q564.2 (S), Q565.2 (S), Q570.2 (S), Q571.2 (S), Q572.2 (S), Q573.2 (S), Q574.2 (S), Q575.2 (S), Q576.2 (S), Q577.2 (S), Q580.2 (S), Q582.2 (S), Q584.2 (S)
- net Read New Instruction: now also J9.1 (Pin_1)
- net TIME STEP 0: now also Q503.1 (G), Q507.1 (G)
- net TIME STEP 1: now also Q504.1 (G), Q508.1 (G)
- net TIME STEP 2: now also Q505.1 (G), Q516.1 (G)
- net TIME STEP IN 0: now also Q502.3 (D), R312.2
- net TIME STEP IN 2: now also Q495.1 (G)
- net VCC: now also J12.1 (Pin_1), R289.1, R290.1, R291.1, R292.1, R293.1, R294.1, R295.1, R296.1, R297.1, R298.1, R299.1, R300.1, R301.1, R302.1, R303.1, R304.1, R305.1, R306.1, R307.1, R308.1, R309.1, R310.1, R311.1, R312.1, R313.1, R314.1, R315.1, R316.1, R317.1, R318.1, R319.1, R320.1, R321.1, R322.1, R323.1, R324.1, R325.1, R326.1, R327.1, R328.1, R329.1, R330.1, R331.1, R332.1, R333.1, R334.1, R335.1, R336.1, R337.1, R338.1, R339.1, R340.1, R341.1, R342.1, R343.1, R344.1, R345.1
- net !TIME STEP 0: now reaches Q409.3 (D), Q410.1 (G), R270.2
- net !TIME STEP 0: now also Q514.1 (G)
- net Store Next Address renamed Store Address ++
- net Store Address ++: now also Q493.1 (G), Q495.3 (D), R309.2
- net Store Temp Address: no longer names the net of Q170.1 (G), Q284.1 (G), Q286.1 (G), Q288.1 (G), Q290.1 (G), Q292.1 (G), Q294.1 (G), Q296.1 (G), Q298.1 (G), Q300.1 (G), Q302.1 (G), Q304.1 (G), Q306.1 (G), Q308.1 (G), Q310.1 (G), Q312.1 (G)
- net Store Temp Address: now also Q493.3 (D), R308.2
- new net: Q544.3 (D), Q545.1 (G), R327.2
- new net: Q473.1 (G), Q479.3 (D), R304.2
- new net: Q456.3 (D), Q457.3 (D), Q475.3 (D), Q480.1 (G), R291.2
- new net: Q480.3 (D), Q481.3 (D), Q482.3 (D), Q483.3 (D), Q484.3 (D), Q485.3 (D), Q486.3 (D), Q487.3 (D), Q488.3 (D), Q489.3 (D), Q490.1 (G), Q491.3 (D), R305.2
- new net: Q458.3 (D), Q459.3 (D), Q482.1 (G), R292.2
- new net: Q498.2 (S), Q499.3 (D)
- new net: Q498.3 (D), Q500.3 (D), Q502.1 (G), R311.2
- new net: Q577.3 (D), Q578.2 (S)
- new net: Q559.3 (D), Q560.1 (G), R332.2
- new net: Q451.3 (D), Q452.2 (S)
- new net: Q452.3 (D), Q453.2 (S)
- new net: J7.1 (Pin_1), Q510.3 (D), Q512.3 (D), Q570.1 (G), R317.2
- new net: Q569.2 (S), Q570.3 (D)
- new net: Q496.2 (S), Q497.3 (D)
- new net: Q499.1 (G), Q507.3 (D), Q508.3 (D), Q509.1 (G), R315.2
- new net: Q578.3 (D), Q579.2 (S)
- new net: Q550.3 (D), Q551.1 (G), R329.2
- new net: Q551.2 (S), Q552.3 (D)
- new net: Q538.3 (D), Q539.1 (G), R325.2
- new net: Q539.2 (S), Q540.3 (D)
- new net: Q545.2 (S), Q546.3 (D)
- new net: Q548.2 (S), Q549.3 (D)
- new net: J10.1 (Pin_1), Q569.1 (G)
- new net: Q569.3 (D), Q571.1 (G), R335.2
- new net: Q494.3 (D), Q495.2 (S)
- new net: Q529.3 (D), Q530.1 (G), R322.2
- new net: Q461.1 (G), Q476.3 (D), R301.2
- new net: Q460.3 (D), Q461.3 (D), Q483.1 (G), R293.2
- new net: Q556.3 (D), Q557.1 (G), R331.2
- new net: Q526.3 (D), Q527.1 (G), R321.2
- new net: Q462.3 (D), Q463.3 (D), Q484.1 (G), R294.2
- new net: Q583.2 (S), Q584.3 (D)
- new net: Q454.3 (D), Q455.3 (D), Q481.1 (G), R290.2
- new net: Q541.3 (D), Q542.1 (G), R326.2
- new net: Q450.3 (D), Q451.2 (S)
- new net: Q523.3 (D), Q524.1 (G), R320.2
- new net: Q472.3 (D), Q473.3 (D), Q489.1 (G), R299.2
- new net: Q469.1 (G), Q478.3 (D), R303.2
- new net: Q520.3 (D), Q521.1 (G), R319.2
- new net: Q468.3 (D), Q469.3 (D), Q487.1 (G), R297.2
- new net: Q562.3 (D), Q563.1 (G), R333.2
- new net: Q501.1 (G), Q503.3 (D), Q504.3 (D), Q505.3 (D), Q506.1 (G), R314.2
- new net: Q446.3 (D), Q447.2 (S)
- new net: Q447.3 (D), Q448.2 (S)
- new net: Q560.2 (S), Q561.3 (D)
- new net: Q553.3 (D), Q554.1 (G), R330.2
- new net: Q500.2 (S), Q501.3 (D)
- new net: Q517.2 (S), Q518.3 (D)
- new net: Q567.3 (D), Q568.2 (S)
- new net: Q563.2 (S), Q564.3 (D)
- new net: Q515.3 (D), Q516.2 (S)
- new net: Q514.2 (S), Q516.3 (D)
- new net: Q491.1 (G), Q492.3 (D), R307.2
- new net: Q557.2 (S), Q558.3 (D)
- new net: Q535.3 (D), Q536.1 (G), R324.2
- new net: Q536.2 (S), Q537.3 (D)
- new net: Q547.3 (D), Q548.1 (G), R328.2
- new net: Q510.2 (S), Q511.3 (D)
- new net: Q527.2 (S), Q528.3 (D)
- new net: Q464.3 (D), Q465.3 (D), Q485.1 (G), R295.2
- new net: Q530.2 (S), Q531.3 (D)
- new net: Q449.3 (D), Q450.2 (S)
- new net: Q565.3 (D), Q566.2 (S)
- new net: Q566.3 (D), Q567.2 (S)
- new net: Q445.3 (D), Q446.2 (S)
- new net: Q444.3 (D), Q445.2 (S)
- new net: Q580.3 (D), Q581.2 (S)
- new net: Q517.1 (G), Q519.3 (D), R318.2
- new net: Q466.3 (D), Q467.3 (D), Q486.1 (G), R296.2
- new net: Q581.3 (D), Q584.1 (G), R343.2
- new net: Q581.1 (G), Q582.3 (D), R345.2
- new net: Q521.2 (S), Q522.3 (D)
- new net: Q524.2 (S), Q525.3 (D)
- new net: Q532.3 (D), Q533.1 (G), R323.2
- new net: Q470.3 (D), Q471.3 (D), Q488.1 (G), R298.2
- new net: Q512.2 (S), Q513.3 (D)
- new net: Q465.1 (G), Q477.3 (D), R302.2
- new net: Q533.2 (S), Q534.3 (D)
- new net: Q542.2 (S), Q543.3 (D)
- new net: J8.1 (Pin_1), Q571.3 (D), R336.2
- new net: Q554.2 (S), Q555.3 (D)
- new net: Q443.3 (D), Q444.2 (S)
- new net: Q448.3 (D), Q449.2 (S)
- new net ADD: Q568.3 (D), R334.2
- new net ALU B = FF: Q572.3 (D), R337.2
- new net AND: Q576.3 (D), R341.2
- new net Carry in: Q583.3 (D), R344.2
- new net Commit jump: Q490.3 (D), Q494.1 (G), R306.2
- new net Main bus -> bus out: Q518.1 (G), Q522.1 (G), Q525.1 (G), Q528.1 (G), Q531.1 (G), Q534.1 (G), Q537.1 (G), Q540.1 (G)
- new net Main bus 0: Q519.1 (G), Q542.3 (D)
- new net Main bus 1: Q520.1 (G), Q545.3 (D)
- new net Main bus 2: Q523.1 (G), Q548.3 (D)
- new net Main bus 3: Q526.1 (G), Q551.3 (D)
- new net Main bus 4: Q529.1 (G), Q554.3 (D)
- new net Main bus 5: Q532.1 (G), Q557.3 (D)
- new net Main bus 6: Q535.1 (G), Q560.3 (D)
- new net Main bus 7: Q538.1 (G), Q563.3 (D)
- new net NOT: Q574.3 (D), R339.2
- new net OR: Q579.3 (D), R342.2
- new net RS: Q575.3 (D), R340.2
- new net Read Write ins: Q496.3 (D), Q500.1 (G), Q513.1 (G), R310.2
- new net R/W out: Q514.3 (D), R300.2
- new net TIME STEP 0or1: Q509.3 (D), Q510.1 (G), R316.2
- new net TIME STEP 0or1or2: Q506.3 (D), Q512.1 (G), R313.2
- new net XOR: Q573.3 (D), R338.2
- new net bus out -> Main bus: Q543.1 (G), Q546.1 (G), Q549.1 (G), Q552.1 (G), Q555.1 (G), Q558.1 (G), Q561.1 (G), Q564.1 (G)
- new net jump type instruction: Q453.3 (D), Q498.1 (G), Q511.1 (G), R289.2
Other:
- note added: "!clock"
- note added: "IGNORE"
- note added: "Inputs/outputs"
- note added: "Kan være alle negativ og positive flagg instruksene er flipet så "branch on" -> "branch not" visa versa"
- note added: "Makes sure we dont read new instructions while a jump or read/write happens"
- note added: "falure point (timing issue) (may need to change inputs for "read new instruction")"
- note added: "falure point (timing issue) (may need to change resistor)"
- note added: "nr 1"
- note added: "nr 2"
- note added: "read / write from memory (1 is read from memory and 0 is wrtite to memory)"

Commit message: cercuit done controller unit v1.0 ?
Parts:
- added Q474, Q585, Q586, Q587, Q588, Q589, Q590, Q591, Q592, Q593, Q594, Q595: 2N7002, Package_TO_SOT_SMD:SOT-23, symbol Transistor_FET:2N7002
- added R346, R347, R348, R349, R350, R351, R352, R353, R354, R355: 10kΩ, PCM_JLCPCB:R_0402, symbol PCM_JLCPCB-Resistors:0402,20kΩ
Connections:
- net Itterate address is gone; now on net Read From stored Address: Q219.1 (G), Q235.1 (G)
- net !Clear: now also Q516.1 (G)
- net !Load: now also Q590.1 (G)
- net !Store: now also Q591.1 (G), Q595.1 (G); no longer Q515.1 (G)
- net !TIME STEP 0: now also Q585.1 (G); no longer Q514.1 (G)
- net AND: no longer Q576.3 (D)
- net FLAG C: now also Q473.1 (G); no longer Q471.1 (G)
- net FLAG N: now also Q594.1 (G); no longer Q455.1 (G)
- net FLAG O: now also Q465.1 (G); no longer Q463.1 (G)
- net FLAG U: now also Q469.1 (G); no longer Q467.1 (G)
- net FLAG Z: now also Q461.1 (G); no longer Q459.1 (G)
- net GND: now also Q514.2 (S), Q586.2 (S), Q587.2 (S), Q589.2 (S), Q590.2 (S), Q591.2 (S), Q593.2 (S), Q594.2 (S), Q595.2 (S); no longer Q515.2 (S)
- net Main bus -> bus out: now also Q593.3 (D), R353.2
- net Read From stored Address: now also Q514.1 (G), Q474.3 (D), R346.2
- net Read New Instruction: no longer J1.5 (Pin_5)
- net Read Write ins: now also Q474.1 (G)
- net Rising Edge: no longer J4.5 (Pin_5), J5.5 (Pin_5)
- net R/W out: now also Q515.3 (D); no longer Q514.3 (D)
- net TIME STEP 2: now also Q586.1 (G), Q587.1 (G); no longer Q516.1 (G)
- net VCC: now also R346.1, R347.1, R348.1, R349.1, R350.1, R351.1, R352.1, R353.1, R354.1, R355.1
- net bus out -> Main bus: now also Q589.3 (D), R349.2
- net at Q479.3 (D), R304.2: now also Q471.1 (G); no longer Q473.1 (G)
- net at Q476.3 (D), R301.2: now also Q459.1 (G); no longer Q461.1 (G)
- net at Q478.3 (D), R303.2: now also Q467.1 (G); no longer Q469.1 (G)
- net at Q516.2 (S): now also Q576.3 (D); no longer Q515.3 (D)
- net at Q516.3 (D): no longer Q514.2 (S)
- net at Q477.3 (D), R302.2: now also Q463.1 (G); no longer Q465.1 (G)
- net Read From Temp Address: no longer names the net of Q332.1 (G), Q337.1 (G), Q342.1 (G), Q347.1 (G), Q352.1 (G), Q357.1 (G), Q362.1 (G), Q367.1 (G), Q372.1 (G), Q377.1 (G), Q382.1 (G), Q387.1 (G), Q392.1 (G), Q397.1 (G), Q402.1 (G), Q407.1 (G)
- net Read From Temp Address: now also Q514.3 (D), R347.2
- new net: Q588.3 (D), Q589.1 (G), R348.2
- new net: Q588.1 (G), Q590.3 (D), R350.2
- new net: Q587.3 (D), Q588.2 (S), Q592.2 (S)
- new net: Q585.2 (S), Q586.3 (D)
- new net: Q592.3 (D), Q593.1 (G), R352.2
- new net: Q515.1 (G), Q595.3 (D), R355.2
- new net: Q591.3 (D), Q592.1 (G), R351.2
- new net: Q455.1 (G), Q594.3 (D), R354.2
- new net: Q474.2 (S), Q515.2 (S), Q585.3 (D)
- new net Faling Edge: J1.5 (Pin_5), J4.5 (Pin_5), J5.5 (Pin_5)
Other:
- note removed: "Kan være alle negativ og positive flagg instruksene er flipet så "branch on" -> "branch not" visa versa"
