File: PCB_S/Controller_Unit_V1.0/Controller_Unit_V1.0.kicad_sch (KiCad schematic)
At the start: 1001 parts, among them J1 Conn_01x21_Socket, J10 Conn_01x01_Pin, J11 Conn_01x01_Pin, J12 Conn_01x01_Pin, J2 Conn_01x21_Socket, J3 Conn_01x21_Socket, J4 Conn_01x21_Socket, J5 Conn_01x21_Socket, J6 Conn_01x21_Socket, J7 Conn_01x01_Pin, J8 Conn_01x01_Pin, J9 Conn_01x01_Pin, Q1 2N7002, Q10 2N7002, Q100 2N7002, Q101 2N7002, Q102 2N7002, Q103 2N7002, Q104 2N7002, Q105 2N7002, Q106 2N7002, Q107 2N7002, Q108 2N7002, Q109 2N7002, Q11 2N7002, Q110 2N7002, Q111 2N7002, Q112 2N7002, Q113 2N7002, Q114 2N7002, Q115 2N7002, Q116 2N7002, Q117 2N7002, Q118 2N7002, Q119 2N7002, Q12 2N7002, Q120 2N7002, Q121 2N7002, Q122 2N7002, Q123 2N7002, Q124 2N7002, Q125 2N7002, Q126 2N7002, Q127 2N7002, Q128 2N7002, Q129 2N7002, Q13 2N7002, Q130 2N7002, Q131 2N7002, Q132 2N7002, Q133 2N7002, Q134 2N7002, Q135 2N7002, Q136 2N7002, Q137 2N7002, Q138 2N7002, Q139 2N7002, Q14 2N7002, Q140 2N7002, Q141 2N7002, Q142 2N7002, Q143 2N7002, Q144 2N7002, Q145 2N7002, Q146 2N7002, Q147 2N7002, Q148 2N7002, Q149 2N7002, Q15 2N7002, Q150 2N7002, Q151 2N7002, Q152 2N7002, Q153 2N7002, Q154 2N7002, Q155 2N7002, Q156 2N7002, Q157 2N7002, Q158 2N7002, Q159 2N7002, Q16 2N7002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

Commit message: Controller unit PCB wip
Parts:
- removed D12, D13, D14: Red, PCM_JLCPCB:D_0603, symbol PCM_JLCPCB-Diodes:LED,0603,Red
- removed J10, J11, J12: Conn_01x01_Pin, Connector_PinSocket_2.54mm:PinSocket_1x01_P2.54mm_Vertical, symbol Connector:Conn_01x01_Pin
- removed Q135, Q36, Q37, Q38, Q39: 2N7002, Package_TO_SOT_SMD:SOT-23, symbol Transistor_FET:2N7002
- removed R20, R21, R22, R74, R75, R76, R77, R78, R79: 10kΩ, PCM_JLCPCB:R_0402, symbol PCM_JLCPCB-Resistors:0402,20kΩ
- added C1, C2: C, Capacitor_THT:C_Disc_D4.7mm_W2.5mm_P5.00mm, symbol Device:C
- added D40, D41, D42, D43, D44, D45, D46, D47, D48, D49, D50, D51, D52, D53, D54, D55, D56, D57, D58, D59, D60, D61, D62, D63, D64, D65, D66, D67, D68, D69, D70, D71, D72, D73, D74, D75, D76, D77, D78, D79, D80, D81, D82, D95, D96: Red, PCM_JLCPCB:D_0603, symbol PCM_JLCPCB-Diodes:LED,0603,Red
- added J10, J11, J12, J13, J14: Conn_02x08_Odd_Even, Connector_PinSocket_2.54mm:PinSocket_2x08_P2.54mm_Vertical, symbol Connector_Generic:Conn_02x08_Odd_Even
- added Q596, Q597, Q598, Q599, Q600, Q601, Q602, Q603, Q604, Q605, Q606, Q607, Q608, Q609, Q610, Q611, Q612, Q613, Q614, Q615, Q616, Q617, Q618, Q619, Q620, Q621, Q622, Q623, Q624, Q625, Q626, Q627, Q628, Q629, Q630, Q631, Q632, Q645, Q646: 2N7002, Package_TO_SOT_SMD:SOT-23, symbol Transistor_FET:2N7002
- added R356, R357, R358, R359, R360, R361, R362, R363, R364, R365, R366, R367, R368, R369, R370, R371, R372, R373, R374, R375, R376, R377, R378, R379, R380, R381, R382, R383, R384, R385, R386, R387, R390, R391, R392, R393, R394, R395, R396, R397, R398, R399, R400, R401, R402, R403, R404, R405, R406, R407, R408, R409, R412, R413, R414, R415, R416, R417, R418, R419, R420, R421, R422, R423, R424, R425, R426, R427, R428, R429, R430, R431, R432, R433, R434, R435, R436, R437, R438, R439, R440, R441, R442, R443, R444, R445, R446, R447, R448, R449, R450, R451, R452, R453, R454, R455, R456, R457, R458, R459, R460, R461, R462, R463, R464, R465, R466, R467, R468, R469, R470, R471, R472, R473, R474, R475, R476, R477, R478, R479, R480, R481, R482, R483, R484, R485, R486, R487, R488, R489, R490, R491, R492, R493, R494, R495, R496, R497, R498, R499, R500, R501, R502, R503, R504, R505, R506, R507, R508, R509, R510, R511, R512, R513, R514, R515, R516, R517, R518, R519, R520, R521, R522, R523, R524, R525, R526, R527, R528, R553, R554, R555, R556: 10kΩ, PCM_JLCPCB:R_0402, symbol PCM_JLCPCB-Resistors:0402,20kΩ
- added R388, R389, R410, R411: R, Resistor_THT:R_Axial_DIN0309_L9.0mm_D3.2mm_P12.70mm_Horizontal, symbol Device:R
- J1, J2, J3, J4, J5, J6: footprint (none) -> Connector_PinHeader_2.54mm:PinHeader_1x21_P2.54mm_Vertical
Connections:
- net A ->ALU A: now also J14.2 (Pin_2)
- net A ->ALU B: now also J14.10 (Pin_10)
- net ADD: now also J13.4 (Pin_4), R454.2, R455.2; no longer R334.2
- net ADR 0: now also J11.1 (Pin_1)
- net ADR 1: now also J11.3 (Pin_3)
- net ADR 10: now also J11.6 (Pin_6)
- net ADR 11: now also J11.8 (Pin_8)
- net ADR 12: now also J11.10 (Pin_10)
- net ADR 13: now also J11.12 (Pin_12)
- net ADR 14: now also J11.14 (Pin_14)
- net ADR 15: now also J11.16 (Pin_16)
- net ADR 2: now also J11.5 (Pin_5)
- net ADR 3: now also J11.7 (Pin_7)
- net ADR 4: now also J11.9 (Pin_9)
- net ADR 5: now also J11.11 (Pin_11)
- net ADR 6: now also J11.13 (Pin_13)
- net ADR 7: now also J11.15 (Pin_15)
- net ADR 8: now also J11.2 (Pin_2)
- net ADR 9: now also J11.4 (Pin_4)
- net ADR++ 0: now also Q630.1 (G)
- net ADR++ 1: now also Q629.1 (G)
- net ADR++ 10: now also Q620.1 (G)
- net ADR++ 11: now also Q619.1 (G)
- net ADR++ 12: now also Q618.1 (G)
- net ADR++ 13: now also Q617.1 (G)
- net ADR++ 14: now also Q615.1 (G)
- net ADR++ 15: now also Q616.1 (G)
- net ADR++ 2: now also Q628.1 (G)
- net ADR++ 3: now also Q627.1 (G)
- net ADR++ 4: now also Q626.1 (G)
- net ADR++ 5: now also Q625.1 (G)
- net ADR++ 6: now also Q624.1 (G)
- net ADR++ 7: now also Q623.1 (G)
- net ADR++ 8: now also Q622.1 (G)
- net ADR++ 9: now also Q621.1 (G)
- net ALU B = FF: now also J14.9 (Pin_9), R456.2
- net ALU FLAG C: now also J13.11 (Pin_11)
- net ALU FLAG N: now also J13.3 (Pin_3)
- net ALU FLAG O: now also J13.9 (Pin_9)
- net ALU FLAG U: now also J13.7 (Pin_7)
- net ALU FLAG Z: now also J13.5 (Pin_5)
- net AND: now also Q516.3 (D), J13.12 (Pin_12), R459.2
- net B ->ALU A: now also J14.4 (Pin_4)
- net B ->ALU B: now also J14.12 (Pin_12)
- net Buss0: now also J10.1 (Pin_1)
- net Buss1: now also J10.3 (Pin_3)
- net Buss2: now also J10.5 (Pin_5)
- net Buss3: now also J10.7 (Pin_7)
- net Buss4: now also J10.9 (Pin_9)
- net Buss5: now also J10.11 (Pin_11)
- net Buss6: now also J10.13 (Pin_13)
- net Buss7: now also J10.15 (Pin_15)
- net C ->ALU A: now also J14.6 (Pin_6)
- net C ->ALU B: now also J14.14 (Pin_14)
- net Carry in: now also J13.13 (Pin_13)
- net Commit jump: now also Q569.1 (G)
- net D ->ALU A: now also J14.8 (Pin_8)
- net D ->ALU B: now also J14.16 (Pin_16)
- net Faling Edge: now also J7.1 (Pin_1), Q609.3 (D), R402.2, R403.2, R404.2, R405.2, R412.2, R413.2, R414.2, R415.2
- net GND: now also Q569.2 (S), J10.10 (Pin_10), J10.14 (Pin_14), J10.4 (Pin_4), J12.12 (Pin_12), J12.16 (Pin_16), J12.4 (Pin_4), J12.8 (Pin_8), J13.1 (Pin_1), J13.15 (Pin_15), J14.15 (Pin_15), Q596.2 (S), Q597.2 (S), Q598.2 (S), Q599.2 (S), Q600.2 (S), Q601.2 (S), Q602.2 (S), Q603.2 (S), Q604.2 (S), Q605.2 (S), Q606.2 (S), Q607.2 (S), Q608.2 (S), Q609.2 (S), Q610.2 (S), Q611.2 (S), Q612.2 (S), Q613.2 (S), Q614.2 (S), Q615.2 (S), Q616.2 (S), Q617.2 (S), Q618.2 (S), Q619.2 (S), Q620.2 (S), Q621.2 (S), Q622.2 (S), Q623.2 (S), Q624.2 (S), Q625.2 (S), Q626.2 (S), Q627.2 (S), Q628.2 (S), Q629.2 (S), Q630.2 (S), Q631.2 (S), Q632.2 (S), Q645.2 (S), Q646.2 (S), R388.2, R389.2, R410.2, R411.2; no longer Q73.2 (S)
- net Main bus -> bus out: now also Q613.1 (G), R441.2
- net Main bus 0: now also J12.1 (Pin_1)
- net Main bus 1: now also J12.3 (Pin_3)
- net Main bus 2: now also J12.5 (Pin_5)
- net Main bus 3: now also J12.7 (Pin_7)
- net Main bus 4: now also J12.9 (Pin_9)
- net Main bus 5: now also J12.11 (Pin_11)
- net Main bus 6: now also J12.13 (Pin_13)
- net Main bus 7: now also J12.15 (Pin_15)
- net NOT: now also J13.8 (Pin_8), R457.2
- net OR: now also J13.14 (Pin_14), R460.2
- net READ A: now also J14.1 (Pin_1)
- net READ B: now also J14.3 (Pin_3)
- net READ C: now also J14.5 (Pin_5)
- net READ D: now also J14.7 (Pin_7)
- net READ FALG: now also Q134.3 (D), Q646.1 (G)
- net REG -> ALU A: now also Q631.1 (G)
- net REG -> ALU B: now also Q645.1 (G)
- net REG Read: now also Q632.1 (G)
- net RS: now also J13.10 (Pin_10), R458.2
- net Read From stored Address: now also Q612.1 (G), R440.2, R443.2, R444.2
- net Read New Instruction: now also Q510.3 (D), Q512.3 (D), Q571.1 (G), R317.2
- net Read Write ins: now also Q611.1 (G)
- net Rising Edge: now also J8.1 (Pin_1), J14.11 (Pin_11), Q608.3 (D), R398.2, R399.2, R400.2, R401.2, R416.2, R417.2, R418.2, R419.2
- net R/W out: now also J10.12 (Pin_12)
- net Store Address ++: now also Q570.1 (G), R448.2, R449.2, R450.2
- net TIME STEP IN 0: now also Q610.1 (G)
- net VCC: now also J10.16 (Pin_16), J10.2 (Pin_2), J12.10 (Pin_10), J12.14 (Pin_14), J12.2 (Pin_2), J12.6 (Pin_6), J13.16 (Pin_16), J13.2 (Pin_2), R356.1, R357.1, R358.1, R359.1, R360.1, R361.1, R362.1, R363.1, R364.1, R365.1, R366.1, R367.1, R368.1, R369.1, R370.1, R371.1, R372.1, R373.1, R374.1, R375.1, R376.1, R377.1, R378.1, R379.1, R380.1, R381.1, R382.1, R383.1, R384.1, R385.1, R386.1, R387.1, R390.1, R391.1, R392.1, R393.1, R394.1, R395.1, R396.1, R397.1, R398.1, R399.1, R400.1, R401.1, R402.1, R403.1, R404.1, R405.1, R406.1, R407.1, R408.1, R409.1, R412.1, R413.1, R414.1, R415.1, R416.1, R417.1, R418.1, R419.1, R420.1, R421.1, R422.1, R423.1, R424.1, R425.1, R426.1, R427.1, R428.1, R429.1, R430.1, R431.1, R432.1, R433.1, R434.1, R435.1, R436.1, R437.1, R438.1, R439.1, R440.1, R441.1, R442.1, R443.1, R444.1, R445.1, R446.1, R447.1, R448.1, R449.1, R450.1, R451.1, R452.1, R453.1, R454.1, R455.1, R456.1, R457.1, R458.1, R459.1, R460.1, R461.1, R462.1, R463.1, R464.1, R465.1, R466.1, R467.1, R468.1, R469.1, R470.1, R471.1, R472.1, R473.1, R474.1, R475.1, R476.1, R477.1, R478.1, R479.1, R480.1, R481.1, R482.1, R483.1, R484.1, R485.1, R486.1, R487.1, R488.1, R489.1, R490.1, R491.1, R492.1, R493.1, R494.1, R495.1, R496.1, R497.1, R498.1, R499.1, R500.1, R501.1, R502.1, R503.1, R504.1, R505.1, R506.1, R507.1, R508.1, R509.1, R510.1, R511.1, R512.1, R513.1, R514.1, R515.1, R516.1, R517.1, R518.1, R519.1, R520.1, R521.1, R522.1, R523.1, R524.1, R525.1, R526.1, R527.1, R528.1, R553.1, R554.1, R555.1, R556.1
- net XOR: now also R334.2, J13.6 (Pin_6)
- net bus out -> Main bus: now also Q614.1 (G), R442.2
- net rst: now also J10.8 (Pin_8), J14.13 (Pin_13)
- net at Q15.1 (G), Q22.1 (G), Q29.1 (G)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: now also D50.1, Q597.3 (D), R365.2, R366.2; no longer J1.15 (Pin_15), Q2.1 (G)
- net at J1.21 (Pin_21), Q8.1 (G): no longer Q62.1 (G)
- net at Q170.1 (G), Q284.1 (G), Q286.1 (G)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: now also R451.2, R452.2, R453.2
- net at Q1.3 (D), Q16.1 (G), Q19.1 (G)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: now also D64.1, Q596.1 (G), R356.2
- net at Q10.1 (G), Q63.1 (G), Q7.3 (D)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: now also D58.1, Q602.1 (G), R361.2
- net at Q12.1 (G), Q47.1 (G), Q5.3 (D)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: now also D60.1, Q600.1 (G), R378.2
- net at Q14.1 (G), Q26.1 (G), Q3.3 (D)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: now also D62.1, Q598.1 (G), R358.2
- net at Q40.1 (G), Q54.1 (G), Q58.1 (G)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: now also D53.1, Q600.3 (D), R371.2, R379.2; no longer J1.18 (Pin_18), Q5.1 (G)
- net at Q25.1 (G), Q42.1 (G), Q49.1 (G)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: now also D52.1, Q599.3 (D), R369.2, R370.2; no longer J1.17 (Pin_17), Q4.1 (G)
- net at Q332.1 (G), Q337.1 (G), Q342.1 (G)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: now also R445.2, R446.2, R447.2
- net at Q53.1 (G), Q59.1 (G): now also D54.1, Q601.3 (D), R372.2, R373.2; no longer J1.19 (Pin_19), Q6.1 (G)
- net at Q8.3 (D), Q9.1 (G), R8.2: now also D57.1, Q603.1 (G), R362.2
- net at Q570.3 (D): now also D42.1; no longer Q569.2 (S)
- net at Q17.1 (G), Q20.1 (G), Q24.1 (G)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: now also D49.1, Q596.3 (D), R363.2, R364.2; no longer J1.14 (Pin_14), Q1.1 (G)
- net at Q21.1 (G), Q27.1 (G), Q44.1 (G)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: now also D51.1, Q598.3 (D), R367.2, R368.2; no longer J1.16 (Pin_16), Q3.1 (G)
- net at J1.20 (Pin_20), Q7.1 (G): no longer Q57.1 (G)
- net at Q13.1 (G), Q4.3 (D), Q41.1 (G)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: now also D61.1, Q599.1 (G), R359.2
- net at Q11.1 (G), Q56.1 (G), Q6.3 (D)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: now also D59.1, Q601.1 (G), R360.2
- net at Q18.1 (G), Q2.3 (D), Q28.1 (G)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: now also D63.1, Q597.1 (G), R357.2
- net at Q72.2 (S), Q79.3 (D): now also Q73.2 (S)
- new net: D66.1, Q616.3 (D)
- new net: D56.1, Q603.3 (D), Q62.1 (G), R376.2, R377.2
- new net: D67.2, R497.2, R498.2
- new net: D72.1, Q622.3 (D)
- new net: D54.2, R471.2, R472.2
- new net: D49.2, R461.2, R462.2
- new net: C1.1, D40.1, Q604.3 (D), Q605.1 (G), R380.2, R381.2, R382.2, R383.2, R406.2, R407.2, R408.2, R409.2
- new net: D48.1, Q614.3 (D)
- new net: D80.1, Q630.3 (D)
- new net: D80.2, R523.2, R524.2
- new net: D71.2, R505.2, R506.2
- new net: D51.2, R465.2, R466.2
- new net: D61.2, R485.2, R486.2
- new net: Q607.3 (D), Q608.1 (G), R394.2, R395.2, R396.2, R397.2
- new net: D75.2, R513.2, R514.2
- new net: D79.2, R521.2, R522.2
- new net: D95.1, Q645.3 (D)
- new net: D64.2, R491.2, R492.2
- new net: D55.1, Q57.1 (G), Q602.3 (D), R374.2, R375.2
- new net: D82.1, Q632.3 (D)
- new net: D82.2, R527.2, R528.2
- new net: D79.1, Q629.3 (D)
- new net: D75.1, Q625.3 (D)
- new net: D65.2, R493.2, R494.2
- new net: C2.2, Q607.1 (G), R389.1, R411.1
- new net: D52.2, R467.2, R468.2
- new net: D50.2, R463.2, R464.2
- new net: D95.2, R553.2, R554.2
- new net: D63.2, R489.2, R490.2
- new net: J1.18 (Pin_18), Q5.1 (G)
- new net: D62.2, R487.2, R488.2
- new net: D41.1, Q569.3 (D)
- new net: J1.14 (Pin_14), Q1.1 (G)
- new net: J1.15 (Pin_15), Q2.1 (G)
- new net: J1.16 (Pin_16), Q3.1 (G)
- new net: J1.17 (Pin_17), Q4.1 (G)
- new net: J1.19 (Pin_19), Q6.1 (G)
- new net: D55.2, R473.2, R474.2
- new net: D56.2, R475.2, R476.2
- new net: D81.1, Q631.3 (D)
- new net: D77.2, R517.2, R518.2
- new net: D73.2, R509.2, R510.2
- new net: D68.2, R499.2, R500.2
- new net: Q606.3 (D), Q609.1 (G), R390.2, R391.2, R392.2, R393.2
- new net: D78.1, Q628.3 (D)
- new net: D78.2, R519.2, R520.2
- new net: D77.1, Q627.3 (D)
- new net: D43.2, R428.2, R429.2
- new net: D44.1, Q610.3 (D)
- new net: D48.2, R438.2, R439.2
- new net: D76.2, R515.2, R516.2
- new net: D53.2, R469.2, R470.2
- new net: D59.2, R481.2, R482.2
- new net: D76.1, Q626.3 (D)
- new net: D44.2, R430.2, R431.2
- new net: D72.2, R507.2, R508.2
- new net: D74.2, R511.2, R512.2
- new net: C1.2, Q606.1 (G), R388.1, R410.1
- new net: D40.2, R424.2, R425.2
- new net: D96.2, R555.2, R556.2
- new net: D58.2, R479.2, R480.2
- new net: C2.1, Q605.3 (D), R384.2, R385.2, R386.2, R387.2, R420.2, R421.2, R422.2, R423.2
- new net: D46.2, R434.2, R435.2
- new net: D81.2, R525.2, R526.2
- new net: D42.2, R426.2, R427.2
- new net: D67.1, Q617.3 (D)
- new net: D71.1, Q621.3 (D)
- new net: D70.2, R503.2, R504.2
- new net: D96.1, Q646.3 (D)
- new net: D70.1, Q620.3 (D)
- new net: D47.2, R436.2, R437.2
- new net: D45.1, Q611.3 (D)
- new net: D45.2, R432.2, R433.2
- new net: D66.2, R495.2, R496.2
- new net: D41.2, R335.2, R336.2
- new net: D65.1, Q615.3 (D)
- new net: D57.2, R477.2, R478.2
- new net: D69.2, R501.2, R502.2
- new net: D74.1, Q624.3 (D)
- new net: D69.1, Q619.3 (D)
- new net: D43.1, Q571.3 (D)
- new net: D68.1, Q618.3 (D)
- new net: D60.2, R483.2, R484.2
- new net: D46.1, Q612.3 (D)
- new net: D73.1, Q623.3 (D)
- new net: D47.1, Q613.3 (D)
- new net CLOCK: J10.6 (Pin_6), Q604.1 (G)
Other:
- note removed: "!clock"
- note removed: ""00001101" = 0x0D"
- note removed: ""00001110" = 0x0E"
- note removed: ""00001111" = 0x0F"
- note removed: "IGNORE"
- note removed: "Makes sure we dont read new instructions while a jump or read/write happens"
- note removed: "falure point (timing issue) (may need to change inputs for "read new instruction")"
- note removed: "falure point (timing issue) (may need to change resistor)"
- note removed: "nr 1"
- note removed: "nr 2"
- moved on the sheet: D1, D10, D11, D15, D16, D17, D18, D19, D2, D20, D21, D22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

Commit message: CONTROLLER UNIT V1.0 done?
JCL : exceed 2048 error
Parts:
- removed R380, R381, R382, R383, R384, R385, R386, R387, R390, R391, R392, R393, R394, R395, R396, R397, R398, R399, R400, R401, R402, R403, R404, R405, R406, R407, R408, R409, R412, R413, R414, R415, R416, R417, R418, R419, R420, R421, R422, R423: 10kΩ, PCM_JLCPCB:R_0402, symbol PCM_JLCPCB-Resistors:0402,20kΩ
- added H1, H25, H26, H27, H28, H29, H30, H31, H32: MountingHole, MountingHole:MountingHole_3.2mm_M3, symbol Mechanical:MountingHole
- added H10, H11, H12, H13, H14, H15, H16, H17, H18, H19, H2, H20, H21, H22, H23, H24, H3, H4, H5, H6, H7, H8, H9: MountingHole, MountingHole:MountingHole_2.2mm_M2, symbol Mechanical:MountingHole
- added R20, R21, R22, R74, R76, R77: R, Resistor_THT:R_Axial_DIN0207_L6.3mm_D2.5mm_P7.62mm_Horizontal, symbol Device:R
- C1, C2: now left out of the parts list
- R388, R389, R410, R411: footprint Resistor_THT:R_Axial_DIN0309_L9.0mm_D3.2mm_P12.70mm_Horizontal -> Resistor_THT:R_Axial_DIN0207_L6.3mm_D2.5mm_P7.62mm_Horizontal; now left out of the parts list
Connections:
- net A ->ALU A: now also J14.16 (Pin_16); no longer J14.2 (Pin_2)
- net A ->ALU B: now also J14.8 (Pin_8); no longer J14.10 (Pin_10)
- net ADD: now also J13.14 (Pin_14); no longer J13.4 (Pin_4)
- net ADR 0: now also J11.15 (Pin_15); no longer J11.1 (Pin_1)
- net ADR 1: now also J11.13 (Pin_13); no longer J11.3 (Pin_3)
- net ADR 10: now also J11.12 (Pin_12); no longer J11.6 (Pin_6)
- net ADR 11: now also J11.10 (Pin_10); no longer J11.8 (Pin_8)
- net ADR 12: now also J11.8 (Pin_8); no longer J11.10 (Pin_10)
- net ADR 13: now also J11.6 (Pin_6); no longer J11.12 (Pin_12)
- net ADR 14: now also J11.4 (Pin_4); no longer J11.14 (Pin_14)
- net ADR 15: now also J11.2 (Pin_2); no longer J11.16 (Pin_16)
- net ADR 2: now also J11.11 (Pin_11); no longer J11.5 (Pin_5)
- net ADR 3: now also J11.9 (Pin_9); no longer J11.7 (Pin_7)
- net ADR 4: now also J11.7 (Pin_7); no longer J11.9 (Pin_9)
- net ADR 5: now also J11.5 (Pin_5); no longer J11.11 (Pin_11)
- net ADR 6: now also J11.3 (Pin_3); no longer J11.13 (Pin_13)
- net ADR 7: now also J11.1 (Pin_1); no longer J11.15 (Pin_15)
- net ADR 8: now also J11.16 (Pin_16); no longer J11.2 (Pin_2)
- net ADR 9: now also J11.14 (Pin_14); no longer J11.4 (Pin_4)
- net ALU B = FF: now also J14.7 (Pin_7); no longer J14.9 (Pin_9)
- net ALU FLAG C: now also J13.5 (Pin_5); no longer J13.11 (Pin_11)
- net ALU FLAG N: now also J13.13 (Pin_13); no longer J13.3 (Pin_3)
- net ALU FLAG O: now also J13.7 (Pin_7); no longer J13.9 (Pin_9)
- net ALU FLAG U: now also J13.9 (Pin_9); no longer J13.7 (Pin_7)
- net ALU FLAG Z: now also J13.11 (Pin_11); no longer J13.5 (Pin_5)
- net AND: now also J13.6 (Pin_6); no longer J13.12 (Pin_12)
- net B ->ALU A: now also J14.14 (Pin_14); no longer J14.4 (Pin_4)
- net B ->ALU B: now also J14.6 (Pin_6); no longer J14.12 (Pin_12)
- net C ->ALU A: now also J14.12 (Pin_12); no longer J14.6 (Pin_6)
- net C ->ALU B: now also J14.4 (Pin_4); no longer J14.14 (Pin_14)
- net Carry in: now also J13.3 (Pin_3); no longer J13.13 (Pin_13)
- net D ->ALU A: now also J14.10 (Pin_10); no longer J14.8 (Pin_8)
- net D ->ALU B: now also J14.2 (Pin_2); no longer J14.16 (Pin_16)
- net Faling Edge: now also R74.2
- net GND: now also J12.10 (Pin_10), J12.14 (Pin_14), J12.2 (Pin_2), J12.6 (Pin_6), J14.1 (Pin_1); no longer J12.12 (Pin_12), J12.16 (Pin_16), J12.4 (Pin_4), J12.8 (Pin_8), J14.15 (Pin_15)
- net Main bus 0: now also J12.15 (Pin_15); no longer J12.1 (Pin_1)
- net Main bus 1: now also J12.13 (Pin_13); no longer J12.3 (Pin_3)
- net Main bus 2: now also J12.11 (Pin_11); no longer J12.5 (Pin_5)
- net Main bus 3: now also J12.9 (Pin_9); no longer J12.7 (Pin_7)
- net Main bus 4: now also J12.7 (Pin_7); no longer J12.9 (Pin_9)
- net Main bus 5: now also J12.5 (Pin_5); no longer J12.11 (Pin_11)
- net Main bus 6: now also J12.3 (Pin_3); no longer J12.13 (Pin_13)
- net Main bus 7: now also J12.1 (Pin_1); no longer J12.15 (Pin_15)
- net NOT: now also J13.10 (Pin_10); no longer J13.8 (Pin_8)
- net OR: now also J13.4 (Pin_4); no longer J13.14 (Pin_14)
- net READ A: now also J14.15 (Pin_15); no longer J14.1 (Pin_1)
- net READ B: now also J14.13 (Pin_13); no longer J14.3 (Pin_3)
- net READ C: now also J14.11 (Pin_11); no longer J14.5 (Pin_5)
- net READ D: now also J14.9 (Pin_9); no longer J14.7 (Pin_7)
- net RS: now also J13.8 (Pin_8); no longer J13.10 (Pin_10)
- net Rising Edge: now also J14.5 (Pin_5), R77.2; no longer J14.11 (Pin_11)
- net VCC: now also J12.12 (Pin_12), J12.16 (Pin_16), J12.4 (Pin_4), J12.8 (Pin_8), R20.1, R21.1, R22.1, R74.1, R76.1, R77.1; no longer J12.10 (Pin_10), J12.14 (Pin_14), J12.2 (Pin_2), J12.6 (Pin_6)
- net XOR: now also J13.12 (Pin_12); no longer J13.6 (Pin_6)
- net rst: now also J14.3 (Pin_3); no longer J14.13 (Pin_13)
- net at C1.1, D40.1, Q604.3 (D)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: now also R21.2
- net at Q607.3 (D), Q608.1 (G): now also R76.2
- net at Q606.3 (D), Q609.1 (G): now also R22.2
- net at C2.1, Q605.3 (D): now also R20.2
