File: PCB_S/Controller_Unit_V1.0/Controller_Unit_V1.0.kicad_sch (KiCad schematic)
At the start: 1247 parts, among them J1 Conn_01x21_Socket, J10 Conn_02x08_Odd_Even, J11 Conn_02x08_Odd_Even, J12 Conn_02x08_Odd_Even, J13 Conn_02x08_Odd_Even, J14 Conn_02x08_Odd_Even, J2 Conn_01x21_Socket, J3 Conn_01x21_Socket, J4 Conn_01x21_Socket, J5 Conn_01x21_Socket, J6 Conn_01x21_Socket, J7 Conn_01x01_Pin, J8 Conn_01x01_Pin, J9 Conn_01x01_Pin, Q1 2N7002, Q10 2N7002, Q100 2N7002, Q101 2N7002, Q102 2N7002, Q103 2N7002, Q104 2N7002, Q105 2N7002, Q106 2N7002, Q107 2N7002, Q108 2N7002, Q109 2N7002, Q11 2N7002, Q110 2N7002, Q111 2N7002, Q112 2N7002, Q113 2N7002, Q114 2N7002, Q115 2N7002, Q116 2N7002, Q117 2N7002, Q118 2N7002, Q119 2N7002, Q12 2N7002, Q120 2N7002, Q121 2N7002, Q122 2N7002, Q123 2N7002, Q124 2N7002, Q125 2N7002, Q126 2N7002, Q127 2N7002, Q128 2N7002, Q129 2N7002, Q13 2N7002, Q130 2N7002, Q131 2N7002, Q132 2N7002, Q133 2N7002, Q134 2N7002, Q136 2N7002, Q137 2N7002, Q138 2N7002, Q139 2N7002, Q14 2N7002, Q140 2N7002, Q141 2N7002, Q142 2N7002, Q143 2N7002, Q144 2N7002, Q145 2N7002, Q146 2N7002, Q147 2N7002, Q148 2N7002, Q149 2N7002, Q15 2N7002, Q150 2N7002, Q151 2N7002, Q152 2N7002, Q153 2N7002, Q154 2N7002, Q155 2N7002, Q156 2N7002, Q157 2N7002, Q158 2N7002, Q159 2N7002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

Commit message: ----
Parts:
- added C10, C11, C12, C13, C14, C15, C16, C17, C18, C3, C4, C5, C6, C7, C8, C9: 22uF, PCM_JLCPCB:C_0805, symbol PCM_JLCPCB-Capacitors:0805,22uF
Connections:
- net GND: now also C10.2, C11.2, C12.2, C13.2, C14.2, C15.2, C16.2, C17.2, C18.2, C3.2, C4.2, C5.2, C6.2, C7.2, C8.2, C9.2
- net VCC: now also C10.1, C11.1, C12.1, C13.1, C14.1, C15.1, C16.1, C17.1, C18.1, C3.1, C4.1, C5.1, C6.1, C7.1, C8.1, C9.1

Commit message: Controller unit v1.0 done & Level Shifter fpga v1.0 done
Parts:
- added C19, C20: C, Capacitor_THT:C_Radial_D16.0mm_H25.0mm_P7.50mm, symbol Device:C
Connections:
- net GND: now also C19.2, C20.2
- net VCC: now also C19.1, C20.1
