File: PCB_S/Controller_Unit_V1.0/Controller_Unit_V1.0.kicad_pcb (KiCad board)
At the start: 6 copper layers, 184.2 x 198.3 mm, 1264 parts, among them J1 Conn_01x21_Socket, J10 Conn_02x08_Odd_Even, J11 Conn_02x08_Odd_Even, J12 Conn_02x08_Odd_Even, J13 Conn_02x08_Odd_Even, J14 Conn_02x08_Odd_Even, J2 Conn_01x21_Socket, J3 Conn_01x21_Socket, J4 Conn_01x21_Socket, J5 Conn_01x21_Socket, J6 Conn_01x21_Socket, J7 Conn_01x01_Pin, J8 Conn_01x01_Pin, J9 Conn_01x01_Pin, Q1 2N7002, Q10 2N7002, Q100 2N7002, Q101 2N7002, Q102 2N7002, Q103 2N7002, Q104 2N7002, Q105 2N7002, Q106 2N7002, Q107 2N7002, Q108 2N7002, Q109 2N7002, Q11 2N7002, Q110 2N7002, Q111 2N7002, Q112 2N7002, Q113 2N7002, Q114 2N7002, Q115 2N7002, Q116 2N7002, Q117 2N7002, Q118 2N7002, Q119 2N7002, Q12 2N7002, Q120 2N7002, Q121 2N7002, Q122 2N7002, Q123 2N7002, Q124 2N7002, Q125 2N7002, Q126 2N7002, Q127 2N7002, Q128 2N7002, Q129 2N7002, Q13 2N7002, Q130 2N7002, Q131 2N7002, Q132 2N7002, Q133 2N7002, Q134 2N7002, Q136 2N7002, Q137 2N7002, Q138 2N7002, Q139 2N7002, Q14 2N7002, Q140 2N7002, Q141 2N7002, Q142 2N7002, Q143 2N7002, Q144 2N7002, Q145 2N7002, Q146 2N7002, Q147 2N7002, Q148 2N7002, Q149 2N7002, Q15 2N7002, Q150 2N7002, Q151 2N7002, Q152 2N7002, Q153 2N7002, Q154 2N7002, Q155 2N7002, Q156 2N7002, Q157 2N7002, Q158 2N7002, Q159 2N7002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

Commit message: CONTROLLER UNIT V1.0 done?
JCL : exceed 2048 error
Parts:
- removed R380, R381, R382, R383, R384, R385, R386, R387, R390, R391, R392, R393, R394, R395, R396, R397, R398, R399, R400, R401, R402, R403, R404, R405, R406, R407, R408, R409, R412, R413, R414, R415, R416, R417, R418, R419, R420, R421, R422, R423: 10kΩ, PCM_JLCPCB:R_0402
- added G***: LOGO, HVL_L:HVL_LOGO_15mm, F.Cu at (107.4, 280.8)
- added H1: MountingHole, MountingHole:MountingHole_3.2mm_M3, F.Cu at (110.0, 300.0)
- added H10: MountingHole, MountingHole:MountingHole_2.2mm_M2, F.Cu at (190.7, 218.6)
- added H11: MountingHole, MountingHole:MountingHole_2.2mm_M2, F.Cu at (132.3, 212.2)
- added H12: MountingHole, MountingHole:MountingHole_2.2mm_M2, F.Cu at (132.3, 218.6)
- added H13: MountingHole, MountingHole:MountingHole_2.2mm_M2, F.Cu at (190.7, 283.7)
- added H14: MountingHole, MountingHole:MountingHole_2.2mm_M2, F.Cu at (190.7, 290.1)
- added H15: MountingHole, MountingHole:MountingHole_2.2mm_M2, F.Cu at (132.3, 283.7)
- added H16: MountingHole, MountingHole:MountingHole_2.2mm_M2, F.Cu at (132.3, 290.1)
- added H17: MountingHole, MountingHole:MountingHole_2.2mm_M2, F.Cu at (190.7, 249.8)
- added H18: MountingHole, MountingHole:MountingHole_2.2mm_M2, F.Cu at (190.7, 256.2)
- added H19: MountingHole, MountingHole:MountingHole_2.2mm_M2, F.Cu at (132.3, 249.8)
- added H2: MountingHole, MountingHole:MountingHole_2.2mm_M2, F.Cu at (106.8, 337.0)
- added H20: MountingHole, MountingHole:MountingHole_2.2mm_M2, F.Cu at (132.3, 256.2)
- added H21: MountingHole, MountingHole:MountingHole_2.2mm_M2, F.Cu at (210.1, 249.8)
- added H22: MountingHole, MountingHole:MountingHole_2.2mm_M2, F.Cu at (210.1, 256.2)
- added H23: MountingHole, MountingHole:MountingHole_2.2mm_M2, F.Cu at (268.5, 256.2)
- added H24: MountingHole, MountingHole:MountingHole_2.2mm_M2, F.Cu at (268.5, 249.8)
- added H25: MountingHole, MountingHole:MountingHole_3.2mm_M3, F.Cu at (103.5, 203.5)
- added H26: MountingHole, MountingHole:MountingHole_3.2mm_M3, F.Cu at (322.4, 203.5)
- added H27: MountingHole, MountingHole:MountingHole_3.2mm_M3, F.Cu at (322.4, 396.5)
- added H28: MountingHole, MountingHole:MountingHole_3.2mm_M3, F.Cu at (103.5, 396.4)
- added H29: MountingHole, MountingHole:MountingHole_3.2mm_M3, F.Cu at (200.0, 252.9)
- added H3: MountingHole, MountingHole:MountingHole_2.2mm_M2, F.Cu at (113.2, 395.4)
- added H30: MountingHole, MountingHole:MountingHole_3.2mm_M3, F.Cu at (214.3, 309.1)
- added H31: MountingHole, MountingHole:MountingHole_3.2mm_M3, F.Cu at (310.0, 290.0)
- added H32: MountingHole, MountingHole:MountingHole_3.2mm_M3, F.Cu at (200.7, 215.3)
- added H4: MountingHole, MountingHole:MountingHole_2.2mm_M2, F.Cu at (113.2, 337.0)
- added H5: MountingHole, MountingHole:MountingHole_2.2mm_M2, F.Cu at (268.5, 212.2)
- added H6: MountingHole, MountingHole:MountingHole_2.2mm_M2, F.Cu at (268.5, 218.6)
- added H7: MountingHole, MountingHole:MountingHole_2.2mm_M2, F.Cu at (210.1, 212.2)
- added H8: MountingHole, MountingHole:MountingHole_2.2mm_M2, F.Cu at (210.1, 218.6)
- added H9: MountingHole, MountingHole:MountingHole_2.2mm_M2, F.Cu at (190.6, 212.1)
- added R20: R, Resistor_THT:R_Axial_DIN0207_L6.3mm_D2.5mm_P7.62mm_Horizontal, F.Cu at (116.8, 267.0)
- added R21: R, Resistor_THT:R_Axial_DIN0207_L6.3mm_D2.5mm_P7.62mm_Horizontal, F.Cu at (145.1, 267.0)
- added R22: R, Resistor_THT:R_Axial_DIN0207_L6.3mm_D2.5mm_P7.62mm_Horizontal, F.Cu at (145.1, 276.0)
- added R74: R, Resistor_THT:R_Axial_DIN0207_L6.3mm_D2.5mm_P7.62mm_Horizontal, F.Cu at (145.1, 279.0)
- added R76: R, Resistor_THT:R_Axial_DIN0207_L6.3mm_D2.5mm_P7.62mm_Horizontal, F.Cu at (116.8, 276.0)
- added R77: R, Resistor_THT:R_Axial_DIN0207_L6.3mm_D2.5mm_P7.62mm_Horizontal, F.Cu at (116.8, 279.0)
- R388, R389, R410, R411: footprint Resistor_THT:R_Axial_DIN0309_L9.0mm_D3.2mm_P12.70mm_Horizontal -> Resistor_THT:R_Axial_DIN0207_L6.3mm_D2.5mm_P7.62mm_Horizontal
- moved Q110 355.3 mm to (208.2, 340.1), turned to -90 degrees
- moved J13 343.4 mm to (313.3, 388.2), turned to 180 degrees
- moved R440 325.8 mm to (154.8, 346.0), turned to 180 degrees
- moved Q516 324.6 mm to (281.9, 309.4)
- moved Q595 323.8 mm to (133.3, 344.5)
- moved R439 321.7 mm to (145.4, 339.1)
- moved Q568 320.2 mm to (282.3, 300.8), turned to -90 degrees
- moved Q515 320.0 mm to (137.8, 344.5)
- moved R443 319.3 mm to (154.8, 345.0), turned to 180 degrees
- moved R346 316.7 mm to (154.8, 343.0), turned to 180 degrees
- moved R444 316.5 mm to (154.8, 344.0), turned to 180 degrees
- moved R343 314.9 mm to (285.2, 315.2)
- moved R448 314.3 mm to (129.2, 346.1), turned to 180 degrees
- moved R342 314.1 mm to (283.2, 313.2), turned to 180 degrees
- moved R344 312.3 mm to (285.2, 314.2)
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Connections:
- J11 pad 1: ADR 0 -> ADR 7
- J11 pad 10: ADR 12 -> ADR 11
- J11 pad 11: ADR 5 -> ADR 2
- J11 pad 12: ADR 13 -> ADR 10
- J11 pad 13: ADR 6 -> ADR 1
- J11 pad 14: ADR 14 -> ADR 9
- J11 pad 15: ADR 7 -> ADR 0
- J11 pad 16: ADR 15 -> ADR 8
- J11 pad 2: ADR 8 -> ADR 15
- J11 pad 3: ADR 1 -> ADR 6
- J11 pad 4: ADR 9 -> ADR 14
- J11 pad 5: ADR 2 -> ADR 5
- J11 pad 6: ADR 10 -> ADR 13
- J11 pad 7: ADR 3 -> ADR 4
- J11 pad 8: ADR 11 -> ADR 12
- J11 pad 9: ADR 4 -> ADR 3
- J12 pad 1: Main bus 0 -> Main bus 7
- J12 pad 10: VCC -> GND
- J12 pad 11: Main bus 5 -> Main bus 2
- J12 pad 12: GND -> VCC
- J12 pad 13: Main bus 6 -> Main bus 1
- J12 pad 14: VCC -> GND
- J12 pad 15: Main bus 7 -> Main bus 0
- J12 pad 16: GND -> VCC
- J12 pad 2: VCC -> GND
- J12 pad 3: Main bus 1 -> Main bus 6
- J12 pad 4: GND -> VCC
- J12 pad 5: Main bus 2 -> Main bus 5
- J12 pad 6: VCC -> GND
- J12 pad 7: Main bus 3 -> Main bus 4
- J12 pad 8: GND -> VCC
- J12 pad 9: Main bus 4 -> Main bus 3
- J13 pad 10: RS -> NOT
- J13 pad 11: ALU FLAG C -> ALU FLAG Z
- J13 pad 12: AND -> XOR
- J13 pad 13: Carry in -> ALU FLAG N
- J13 pad 14: OR -> ADD
- J13 pad 3: ALU FLAG N -> Carry in
- J13 pad 4: ADD -> OR
- J13 pad 5: ALU FLAG Z -> ALU FLAG C
- J13 pad 6: XOR -> AND
- J13 pad 7: ALU FLAG U -> ALU FLAG O
- J13 pad 8: NOT -> RS
- J13 pad 9: ALU FLAG O -> ALU FLAG U
- J14 pad 1: READ A -> GND
- J14 pad 10: A ->ALU B -> D ->ALU A
- J14 pad 11: Rising Edge -> READ C
- J14 pad 12: B ->ALU B -> C ->ALU A
- J14 pad 13: rst -> READ B
- J14 pad 14: C ->ALU B -> B ->ALU A
- J14 pad 15: GND -> READ A
- J14 pad 16: D ->ALU B -> A ->ALU A
- J14 pad 2: A ->ALU A -> D ->ALU B
- J14 pad 3: READ B -> rst
- J14 pad 4: B ->ALU A -> C ->ALU B
- J14 pad 5: READ C -> Rising Edge
- J14 pad 6: C ->ALU A -> B ->ALU B
- J14 pad 7: READ D -> ALU B = FF
- J14 pad 8: D ->ALU A -> A ->ALU B
- J14 pad 9: ALU B = FF -> READ D
Routing:
- net GND: track 578.0 -> 2020.1 mm, vias 83 -> 154
- net VCC: track 486.7 -> 1180.5 mm, vias 81 -> 115
- net rst: track 0.00 -> 557.0 mm, vias 0 -> 6
- net Buss1: track 0.00 -> 413.1 mm, vias 0 -> 4
- net Buss0: track 0.00 -> 413.0 mm, vias 0 -> 4
- net Buss2: track 0.00 -> 412.2 mm, vias 0 -> 4
- net Buss3: track 0.00 -> 410.6 mm, vias 0 -> 4
- net Buss4: track 0.00 -> 408.5 mm, vias 0 -> 4
- net Buss5: track 0.00 -> 407.0 mm, vias 0 -> 4
- net Buss6: track 0.00 -> 406.8 mm, vias 0 -> 4
- net Buss7: track 0.00 -> 404.3 mm, vias 0 -> 4
- net bus out -> Main bus: track 0.00 -> 382.8 mm, vias 0 -> 11
- net TIME STEP 0: track 0.00 -> 363.2 mm, vias 0 -> 3
- net Store Address ++: track 0.00 -> 360.8 mm, vias 0 -> 20
- net Read From stored Address: track 9.51 -> 345.6 mm, vias 0 -> 18
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Other:
- board size 184.2 x 198.3 mm -> 225.9 x 200 mm
- board text added: "+ - + - + - + -"
- board text added: "+ - clk rst - r/w - +"
- board text added: "+ ADD XOR NOT RS AND OR +"
- board text added: "- N Z U O Co Ci -"
- board text added: "0 1 2 3 4 5 6 7"
- board text added: "15 14 13 12 11 10 9 8"
- board text added: "7 6 5 4 3 2 1 0"
- board text added: "AA"
- board text added: "AB"
- board text added: "ADC"
- board text added: "ADD"
- board text added: "ADR"
- board text added: "ADR HH"
- board text added: "ADR LL"
- board text added: "ALU_ A->A B->A C->A D->A A->B B->B C->B D->B"
- board text added: "AND"
- board text added: "BA"
- board text added: "BB"
- board text added: "BNC"
- board text added: "BNO"
- board text added: "BNU"
- board text added: "BNZ"
- board text added: "BOC"
- board text added: "BON"
- board text added: "BOO"
- board text added: "BOP"
- board text added: "BOU"
- board text added: "BOZ"
- board text added: "BUS BUFFER"
- board text added: "CA"
- board text added: "CB"
- board text added: "CLEAR"
- board text added: "CLOCK RISING EDGE FALING EDGE"
- board text added: "CPU CONTROLL UNIT V1.0"
- board text added: "CPU FLAG AND TIMING"
- board text added: "DA"
- board text added: "DATA"
- board text added: "DB"
- board text added: "DEC"
- board text added: "INC"
- board text added: "INS REGISTER"
- board text added: "INSTRUCTION DECODING"
- board text added: "JMP"
- board text added: "LOAD"
- board text added: "MAIN BUS"
- board text added: "MEMORY INCRIMENTER"
- board text added: "MOV"
- board text added: "MSB"
- board text added: "NEXT ADR SEL MUX"
- board text added: "NOT"
- board text added: "NOW ADR SEL MUX"
- board text added: "OR"
- board text added: "RA"
- board text added: "RA RB RC RD ABF RE rst -"
- board text added: "RB"
- board text added: "RC"
- board text added: "RD"
- board text added: "REG READ"
- board text added: "RS"
- board text added: "SJ"
- board text added: "STORE"
- board text added: "TEMP ADR HH"
- board text added: "TEMP ADR LL"
- board text added: "TO ALU A"
- board text added: "TO ALU B"
- board text added: "XOR"
