File: PCB_S/Controller_Unit_V1.0/Controller_Unit_V1.0.kicad_pcb (KiCad board)
At the start: 6 copper layers, 225.9 x 200 mm, 1263 parts, among them J1 Conn_01x21_Socket, J10 Conn_02x08_Odd_Even, J11 Conn_02x08_Odd_Even, J12 Conn_02x08_Odd_Even, J13 Conn_02x08_Odd_Even, J14 Conn_02x08_Odd_Even, J2 Conn_01x21_Socket, J3 Conn_01x21_Socket, J4 Conn_01x21_Socket, J5 Conn_01x21_Socket, J6 Conn_01x21_Socket, J7 Conn_01x01_Pin, J8 Conn_01x01_Pin, J9 Conn_01x01_Pin, Q1 2N7002, Q10 2N7002, Q100 2N7002, Q101 2N7002, Q102 2N7002, Q103 2N7002, Q104 2N7002, Q105 2N7002, Q106 2N7002, Q107 2N7002, Q108 2N7002, Q109 2N7002, Q11 2N7002, Q110 2N7002, Q111 2N7002, Q112 2N7002, Q113 2N7002, Q114 2N7002, Q115 2N7002, Q116 2N7002, Q117 2N7002, Q118 2N7002, Q119 2N7002, Q12 2N7002, Q120 2N7002, Q121 2N7002, Q122 2N7002, Q123 2N7002, Q124 2N7002, Q125 2N7002, Q126 2N7002, Q127 2N7002, Q128 2N7002, Q129 2N7002, Q13 2N7002, Q130 2N7002, Q131 2N7002, Q132 2N7002, Q133 2N7002, Q134 2N7002, Q136 2N7002, Q137 2N7002, Q138 2N7002, Q139 2N7002, Q14 2N7002, Q140 2N7002, Q141 2N7002, Q142 2N7002, Q143 2N7002, Q144 2N7002, Q145 2N7002, Q146 2N7002, Q147 2N7002, Q148 2N7002, Q149 2N7002, Q15 2N7002, Q150 2N7002, Q151 2N7002, Q152 2N7002, Q153 2N7002, Q154 2N7002, Q155 2N7002, Q156 2N7002, Q157 2N7002, Q158 2N7002, Q159 2N7002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

Commit message: Controller unit v1.0 done & Level Shifter fpga v1.0 done
Parts:
- added C10: 22uF, PCM_JLCPCB:C_0805, F.Cu at (164.4, 134.1)
- added C11: 22uF, PCM_JLCPCB:C_0805, F.Cu at (99.2, 159.3)
- added C12: 22uF, PCM_JLCPCB:C_0805, F.Cu at (102.2, 159.3)
- added C13: 22uF, PCM_JLCPCB:C_0805, F.Cu at (105.3, 159.3)
- added C14: 22uF, PCM_JLCPCB:C_0805, F.Cu at (108.3, 159.3)
- added C15: 22uF, PCM_JLCPCB:C_0805, F.Cu at (37.6, 60.7)
- added C16: 22uF, PCM_JLCPCB:C_0805, F.Cu at (37.6, 63.8)
- added C17: 22uF, PCM_JLCPCB:C_0805, F.Cu at (37.6, 66.8)
- added C18: 22uF, PCM_JLCPCB:C_0805, F.Cu at (37.6, 69.8)
- added C19: C, Capacitor_THT:C_Radial_D16.0mm_H25.0mm_P7.50mm, F.Cu at (216.2, 86.0)
- added C20: C, Capacitor_THT:C_Radial_D16.0mm_H25.0mm_P7.50mm, F.Cu at (216.2, 102.5)
- added C3: 22uF, PCM_JLCPCB:C_0805, F.Cu at (193.9, 109.1)
- added C4: 22uF, PCM_JLCPCB:C_0805, F.Cu at (196.9, 109.1)
- added C5: 22uF, PCM_JLCPCB:C_0805, F.Cu at (200.0, 109.1)
- added C6: 22uF, PCM_JLCPCB:C_0805, F.Cu at (203.1, 109.1)
- added C7: 22uF, PCM_JLCPCB:C_0805, F.Cu at (155.3, 134.1)
- added C8: 22uF, PCM_JLCPCB:C_0805, F.Cu at (158.3, 134.1)
- added C9: 22uF, PCM_JLCPCB:C_0805, F.Cu at (161.4, 134.1)
- added H3: MountingHole, MountingHole:MountingHole_2.2mm_M2, F.Cu at (26.8, 198.4)
- moved J1 212.6 mm to (30.0, 194.6)
- moved H2 212.6 mm to (26.8, 140.0)
- moved H4 212.6 mm to (33.2, 140.0)
- moved H3 212.6 mm to (33.2, 198.4)
- moved D49 197.0 mm to (48.9, 210.1)
- moved D54 197.0 mm to (48.9, 188.1)
- moved D59 197.0 mm to (39.4, 188.1)
- moved D64 197.0 mm to (39.4, 210.1)
- moved H14 197.0 mm to (110.7, 110.1)
- moved H16 197.0 mm to (52.3, 110.1)
- moved H30 197.0 mm to (134.3, 129.1)
- moved Q1 197.0 mm to (43.2, 211.1)
- moved Q100 197.0 mm to (124.2, 150.1)
- moved Q101 197.0 mm to (128.2, 150.1)
- moved Q102 197.0 mm to (132.2, 150.1)
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Routing:
- net VCC: track 1180.5 -> 1227.3 mm, vias 115 -> 119
- net GND: track 2020.1 -> 2066.0 mm, vias 154 -> 158
- net Net-(J1-Pin_17): track 39.3 -> 56.4 mm
- net Read New Instruction: track 75.6 -> 58.6 mm
- net Buss7: track 404.3 -> 387.3 mm
- net Net-(J1-Pin_18): track 37.5 -> 54.5 mm
- net Net-(J1-Pin_16): track 41.2 -> 58.2 mm
- net Faling Edge: track 292.8 -> 275.8 mm
- net Buss1: track 413.1 -> 396.1 mm
- net Net-(J1-Pin_15): track 43.0 -> 60.0 mm
- net Net-(J1-Pin_21): track 31.8 -> 48.8 mm
- net Net-(J1-Pin_20): track 33.7 -> 50.7 mm
- net Net-(J1-Pin_19): track 35.6 -> 52.6 mm
- net Buss6: track 406.8 -> 389.8 mm
- net Buss4: track 408.5 -> 391.5 mm
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Other:
- board text added: "+"
- board text added: "++"
- board text added: "-"
- board text added: "0"
- board text added: "0x02"
- board text added: "0x03"
- board text added: "0x04"
- board text added: "0x05"
- board text added: "0x06"
- board text added: "0x07"
- board text added: "0x08"
- board text added: "0x09"
- board text added: "0x0A"
- board text added: "0x0B"
- board text added: "0x0C"
- board text added: "0x10-0x13"
- board text added: "0x14 - 0x17"
- board text added: "0x18 - 0x1B"
- board text added: "0x1C - 0x1F"
- board text added: "0x20 - 0x23"
- board text added: "0x24 - 0x27"
- board text added: "0x28 - 0x2B"
- board text added: "0x30 - 0x3F"
- board text added: "0x40 - 0x4F"
- board text added: "0x50 - 0x5F"
- board text added: "0x60 - 0x6F"
- board text added: "0x70 - 0x7F"
- board text added: "0x80 - 0x8F"
- board text added: "1"
- board text added: "10"
- board text added: "11"
- board text added: "12"
- board text added: "13"
- board text added: "14"
- board text added: "15"
- board text added: "2"
- board text added: "3"
- board text added: "4"
- board text added: "5"
- board text added: "6"
- board text added: "7"
- board text added: "8"
- board text added: "9"
- board text added: "ALUA"
- board text added: "ALUB"
- board text added: "BO->MB"
- board text added: "FLAG"
- board text added: "MB->BO"
- board text added: "NEW INS"
- board text added: "RW INS"
- board text added: "Read"
- board text added: "STEP 0"
- board text added: "Stored"
- board text added: "com jump"
