File: PCB_S/Whole_CPU_V1.0/Whole_CPU_V1.0.kicad_sch (KiCad schematic)
At the start: 2108 parts, among them J1 Conn_01x21_Socket, J10 Conn_02x08_Odd_Even, J11 Conn_02x08_Odd_Even, J12 Conn_02x08_Odd_Even, J13 Conn_02x08_Odd_Even, J14 Conn_02x08_Odd_Even, J15 Conn_02x08_Odd_Even, J16 Conn_02x08_Odd_Even, J17 Conn_01x02_Pin, J18 Conn_01x02_Pin, J19 Conn_01x02_Pin, J2 Conn_01x21_Socket, J20 Conn_02x08_Odd_Even, J21 Conn_01x21_Socket, J22 Conn_01x21_Socket, J23 Conn_01x21_Socket, J24 Conn_01x21_Socket, J25 Conn_02x08_Odd_Even, J26 Conn_02x08_Odd_Even, J27 Conn_01x02_Pin, J28 Conn_01x02_Pin, J29 Conn_02x08_Odd_Even, J3 Conn_01x21_Socket, J4 Conn_01x21_Socket, J5 Conn_01x21_Socket, J52 Conn_02x08_Odd_Even, J6 Conn_01x21_Socket, J7 Conn_01x01_Pin, J8 Conn_01x01_Pin, J9 Conn_01x01_Pin, Q1 2N7002, Q10 2N7002, Q100 2N7002, Q1000 2N7002, Q1001 2N7002, Q1002 2N7002, Q1003 2N7002, Q1004 2N7002, Q1005 2N7002, Q1006 2N7002, Q1007 2N7002, Q1008 2N7002, Q1009 2N7002, Q101 2N7002, Q1010 2N7002, Q1011 2N7002, Q1012 2N7002, Q1013 2N7002, Q1014 2N7002, Q1015 2N7002, Q1016 2N7002, Q1017 2N7002, Q1018 2N7002, Q1019 2N7002, Q102 2N7002, Q1020 2N7002, Q1021 2N7002, Q1022 2N7002, Q1023 2N7002, Q1024 2N7002, Q1025 2N7002, Q1026 2N7002, Q1027 2N7002, Q1028 2N7002, Q1029 2N7002, Q103 2N7002, Q1030 2N7002, Q1031 2N7002, Q1032 2N7002, Q1033 2N7002, Q1034 2N7002, Q1035 2N7002, Q1036 2N7002, Q1037 2N7002, Q1038 2N7002, Q1039 2N7002, Q104 2N7002, Q1040 2N7002, Q1041 2N7002, Q1042 2N7002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

Commit message: almost done
Parts:
- removed C19, C20: C, Capacitor_THT:C_Radial_D16.0mm_H25.0mm_P7.50mm, symbol Device:C
- removed H35, H53, H54, H55: MountingHole, MountingHole:MountingHole_3.2mm_M3, symbol Mechanical:MountingHole
- removed J12, J13, J14, J15, J16, J20, J25, J26, J29, J52: Conn_02x08_Odd_Even, Connector_PinSocket_2.54mm:PinSocket_2x08_P2.54mm_Vertical, symbol Connector_Generic:Conn_02x08_Odd_Even
- added D12, D13, D132, D133, D134, D135, D136, D137, D138, D139, D14, D140, D141, D142, D143, D144, D145, D146, D147, D83, D84, D85, D86, D87: Red, PCM_JLCPCB:D_0603, symbol PCM_JLCPCB-Diodes:LED,0603,Red
- added Q135, Q36, Q37, Q38, Q39, Q633, Q634, Q635, Q793, Q794, Q795, Q796, Q797, Q798, Q799, Q800, Q801, Q802, Q803, Q804, Q805, Q806, Q807, Q808: 2N7002, Package_TO_SOT_SMD:SOT-23, symbol Transistor_FET:2N7002
- added R380, R381, R382, R383, R384, R385, R386, R387, R390, R391, R392, R393, R394, R75, R760, R761, R762, R763, R764, R765, R766, R767, R768, R769, R770, R771, R772, R773, R774, R775, R776, R777, R778, R779, R78, R780, R781, R782, R783, R784, R785, R786, R787, R788, R789, R79, R790, R791: 10kΩ, PCM_JLCPCB:R_0402, symbol PCM_JLCPCB-Resistors:0402,20kΩ
Connections:
- net ALU B -> FF is gone; now on net ALU B = FF: Q688.1 (G), Q689.1 (G), Q699.1 (G), Q708.1 (G), Q709.1 (G), Q710.1 (G), Q720.1 (G), Q729.1 (G)
- net C_in is gone; now on net Carry in: Q912.1 (G)
- net C_out is gone; now on net ALU FLAG C: Q1115.3 (D), Q905.1 (G), R742.2
- net Main bus 7 is gone; now on net ALU FLAG N: Q538.1 (G), Q563.3 (D)
- net N is gone; now on net ALU FLAG N: Q1023.1 (G), Q1024.1 (G), Q1087.3 (D), Q901.1 (G), Q917.1 (G), Q919.1 (G), R713.2
- net O is gone; now on net ALU FLAG O: Q904.1 (G), Q908.3 (D), R570.2
- net RST is gone; now on net rst: J21.3 (Pin_3), J22.3 (Pin_3), J23.3 (Pin_3), J24.3 (Pin_3)
- net Rising_Edge is gone; now on net Rising Edge: J21.5 (Pin_5), J22.5 (Pin_5), J23.5 (Pin_5), J24.5 (Pin_5)
- net U is gone; now on net ALU FLAG U: Q1116.3 (D), Q903.1 (G), R744.2
- net Z is gone; now on net ALU FLAG Z: Q1006.3 (D), Q1009.3 (D), Q1012.3 (D), Q1023.3 (D), Q902.1 (G), Q979.3 (D), Q982.3 (D), Q993.3 (D), Q996.3 (D), R621.2
- net A ->ALU A: now also Q654.1 (G), Q655.1 (G), Q656.1 (G), Q657.1 (G), Q658.1 (G), Q659.1 (G), Q660.1 (G), Q661.1 (G), Q662.1 (G)
- net A ->ALU B: now also Q671.1 (G), Q672.1 (G), Q673.1 (G), Q674.1 (G), Q675.1 (G), Q676.1 (G), Q677.1 (G), Q678.1 (G), Q679.1 (G)
- net ADD: now also Q1119.1 (G), Q1121.1 (G), Q1126.1 (G), Q1138.1 (G), Q1150.1 (G), Q1162.1 (G), Q1174.1 (G), Q1186.1 (G), Q1198.1 (G), Q1210.1 (G), Q1220.1 (G)
- net ADR 0: now also Q800.1 (G)
- net ADR 1: now also Q799.1 (G)
- net ADR 10: now also Q633.1 (G)
- net ADR 11: now also Q135.1 (G)
- net ADR 12: now also Q39.1 (G)
- net ADR 13: now also Q38.1 (G)
- net ADR 14: now also Q37.1 (G)
- net ADR 15: now also Q36.1 (G)
- net ADR 2: now also Q798.1 (G)
- net ADR 3: now also Q797.1 (G)
- net ADR 4: now also Q796.1 (G)
- net ADR 5: now also Q795.1 (G)
- net ADR 6: now also Q794.1 (G)
- net ADR 7: now also Q793.1 (G)
- net ADR 8: now also Q635.1 (G)
- net ADR 9: now also Q634.1 (G)
- net ALU FLAG N: now also J21.13 (Pin_13), J22.13 (Pin_13), J23.13 (Pin_13), J24.13 (Pin_13)
- net AND: now also Q1110.1 (G), Q1114.1 (G), Q1130.1 (G), Q1142.1 (G), Q1154.1 (G), Q1166.1 (G), Q1178.1 (G), Q1190.1 (G), Q1202.1 (G), Q1214.1 (G)
- net B ->ALU A: now also Q690.1 (G), Q691.1 (G), Q692.1 (G), Q693.1 (G), Q694.1 (G), Q695.1 (G), Q696.1 (G), Q697.1 (G), Q698.1 (G)
- net B ->ALU B: now also Q711.1 (G), Q712.1 (G), Q713.1 (G), Q714.1 (G), Q715.1 (G), Q716.1 (G), Q717.1 (G), Q718.1 (G), Q719.1 (G)
- net Buss0: now also Q808.1 (G)
- net Buss1: now also Q807.1 (G)
- net Buss2: now also Q806.1 (G)
- net Buss3: now also Q805.1 (G)
- net Buss4: now also Q804.1 (G)
- net Buss5: now also Q803.1 (G)
- net Buss6: now also Q802.1 (G)
- net Buss7: now also Q801.1 (G)
- net C ->ALU A: now also Q730.1 (G), Q731.1 (G), Q732.1 (G), Q733.1 (G), Q734.1 (G), Q735.1 (G), Q736.1 (G), Q737.1 (G), Q738.1 (G)
- net C ->ALU B: now also Q747.1 (G), Q748.1 (G), Q749.1 (G), Q750.1 (G), Q751.1 (G), Q752.1 (G), Q753.1 (G), Q754.1 (G), Q755.1 (G)
- net D ->ALU A: now also Q764.1 (G), Q765.1 (G), Q766.1 (G), Q767.1 (G), Q768.1 (G), Q769.1 (G), Q770.1 (G), Q771.1 (G), Q772.1 (G)
- net D ->ALU B: now also Q781.1 (G), Q782.1 (G), Q783.1 (G), Q784.1 (G), Q785.1 (G), Q786.1 (G), Q787.1 (G), Q788.1 (G), Q789.1 (G)
- net GND: now also Q135.2 (S), Q36.2 (S), Q37.2 (S), Q38.2 (S), Q39.2 (S), Q633.2 (S), Q634.2 (S), Q635.2 (S), Q793.2 (S), Q794.2 (S), Q795.2 (S), Q796.2 (S), Q797.2 (S), Q798.2 (S), Q799.2 (S), Q800.2 (S), Q801.2 (S), Q802.2 (S), Q803.2 (S), Q804.2 (S), Q805.2 (S), Q806.2 (S), Q807.2 (S), Q808.2 (S)
- net Main bus 0: now also J21.6 (Pin_6), J22.6 (Pin_6), J23.6 (Pin_6), J24.6 (Pin_6), Q1045.3 (D), Q979.1 (G), Q980.1 (G), R680.2
- net Main bus 1: now also J21.7 (Pin_7), J22.7 (Pin_7), J23.7 (Pin_7), J24.7 (Pin_7), Q1055.3 (D), Q982.1 (G), Q983.1 (G), R688.2
- net Main bus 2: now also J21.8 (Pin_8), J22.8 (Pin_8), J23.8 (Pin_8), J24.8 (Pin_8), Q1058.3 (D), Q993.1 (G), Q994.1 (G), R690.2
- net Main bus 3: now also J21.9 (Pin_9), J22.9 (Pin_9), J23.9 (Pin_9), J24.9 (Pin_9), Q1060.3 (D), Q996.1 (G), Q997.1 (G), R691.2
- net Main bus 4: now also J21.10 (Pin_10), J22.10 (Pin_10), J23.10 (Pin_10), J24.10 (Pin_10), Q1006.1 (G), Q1007.1 (G), Q1071.3 (D), R698.2
- net Main bus 5: now also J21.11 (Pin_11), J22.11 (Pin_11), J23.11 (Pin_11), J24.11 (Pin_11), Q1009.1 (G), Q1010.1 (G), Q1074.3 (D), R701.2
- net Main bus 6: now also J21.12 (Pin_12), J22.12 (Pin_12), J23.12 (Pin_12), J24.12 (Pin_12), Q1012.1 (G), Q1013.1 (G), Q1084.3 (D), R710.2
- net NOT: now also Q1113.1 (G), Q1122.1 (G), Q1134.1 (G), Q1146.1 (G), Q1158.1 (G), Q1170.1 (G), Q1182.1 (G), Q1194.1 (G), Q1206.1 (G), Q1216.1 (G)
- net OR: now also Q1108.1 (G), Q1112.1 (G), Q1128.1 (G), Q1140.1 (G), Q1152.1 (G), Q1164.1 (G), Q1176.1 (G), Q1188.1 (G), Q1200.1 (G), Q1212.1 (G)
- net READ A: now also J21.4 (Pin_4)
- net READ B: now also J22.4 (Pin_4)
- net READ C: now also J23.4 (Pin_4)
- net READ D: now also J24.4 (Pin_4)
- net RS: now also Q1111.1 (G), Q1118.1 (G), Q1124.1 (G), Q1132.1 (G), Q1144.1 (G), Q1156.1 (G), Q1168.1 (G), Q1180.1 (G), Q1192.1 (G), Q1204.1 (G)
- net VCC: now also R380.1, R381.1, R382.1, R383.1, R384.1, R385.1, R386.1, R387.1, R390.1, R391.1, R392.1, R393.1, R394.1, R75.1, R760.1, R761.1, R762.1, R763.1, R764.1, R765.1, R766.1, R767.1, R768.1, R769.1, R770.1, R771.1, R772.1, R773.1, R774.1, R775.1, R776.1, R777.1, R778.1, R779.1, R78.1, R780.1, R781.1, R782.1, R783.1, R784.1, R785.1, R786.1, R787.1, R788.1, R789.1, R79.1, R790.1, R791.1
- net XOR: now also Q1117.1 (G), Q1125.1 (G), Q1136.1 (G), Q1148.1 (G), Q1160.1 (G), Q1172.1 (G), Q1184.1 (G), Q1196.1 (G), Q1208.1 (G), Q1218.1 (G)
- net AA7: now reaches Q1047.1 (G), Q1101.1 (G), Q1103.1 (G), Q1107.1 (G), Q906.1 (G), Q928.1 (G)
- net AA7: now also Q643.3 (D), R404.2
- net AA0: now reaches Q1062.1 (G), Q922.1 (G), Q924.1 (G), Q934.1 (G)
- net AA0: now also Q636.3 (D), R397.2
- net AA4: now reaches Q1005.1 (G), Q1027.1 (G), Q1029.1 (G), Q1089.1 (G)
- net AA4: now also Q640.3 (D), R401.2
- net AA3: now reaches Q639.3 (D), R400.2
- net AA3: now also Q1001.1 (G), Q1086.1 (G), Q981.1 (G), Q999.1 (G)
- net AB2: now reaches Q1143.1 (G), Q935.1 (G), Q960.1 (G), Q971.1 (G)
- net AB2: now also Q648.3 (D), R407.2
- net AB7: now reaches Q653.3 (D), R414.2
- net AB7: now also Q1044.1 (G), Q1100.1 (G), Q1203.1 (G), Q907.1 (G), Q930.1 (G), Q959.1 (G)
- net AA2: now reaches Q1083.1 (G), Q969.1 (G), Q972.1 (G), Q974.1 (G)
- net AA2: now also Q638.3 (D), R399.2
- net AA1: now reaches Q637.3 (D), R398.2
- net AA1: now also Q1073.1 (G), Q949.1 (G), Q951.1 (G), Q955.1 (G)
- net AB4: now reaches Q1026.1 (G), Q1167.1 (G), Q947.1 (G), Q995.1 (G)
- net AB4: now also Q650.3 (D), R409.2
- net AB6: now reaches Q1033.1 (G), Q1076.1 (G), Q1191.1 (G), Q958.1 (G)
- net AB6: now also Q652.3 (D), R413.2
- net AB0: now reaches Q644.3 (D), R405.2
- net AB0: now also Q1123.1 (G), Q921.1 (G), Q931.1 (G), Q932.1 (G)
- net AA5: now reaches Q641.3 (D), R402.2
- net AA5: now also Q1022.1 (G), Q1049.1 (G), Q1051.1 (G), Q1090.1 (G)
- net AB3: now reaches Q1155.1 (G), Q945.1 (G), Q978.1 (G), Q998.1 (G)
- net AB3: now also Q649.3 (D), R408.2
- net AB5: now reaches Q1011.1 (G), Q1048.1 (G), Q1179.1 (G), Q956.1 (G)
- net AB5: now also Q651.3 (D), R412.2
- net AB1: now reaches Q647.3 (D), R406.2
- net AB1: now also Q1131.1 (G), Q933.1 (G), Q946.1 (G), Q948.1 (G)
- net AA6: now reaches Q642.3 (D), R403.2
- net AA6: now also Q1034.1 (G), Q1077.1 (G), Q1079.1 (G), Q1099.1 (G)
- new net: D87.2, R393.2, R394.2
- new net: D132.1, Q793.3 (D)
- new net: D133.1, Q794.3 (D)
- new net: D133.2, R762.2, R763.2
- new net: D134.2, R764.2, R765.2
- new net: D142.2, R780.2, R781.2
- new net: D143.1, Q804.3 (D)
- new net: D143.2, R782.2, R783.2
- new net: D141.1, Q802.3 (D)
- new net: D141.2, R778.2, R779.2
- new net: D132.2, R760.2, R761.2
- new net: D135.2, R766.2, R767.2
- new net: D142.1, Q803.3 (D)
- new net: D13.2, R380.2, R79.2
- new net: D140.2, R776.2, R777.2
- new net: D140.1, Q801.3 (D)
- new net: D138.2, R772.2, R773.2
- new net: D84.2, R385.2, R386.2
- new net: D139.2, R774.2, R775.2
- new net: D138.1, Q799.3 (D)
- new net: D146.1, Q807.3 (D)
- new net: D146.2, R788.2, R789.2
- new net: D86.2, R391.2, R392.2
- new net: D144.2, R784.2, R785.2
- new net: D135.1, Q796.3 (D)
- new net: D137.1, Q798.3 (D)
- new net: D137.2, R770.2, R771.2
- new net: D147.1, Q808.3 (D)
- new net: D84.1, Q135.3 (D)
- new net: D87.1, Q635.3 (D)
- new net: D147.2, R790.2, R791.2
- new net: D14.2, R381.2, R382.2
- new net: D145.2, R786.2, R787.2
- new net: D14.1, Q38.3 (D)
- new net: D12.2, R75.2, R78.2
- new net: D136.2, R768.2, R769.2
- new net: D134.1, Q795.3 (D)
- new net: D139.1, Q800.3 (D)
- new net: D83.1, Q39.3 (D)
- new net: D83.2, R383.2, R384.2
- new net: D85.2, R387.2, R390.2
- new net: D85.1, Q633.3 (D)
- new net: D86.1, Q634.3 (D)
- new net: D13.1, Q37.3 (D)
- new net: D12.1, Q36.3 (D)
- new net: D144.1, Q805.3 (D)
- new net: D145.1, Q806.3 (D)
- new net: D136.1, Q797.3 (D)
