File: PCB_S/Level_shifter_FPGA_V1.0/Level_shifter_FPGA_V1.0/Level_shifter_FPGA_V1.0.kicad_sch (KiCad schematic)
At the start: 165 parts, among them J1 Conn_02x20_Counter_Clockwise, J2 Conn_02x05_Counter_Clockwise, J3 Conn_01x02_Pin, J4 Conn_01x02_Pin, J5 Conn_01x02_Pin, J6 Conn_02x08_Counter_Clockwise, J7 Conn_02x08_Counter_Clockwise, Q10 2N7002, Q11 2N7002, Q12 2N7002, Q13 2N7002, Q14 2N7002, Q15 2N7002, Q16 2N7002, Q17 2N7002, Q18 2N7002, Q19 2N7002, Q20 2N7002, Q21 2N7002, Q22 2N7002, Q23 2N7002, Q24 2N7002, Q25 2N7002, Q26 2N7002, Q27 2N7002, Q28 2N7002, Q29 2N7002, Q30 2N7002, Q31 2N7002, Q32 2N7002, Q33 2N7002, Q34 2N7002, Q35 2N7002, Q36 2N7002, Q37 2N7002, Q38 2N7002, Q39 2N7002, Q40 2N7002, Q41 2N7002, Q42 2N7002, Q43 2N7002, Q44 2N7002, Q45 2N7002, Q46 2N7002, Q47 2N7002, Q48 2N7002, Q49 2N7002, Q5 2N7002, Q50 2N7002, Q51 2N7002, Q52 2N7002, Q53 2N7002, Q54 2N7002, Q55 2N7002, Q56 2N7002, Q57 2N7002, Q58 2N7002, Q59 2N7002, Q6 2N7002, Q60 2N7002, Q61 2N7002, Q62 2N7002, Q63 2N7002, Q64 2N7002, Q65 2N7002, Q66 2N7002, Q67 2N7002, Q68 2N7002, Q69 2N7002, Q7 2N7002, Q70 2N7002, Q71 2N7002, Q72 2N7002, Q73 2N7002, Q74 2N7002, Q75 2N7002, Q76 2N7002, Q77 2N7002, Q78 2N7002, Q79 2N7002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

Commit message: Controller unit v1.0 done & Level Shifter fpga v1.0 done
Parts:
- removed J1: Conn_02x20_Counter_Clockwise, Connector_PinSocket_2.54mm:PinSocket_2x20_P2.54mm_Vertical, symbol Connector_Generic:Conn_02x20_Counter_Clockwise
- removed J2: Conn_02x05_Counter_Clockwise, Connector_PinHeader_2.54mm:PinHeader_2x05_P2.54mm_Vertical, symbol Connector_Generic:Conn_02x05_Counter_Clockwise
- removed J3, J4: Conn_01x02_Pin, Connector_PinSocket_2.54mm:PinSocket_1x02_P2.54mm_Vertical, symbol Connector:Conn_01x02_Pin
- removed J6, J7: Conn_02x08_Counter_Clockwise, Connector_PinHeader_2.54mm:PinHeader_2x08_P2.54mm_Vertical, symbol Connector_Generic:Conn_02x08_Counter_Clockwise
- removed Q88, Q89, Q90, Q91: 2N7002, Package_TO_SOT_SMD:SOT-23, symbol Transistor_FET:2N7002
- removed R22, R24: 3.3kΩ, PCM_JLCPCB:R_0402, symbol PCM_JLCPCB-Resistors:0402,3.3kΩ
- removed R70, R71: R, Resistor_THT:R_Axial_DIN0204_L3.6mm_D1.6mm_P7.62mm_Horizontal, symbol Device:R
- added C1, C2, C3, C4, C5, C6, C7, C8: 22uF, PCM_JLCPCB:C_0805, symbol PCM_JLCPCB-Capacitors:0805,22uF
- added D1, D2, D3: LED, LED_THT:LED_D3.0mm_FlatTop, symbol Device:LED
- added J1, J8: Conn_02x08_Odd_Even, Connector_PinSocket_2.54mm:PinSocket_2x08_P2.54mm_Vertical, symbol Connector_Generic:Conn_02x08_Odd_Even
- added J2: Conn_02x20_Odd_Even, Connector_PinSocket_2.54mm:PinSocket_2x20_P2.54mm_Vertical, symbol Connector_Generic:Conn_02x20_Odd_Even
- added J3: Conn_02x05_Odd_Even, Connector_PinSocket_2.54mm:PinSocket_2x05_P2.54mm_Vertical, symbol Connector_Generic:Conn_02x05_Odd_Even
- added J4: Conn_02x03_Odd_Even, Connector_PinSocket_2.54mm:PinSocket_2x03_P2.54mm_Vertical, symbol Connector_Generic:Conn_02x03_Odd_Even
- added J6, J7: Conn_01x02_Pin, Connector_PinSocket_2.54mm:PinSocket_1x02_P2.54mm_Vertical, symbol Connector:Conn_01x02_Pin
- added Q1, Q2, Q3, Q4: 2N7002, Package_TO_SOT_SMD:SOT-23, symbol Transistor_FET:2N7002
- added R22, R24: R, Resistor_THT:R_Axial_DIN0204_L3.6mm_D1.6mm_P7.62mm_Horizontal, symbol Device:R
- added R70, R71, R72, R73, R74: 3.3kΩ, PCM_JLCPCB:R_0402, symbol PCM_JLCPCB-Resistors:0402,3.3kΩ
Connections:
- net 3.3V: now also R11.1, R14.1, R19.1, R23.1, R28.1, R31.1, R34.1, R40.1, R42.1, R44.1, R48.1, R50.1, R54.1, R56.1, R58.1, R60.1, R62.1, R64.1, R66.1, R68.1, J2.30 (Pin_30), J4.2 (Pin_2), R70.1, R72.1, R73.1; no longer R12.1, R15.1, R18.1, R21.1, R27.1, R30.1, R35.1, R39.1, R41.1, R43.1, R47.1, R49.1, R51.1, R55.1, R57.1, R59.1, R61.1, R63.1, R65.1, R67.1
- net 5V: now also J2.12 (Pin_12), J4.4 (Pin_4), R74.1
- net A0: now also Q56.1 (G), J1.15 (Pin_15); no longer Q54.1 (G)
- net A1: now also Q58.1 (G), J1.13 (Pin_13); no longer Q56.1 (G)
- net A10: now also Q76.1 (G), J1.12 (Pin_12); no longer Q74.1 (G)
- net A11: now also Q78.1 (G), J1.10 (Pin_10); no longer Q76.1 (G)
- net A12: now also Q80.1 (G), J1.8 (Pin_8); no longer Q78.1 (G)
- net A13: now also Q82.1 (G), J1.6 (Pin_6); no longer Q80.1 (G)
- net A14: now also Q84.1 (G), J1.4 (Pin_4); no longer Q82.1 (G)
- net A15: now also Q86.1 (G), J1.2 (Pin_2); no longer Q84.1 (G)
- net A2: now also Q60.1 (G), J1.11 (Pin_11); no longer Q58.1 (G)
- net A3: now also Q62.1 (G), J1.9 (Pin_9); no longer Q60.1 (G)
- net A4: now also Q64.1 (G), J1.7 (Pin_7); no longer Q62.1 (G)
- net A5: now also Q66.1 (G), J1.5 (Pin_5); no longer Q64.1 (G)
- net A6: now also Q68.1 (G), J1.3 (Pin_3); no longer Q66.1 (G)
- net A7: now also Q70.1 (G), J1.1 (Pin_1); no longer Q68.1 (G)
- net A8: now also Q72.1 (G), J1.16 (Pin_16); no longer Q70.1 (G)
- net A9: now also Q74.1 (G), J1.14 (Pin_14); no longer Q72.1 (G)
- net ADR0: now also Q57.3 (D), R42.2, J2.14 (Pin_14); no longer Q55.3 (D), R35.2
- net ADR1: now also Q59.3 (D), R44.2, J2.13 (Pin_13); no longer Q57.3 (D), R37.2
- net ADR10: now also Q77.3 (D), R62.2, J2.24 (Pin_24); no longer Q75.3 (D), R55.2
- net ADR11: now also Q79.3 (D), R64.2, J2.23 (Pin_23); no longer Q77.3 (D), R57.2
- net ADR12: now also Q81.3 (D), R66.2, J2.26 (Pin_26); no longer Q79.3 (D), R59.2
- net ADR13: now also Q83.3 (D), R68.2, J2.25 (Pin_25); no longer Q81.3 (D), R61.2
- net ADR14: now also Q85.3 (D), J2.28 (Pin_28), R70.2; no longer Q83.3 (D), R63.2
- net ADR15: now also Q87.3 (D), J2.27 (Pin_27), R72.2; no longer Q85.3 (D), R65.2
- net ADR2: now also Q61.3 (D), R46.2, J2.16 (Pin_16); no longer Q59.3 (D), R39.2
- net ADR3: now also Q63.3 (D), R48.2, J2.15 (Pin_15); no longer Q61.3 (D), R41.2
- net ADR4: now also Q65.3 (D), R50.2, J2.18 (Pin_18); no longer Q63.3 (D), R43.2
- net ADR5: now also Q67.3 (D), R53.2, J2.17 (Pin_17); no longer Q65.3 (D), R46.2
- net ADR6: now also Q69.3 (D), R54.2, J2.20 (Pin_20); no longer Q67.3 (D), R47.2
- net ADR7: now also Q71.3 (D), R56.2, J2.19 (Pin_19); no longer Q69.3 (D), R49.2
- net ADR8: now also Q73.3 (D), R58.2, J2.22 (Pin_22); no longer Q71.3 (D), R51.2
- net ADR9: now also Q75.3 (D), R60.2, J2.21 (Pin_21); no longer Q73.3 (D), R53.2
- net Buss0: now also Q5.1 (G), Q6.3 (D), J8.1 (Pin_1); no longer Q7.1 (G), Q8.3 (D)
- net Buss1: now also Q12.1 (G), J8.3 (Pin_3); no longer Q13.1 (G)
- net Buss2: now also Q21.3 (D), J8.5 (Pin_5); no longer Q20.3 (D)
- net Buss3: now also Q27.1 (G), Q28.3 (D), J8.7 (Pin_7); no longer Q25.1 (G), Q26.3 (D)
- net Buss4: now also Q33.1 (G), Q34.3 (D), J8.9 (Pin_9); no longer Q31.1 (G), Q32.3 (D)
- net Buss5: now also Q39.1 (G), Q40.3 (D), J8.11 (Pin_11); no longer Q37.1 (G), Q38.3 (D)
- net Buss6: now also Q45.1 (G), Q46.3 (D), J8.13 (Pin_13); no longer Q43.1 (G), Q44.3 (D)
- net Buss7: now also Q51.1 (G), Q52.3 (D), J8.15 (Pin_15); no longer Q49.1 (G), Q50.3 (D)
- net CLK: now also Q25.3 (D), J8.6 (Pin_6), R24.1
- net CLK L: now also Q20.1 (G), J2.32 (Pin_32)
- net D0: now also Q8.3 (D), R14.2, Q4.1 (G); no longer Q10.3 (D), Q6.1 (G), R12.2
- net D1: now also Q11.1 (G), R19.2; no longer Q12.1 (G), R15.2
- net D2: now also Q23.3 (D), R23.2; no longer Q22.3 (D), R18.2
- net D3: now also Q26.1 (G), Q30.3 (D), R28.2; no longer Q24.1 (G), Q28.3 (D), R21.2
- net D4: now also Q32.1 (G), Q36.3 (D), R31.2; no longer Q30.1 (G), Q34.3 (D)
- net D5: now also Q38.1 (G), Q42.3 (D), R34.2; no longer Q36.1 (G), Q40.3 (D), R27.2
- net D6: now also Q44.1 (G), Q48.3 (D), R37.2; no longer Q42.1 (G), Q46.3 (D), R30.2
- net D7: now also Q50.1 (G), Q54.3 (D), R40.2; no longer Q48.1 (G), Q52.3 (D)
- net GND: now also Q10.2 (S), Q20.2 (S), Q22.2 (S), Q26.2 (S), Q32.2 (S), Q38.2 (S), Q44.2 (S), Q50.2 (S), C1.2, C2.2, C3.2, C4.2, C5.2, C6.2, C7.2, C8.2, D1.1 (K), D2.1 (K), D3.1 (K), J2.11 (Pin_11), J2.29 (Pin_29), J3.9 (Pin_9), J4.1 (Pin_1), J4.3 (Pin_3), J4.5 (Pin_5), J6.2 (Pin_2), J7.2 (Pin_2), J8.10 (Pin_10), J8.14 (Pin_14), J8.4 (Pin_4), Q1.2 (S), Q2.2 (S), Q3.2 (S), Q4.2 (S); no longer Q21.2 (S), Q23.2 (S), Q30.2 (S), Q36.2 (S), Q42.2 (S), Q48.2 (S), Q54.2 (S), Q6.2 (S)
- net RST: now also Q13.3 (D), R18.2, J8.8 (Pin_8); no longer R69.2
- net RST L: now also Q10.1 (G), J2.33 (Pin_33)
- net RW L: now also R11.2, J2.31 (Pin_31), Q3.3 (D); no longer Q87.3 (D), R67.2
- net R/W: now also Q22.1 (G), Q29.1 (G), Q35.1 (G), Q41.1 (G), Q47.1 (G), Q53.1 (G), Q7.1 (G), J8.12 (Pin_12), Q1.1 (G), Q2.1 (G); no longer Q21.1 (G), Q27.1 (G), Q33.1 (G), Q39.1 (G), Q45.1 (G), Q5.1 (G), Q51.1 (G), Q86.1 (G), Q9.1 (G)
- net VCC: now also R12.1, R15.1, R18.1, R21.1, R27.1, R30.1, R33.1, R35.1, R39.1, R41.1, R43.1, R45.1, R47.1, R49.1, R51.1, R55.1, R57.1, R59.1, R61.1, R63.1, R65.1, R67.1, C1.1, C2.1, C3.1, C4.1, C5.1, C6.1, C7.1, C8.1, J4.6 (Pin_6), J6.1 (Pin_1), J7.1 (Pin_1), J8.16 (Pin_16), J8.2 (Pin_2), R22.2, R24.2, R71.1; no longer R11.1, R14.1, R19.1, R23.1, R28.1, R31.1, R34.1, R40.1, R42.1, R44.1, R48.1, R50.1, R54.1, R56.1, R58.1, R60.1, R62.1, R64.1, R66.1, R68.1
- net at Q60.3 (D), Q61.1 (G): now also R45.2; no longer R40.2
- net at Q72.3 (D), Q73.1 (G): now also R57.2; no longer R52.2
- net at Q86.3 (D), Q87.1 (G): now also R71.2; no longer R66.2
- net at Q45.3 (D): now also Q48.1 (G), R36.2; no longer Q44.2 (S)
- net at Q33.3 (D): now also Q36.1 (G), R30.2; no longer Q32.2 (S)
- net at Q39.3 (D): now also Q42.1 (G), R33.2; no longer Q38.2 (S)
- net at Q82.3 (D), Q83.1 (G): now also R67.2; no longer R62.2
- net at Q76.3 (D), Q77.1 (G): now also R61.2; no longer R56.2
- net at Q74.3 (D), Q75.1 (G): now also R59.2; no longer R54.2
- net at Q27.3 (D): now also Q30.1 (G), R26.2; no longer Q26.2 (S)
- net at Q78.3 (D), Q79.1 (G): now also R63.2; no longer R58.2
- net at Q62.3 (D), Q63.1 (G): now also R47.2; no longer R42.2
- net at R4.2: now also J2.10 (Pin_10)
- net at Q84.3 (D), Q85.1 (G): now also R69.2; no longer R64.2
- net at Q70.3 (D), Q71.1 (G): now also R55.2; no longer R50.2
- net at Q68.3 (D), Q69.1 (G): now also R52.2; no longer R48.2
- net at Q80.3 (D), Q81.1 (G): now also R65.2; no longer R60.2
- net at Q66.3 (D), Q67.1 (G): now also R51.2
- net at Q51.3 (D): now also Q54.1 (G), R39.2; no longer Q50.2 (S)
- net at R5.1: now also J2.3 (Pin_3)
- net at Q58.3 (D), Q59.1 (G): now also R43.2; no longer R38.2
- net at Q64.3 (D), Q65.1 (G): now also R49.2; no longer R44.2
- net at R1.2: now also J2.4 (Pin_4)
- net at Q11.3 (D): now also Q14.1 (G), R16.2; no longer Q10.2 (S)
- net at R2.2: now also J2.6 (Pin_6)
- net at R7.1: now also J2.7 (Pin_7)
- net at Q56.3 (D), Q57.1 (G): now also R41.2; no longer R36.2
- net at R3.2: now also J2.8 (Pin_8)
- net at R8.1: now also J2.9 (Pin_9)
- net at R6.1: now also J2.5 (Pin_5)
- new net: Q38.3 (D), Q40.1 (G), R32.2
- new net: Q10.3 (D), Q13.1 (G), R15.2
- new net: Q26.3 (D), Q28.1 (G), R25.2
- new net: Q42.2 (S), Q43.3 (D)
- new net: Q17.1 (G), Q2.3 (D), Q24.1 (G), Q31.1 (G), Q37.1 (G), Q43.1 (G), Q49.1 (G), Q55.1 (G), Q9.1 (G), R10.2
- new net: Q30.2 (S), Q31.3 (D)
- new net: Q44.3 (D), Q46.1 (G), R35.2
- new net: Q50.3 (D), Q52.1 (G), R38.2
- new net: Q48.2 (S), Q49.3 (D)
- new net: Q54.2 (S), Q55.3 (D)
- new net: Q32.3 (D), Q34.1 (G), R29.2
- new net: Q5.3 (D), Q8.1 (G), R13.2
- new net: J2.39 (Pin_39), J3.1 (Pin_1)
- new net: J2.2 (Pin_2), J3.10 (Pin_10)
- new net: J2.40 (Pin_40), J3.2 (Pin_2)
- new net: J2.37 (Pin_37), J3.3 (Pin_3)
- new net: J2.38 (Pin_38), J3.4 (Pin_4)
- new net: J2.35 (Pin_35), J3.5 (Pin_5)
- new net: J2.36 (Pin_36), J3.6 (Pin_6)
- new net: J2.1 (Pin_1), J3.7 (Pin_7)
- new net: J2.34 (Pin_34), J3.8 (Pin_8)
- new net: Q19.3 (D), Q23.1 (G), R21.2
- new net: Q23.2 (S), Q24.3 (D)
- new net: Q18.3 (D), Q21.1 (G), R20.2
- new net: Q21.2 (S), Q22.3 (D)
- new net: Q12.3 (D), Q16.1 (G), R17.2
- new net: Q1.3 (D), Q3.1 (G), R9.2
- new net: Q6.2 (S), Q7.3 (D)
- new net: D3.2 (A), R74.2
- new net: D2.2 (A), R73.2
- new net: Q4.3 (D), Q6.1 (G), R12.2
- new net: Q20.3 (D), Q25.1 (G), R22.1
- new net: D1.2 (A), R27.2
- new net: Q36.2 (S), Q37.3 (D)

Commit message: order tomorrow
Parts:
- removed D1, D2, D3: LED, LED_THT:LED_D3.0mm_FlatTop, symbol Device:LED
- removed R1, R2, R22, R24, R3, R4, R5, R6, R7, R8: R, Resistor_THT:R_Axial_DIN0204_L3.6mm_D1.6mm_P7.62mm_Horizontal, symbol Device:R
- added D1, D2, D3: Red, PCM_JLCPCB:D_0603, symbol PCM_JLCPCB-Diodes:LED,0603,Red
- added R1, R2, R22, R24, R3, R4, R5, R6, R7, R8: 10kΩ, PCM_JLCPCB:R_1206, symbol PCM_JLCPCB-Resistors:1206,10kΩ
Connections:
- net 3.3V: now also J2.11 (Pin_11); no longer J2.30 (Pin_30)
- net 5V: now also J2.29 (Pin_29); no longer J2.12 (Pin_12)
- net CLK: now also R24.2
- net D0: now also R1.1
- net D1: now also R2.2
- net D2: now also R3.1
- net D3: now also R4.2
- net D4: now also R5.1
- net D5: now also R6.2
- net D6: now also R7.1
- net D7: now also R8.2
- net GND: now also J2.12 (Pin_12), J2.30 (Pin_30), D1.1, D2.1, D3.1; no longer J2.11 (Pin_11), J2.29 (Pin_29)
- net VCC: now also R22.1, R24.1
- net at J2.10 (Pin_10): now also R7.2
- net at J2.6 (Pin_6): now also R3.2
- net at J2.7 (Pin_7): now also R6.1
- net at J2.3 (Pin_3): now also R2.1
- net at J2.4 (Pin_4): now also R1.2
- net at J2.5 (Pin_5): now also R4.1
- net at J2.8 (Pin_8): now also R5.2
- net at J2.9 (Pin_9): now also R8.1
- net at R74.2: now also D3.2
- net at R73.2: now also D2.2
- net at Q20.3 (D), Q25.1 (G): now also R22.2
- net at R27.2: now also D1.2
